File: karca.kicad_sch (KiCad schematic)
At the start: 14 parts

Commit message: i am very smart. no person can match my intellectual prowess. chinese pcb manufacturers tremble before me
Parts:
- added BT1: Battery, symbol Device:Battery
- added D5: D, symbol Device:D
- added SW1: SW_SPDT, symbol Switch:SW_SPDT
- C1, C2, C3, C4: renamed from C?; footprint (none) -> Capacitor_SMD:C_1206_3216Metric
- R1, R2, R3, R4: renamed from R?; footprint (none) -> Resistor_SMD:R_1206_3216Metric
- U1: renamed from U?; footprint (none) -> Package_TO_SOT_SMD:TO-263-3_TabPin2
- gave numbers to parts that had none: 5
Connections:
- net GND: now also C4.2, BT1.2 (-)
- net +12V: now reaches C1.1, D1.1 (K), U1.3 (VI)
- net +12V: now also C2.1, D2.1 (K), U2.3 (VI), D5.1 (K)
- new net: BT1.1 (+), SW1.2 (B)
- new net: D5.2 (A), SW1.1 (A)
- no-connect marks 0 -> 1

Commit message: commit
Parts:
- removed BT1: Battery, symbol Device:Battery
- removed C1, C2, C3, C4: C, Capacitor_SMD:C_1206_3216Metric, symbol Device:C
- removed D1, D2: D_Schottky, symbol Device:D_Schottky
- removed D3, D4: LED, symbol Device:LED
- removed D5: D, symbol Device:D
- removed R1, R2, R3, R4: R_US, Resistor_SMD:R_1206_3216Metric, symbol Device:R_US
- removed SW1: SW_SPDT, symbol Switch:SW_SPDT
- removed U1: LM1084-ADJ, Package_TO_SOT_SMD:TO-263-3_TabPin2, symbol Regulator_Linear:LM1084-ADJ
- removed U2: LM1084-5.0, symbol Regulator_Linear:LM1084-5.0
Connections:
- no-connect marks 1 -> 2
Other:
- added sheet Drivers (drivers.kicad_sch)
- added sheet Load Cell Inamps (lc_inamps.kicad_sch)
- added sheet regulators (regulators.kicad_sch)

Commit message: secret arca meetings
Other:
- added sheet Load Cell Anti-Aliasing (lc_anti_alias.kicad_sch)
- added sheet PT Amplification (pt_amps.kicad_sch)

Commit message: Added pages
Other:
- added sheet ADCs (adc.kicad_sch)
- added sheet Raspberry Pi (pi.kicad_sch)
- added sheet Thermocouples (thermocouples.kicad_sch)
Changed lines of the file:
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@@
   (no_connect (at 95.25 86.36))
   (no_connect (at 156.21 69.85))
+  (sheet (at 91.44 93.98) (size 21.59 16.51) (fields_autoplaced)
+    (stroke (width 0.1524) (type solid) (color 0 0 0 0))
+    (fill (color 0 0 0 0.0000))
+    (property "Sheet name" "Raspberry Pi" (id 0) (at 91.44 93.2684 0)
+      (effects (font (size 1.27 1.27)) (justify left bottom))
+    )
+    (property "Sheet file" "pi.kicad_sch" (id 1) (at 91.44 111.0746 0)
+      (effects (font (size 1.27 1.27)) (justify left top))
+    )
+  )
   (sheet (at 36.83 40.64) (size 25.4 17.78) (fields_autoplaced)
     (stroke (width 0.1524) (type solid) (color 0 0 0 0))
@@
     )
     (property "Sheet file" "regulators.kicad_sch" (id 1) (at 36.83 59.0046 0)
+      (effects (font (size 1.27 1.27)) (justify left top))
+    )
+  )
+  (sheet (at 92.71 35.56) (size 21.59 15.24) (fields_autoplaced)
+    (stroke (width 0.1524) (type solid) (color 0 0 0 0))
+    (fill (color 0 0 0 0.0000))
+    (property "Sheet name" "Thermocouples" (id 0) (at 92.71 34.8484 0)
+      (effects (font (size 1.27 1.27)) (justify left bottom))
+    )
+    (property "Sheet file" "thermocouples.kicad_sch" (id 1) (at 92.71 51.3846 0)
       (effects (font (size 1.27 1.27)) (justify left top))
     )
@@
     )
   )
+  (sheet (at 90.17 68.58) (size 21.59 13.97) (fields_autoplaced)
+    (stroke (width 0.1524) (type solid) (color 0 0 0 0))
+    (fill (color 0 0 0 0.0000))
+    (property "Sheet name" "ADCs" (id 0) (at 90.17 67.8684 0)
+      (effects (font (size 1.27 1.27)) (justify left bottom))
+    )
+    (property "Sheet file" "adc.kicad_sch" (id 1) (at 90.17 83.1346 0)
+      (effects (font (size 1.27 1.27)) (justify left top))
+    )
+  )
   (sheet_instances
     (path "/" (page "1"))
@@
     (path "/5be75c7d-aeaf-4651-903f-4fa3c98c0d90" (page "5"))
     (path "/d974749e-215f-46b5-a007-0416cfb921b4" (page "6"))
+    (path "/2ecca342-0668-4e36-84dc-b8a6ec02bba5" (page "7"))
+    (path "/f9b56273-510a-4f1f-8845-adebb323cd86" (page "8"))
+    (path "/1d2f7b4c-e83f-4cee-b3c6-61e1093bdc7e" (page "9"))
   )
   (symbol_instances

Commit message: first revision of full schematic copied over
Other:
- note added: "ARCA 2.0"
- note added: "Control system and data collection for inert flow and static hot fires of experimental hybrid engines. Compatible Engines: - Luna - Proxima - Titan II ARCA 2.0 is a re-spin of ARCA, which is a design upgrade on "Mk 1.1" Avionics Lead: Spencer Darwall Subteam Lead: Amy Danjul Avionics Engineers: Clayton Ramsey, Justin Guilak, Riley Kuhlman, Matthew Nutt, Mitchell Hoffman, Jonah Yi, Jonathan Enriqu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"
- company: (none) -> Rice Eclipse
- title: (none) -> ARCA 2.0

Commit message: added schematic pdf for review
Other:
- note added: "Control system and data collection for inert flow and static hot fires of experimental hybrid engines. Compatible Engines: - Luna - Proxima - Titan II ARCA 2.0 is a re-spin of ARCA, which is a design upgrade on "Mk 1.1" Avionics Lead: Spencer Darwall Subteam Lead: Amy Danjul Avionics Engineers: Clayton Ramsey, Rosemary Lach, Justin Guilak, Riley Kuhlman, Matthew Nutt, Mitchell Hoffman, Jonah Yi, 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"
- note removed: "Control system and data collection for inert flow and static hot fires of experimental hybrid engines. Compatible Engines: - Luna - Proxima - Titan II ARCA 2.0 is a re-spin of ARCA, which is a design upgrade on "Mk 1.1" Avionics Lead: Spencer Darwall Subteam Lead: Amy Danjul Avionics Engineers: Clayton Ramsey, Justin Guilak, Riley Kuhlman, Matthew Nutt, Mitchell Hoffman, Jonah Yi, Jonathan Enriqu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"
