File: karca.kicad_sch (KiCad schematic)
At the start: 0 parts

Commit message: done schematiccing after design review
Other:
- sheet Load Cell Inamps renamed Load Cells
- removed sheet ADCs
- removed sheet Load Cell Anti-Aliasing
- sheet Drivers ports: added DRV_CTL_1, DRV_CTL_2, DRV_CTL_3, DRV_CTL_4, DRV_CTL_5, DRV_CTL_6; removed none
- sheet Load Cells ports: added CS, SPI_CLK, SPI_MISO, SPI_MOSI; removed none
- sheet PT Amplification ports: added CS, SPI_CLK, SPI_MISO, SPI_MOSI; removed none
- sheet Raspberry Pi ports: added ADC1_CS, ADC2_CS, ADC3_CS, DRV_CTL_1, DRV_CTL_2, DRV_CTL_3, DRV_CTL_4, DRV_CTL_5, DRV_CTL_6, SPI_CLK, SPI_MISO, SPI_MOSI; removed none
- sheet Thermocouples ports: added CS, SPI_CLK, SPI_MISO, SPI_MOSI; removed none

Commit message: cleaned up PT footprint
Parts:
- added H1, H2, H3, H4: MountingHole, MountingHole:MountingHole_3.2mm_M3, symbol Mechanical:MountingHole
