File: regulators.kicad_sch (KiCad schematic)
At the start: 24 parts, among them J1 Conn_01x02_Female, J2 Conn_01x02_Female, J3 Conn_01x02_Female, J4 Conn_01x04_Female, J5 Conn_01x02_Female, SW1 1101M2S3CQE2, SW2 1101M2S3CQE2, U1 LM1084-ADJ, U2 LM1084-5.0

Commit message: grouped components on PCB
Changed lines of the file:
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@@
   (junction (at 140.97 83.82) (diameter 0) (color 0 0 0 0)
-  )
-  (junction (at 90.17 59.69) (diameter 0) (color 0 0 0 0)
   )
   (junction (at 162.56 83.82) (diameter 0) (color 0 0 0 0)
@@
     (stroke (width 0) (type default) (color 0 0 0 0))
   )
+  (wire (pts (xy 85.09 59.69) (xy 92.71 59.69))
+    (stroke (width 0) (type default) (color 0 0 0 0))
+  )
   (wire (pts (xy 191.77 44.45) (xy 189.23 44.45))
     (stroke (width 0) (type default) (color 0 0 0 0))
@@
     (stroke (width 0) (type default) (color 0 0 0 0))
   )
-  (wire (pts (xy 85.09 59.69) (xy 90.17 59.69))
-    (stroke (width 0) (type default) (color 0 0 0 0))
-  )
   (wire (pts (xy 137.16 128.27) (xy 140.97 128.27))
     (stroke (width 0) (type default) (color 0 0 0 0))
@@
   )
   (wire (pts (xy 140.97 93.98) (xy 140.97 92.71))
-    (stroke (width 0) (type default) (color 0 0 0 0))
-  )
-  (wire (pts (xy 90.17 59.69) (xy 92.71 59.69))
     (stroke (width 0) (type default) (color 0 0 0 0))
   )
@@
   (symbol (lib_id "Connector:Conn_01x02_Female") (at 133.35 58.42 0) (unit 1)
     (in_bom yes) (on_board yes) (fields_autoplaced)
-    (property "Reference" "J3" (id 0) (at 134.62 58.4199 0)
+    (property "Reference" "J3" (id 0) (at 134.62 59.6899 0)
       (effects (font (size 1.27 1.27)) (justify left))
     )
     (property "Value" "Conn_01x02_Female" (id 1) (at 134.62 60.9599 0)
-      (effects (font (size 1.27 1.27)) (justify left))
+      (effects (font (size 1.27 1.27)) (justify left) hide)
     )
     (property "Footprint" "Connector_PinHeader_2.54mm:PinHeader_1x02_P2.54mm_Vertical" (id 2) (at 133.35 58.42 0)
@@
   (symbol (lib_id "Connector:Conn_01x02_Female") (at 194.31 60.96 0) (unit 1)
     (in_bom yes) (on_board yes) (fields_autoplaced)
-    (property "Reference" "J5" (id 0) (at 195.58 60.9599 0)
+    (property "Reference" "J5" (id 0) (at 195.58 62.2299 0)
       (effects (font (size 1.27 1.27)) (justify left))
     )
     (property "Value" "Conn_01x02_Female" (id 1) (at 195.58 63.4999 0)
-      (effects (font (size 1.27 1.27)) (justify left))
+      (effects (font (size 1.27 1.27)) (justify left) hide)
     )
     (property "Footprint" "Connector_PinHeader_2.54mm:PinHeader_1x02_P2.54mm_Vertical" (id 2) (at 194.31 60.96 0)
@@
   (symbol (lib_id "Connector:Conn_01x04_Female") (at 196.85 39.37 0) (unit 1)
     (in_bom yes) (on_board yes) (fields_autoplaced)
-    (property "Reference" "J4" (id 0) (at 198.12 39.3699 0)
+    (property "Reference" "J4" (id 0) (at 198.12 40.6399 0)
       (effects (font (size 1.27 1.27)) (justify left))
     )
     (property "Value" "Conn_01x04_Female" (id 1) (at 198.12 41.9099 0)
-      (effects (font (size 1.27 1.27)) (justify left))
+      (effects (font (size 1.27 1.27)) (justify left) hide)
     )
     (property "Footprint" "Connector_PinHeader_2.54mm:PinHeader_1x04_P2.54mm_Vertical" (id 2) (at 196.85 39.37 0)
@@
   (symbol (lib_id "Connector:Conn_01x02_Female") (at 43.18 62.23 0) (mirror y) (unit 1)
     (in_bom yes) (on_board yes) (fields_autoplaced)
-    (property "Reference" "J1" (id 0) (at 43.815 57.15 0))
-    (property "Value" "Conn_01x02_Female" (id 1) (at 43.815 59.69 0))
+    (property "Reference" "J1" (id 0) (at 43.815 59.69 0))
+    (property "Value" "Conn_01x02_Female" (id 1) (at 43.815 59.69 0)
+      (effects (font (size 1.27 1.27)) hide)
+    )
     (property "Footprint" "Connector_PinHeader_2.54mm:PinHeader_1x02_P2.54mm_Vertical" (id 2) (at 43.18 62.23 0)
       (effects (font (size 1.27 1.27)) hide)
@@
   (symbol (lib_id "Connector:Conn_01x02_Female") (at 162.56 43.18 0) (unit 1)
     (in_bom yes) (on_board yes) (fields_autoplaced)
-    (property "Reference" "J2" (id 0) (at 163.83 43.1799 0)
+    (property "Reference" "J2" (id 0) (at 163.83 44.4499 0)
       (effects (font (size 1.27 1.27)) (justify left))
     )
     (property "Value" "Conn_01x02_Female" (id 1) (at 163.83 45.7199 0)
-      (effects (font (size 1.27 1.27)) (justify left))
+      (effects (font (size 1.27 1.27)) (justify left) hide)
     )
     (property "Footprint" "Connector_PinHeader_2.54mm:PinHeader_1x02_P2.54mm_Vertical" (id 2) (at 162.56 43.18 0)
@@
     (pin "1")
   )
-  (symbol (lib_id "power:PWR_FLAG") (at 90.17 59.69 0) (unit 1)
+  (symbol (lib_id "power:PWR_FLAG") (at 92.71 59.69 0) (unit 1)
     (in_bom yes) (on_board yes)
-    (property "Reference" "#FLG02" (id 0) (at 90.17 57.785 0)
-      (effects (font (size 1.27 1.27)) hide)
-    )
-    (property "Value" "PWR_FLAG" (id 1) (at 91.44 55.88 0))
-    (property "Footprint" "" (id 2) (at 90.17 59.69 0)
-      (effects (font (size 1.27 1.27)) hide)
-    )
-    (property "Datasheet" "~" (id 3) (at 90.17 59.69 0)
-      (effects (font (size 1.27 1.27)) hide)
-    )
+    (property "Reference" "#FLG02" (id 0) (at 92.71 57.785 0)
+      (effects (font (size 1.27 1.27)) hide)
+    )
+    (property "Value" "PWR_FLAG" (id 1) (at 93.98 55.88 0))
+    (property "Footprint" "" (id 2) (at 92.71 59.69 0)
+      (effects (font (size 1.27 1.27)) hide)
+    )
+    (property "Datasheet" "~" (id 3) (at 92.71 59.69 0)
+      (effects (font (size 1.27 1.27)) hide)
+    )
