File: regulators.kicad_sch (KiCad schematic)
At the start: 24 parts, among them J5 Conn_01x04_Female, SW1 S101031MS02Q, SW2 S101031MS02Q, U1 LM1084-ADJ, U2 LM1084-5.0

Commit message: enshrinkening of the board
Parts:
- removed CON_IGN_12: Screw_Terminal_01x02, 1190363:1190363, symbol Connector:Screw_Terminal_01x02
Other:
- note removed: "IGNITION RELAY"
Changed lines of the file:
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@@
   (junction (at 115.57 118.11) (diameter 0) (color 0 0 0 0)
   )
-  (junction (at 105.41 43.18) (diameter 0) (color 0 0 0 0)
-  )
   (wire (pts (xy 140.97 83.82) (xy 137.16 83.82))
     (stroke (width 0) (type default) (color 0 0 0 0))
@@
     (stroke (width 0) (type default) (color 0 0 0 0))
   )
-  (wire (pts (xy 105.41 27.94) (xy 105.41 43.18))
+  (wire (pts (xy 105.41 27.94) (xy 105.41 58.42))
     (stroke (width 0) (type default) (color 0 0 0 0))
   )
@@
     (stroke (width 0) (type default) (color 0 0 0 0))
   )
-  (wire (pts (xy 114.935 46.99) (xy 114.935 45.72))
-    (stroke (width 0) (type default) (color 0 0 0 0))
-  )
   (wire (pts (xy 83.185 59.69) (xy 92.71 59.69))
     (stroke (width 0) (type default) (color 0 0 0 0))
@@
     (stroke (width 0) (type default) (color 0 0 0 0))
   )
-  (wire (pts (xy 105.41 43.18) (xy 105.41 58.42))
-    (stroke (width 0) (type default) (color 0 0 0 0))
-  )
   (wire (pts (xy 165.1 83.82) (xy 162.56 83.82))
     (stroke (width 0) (type default) (color 0 0 0 0))
@@
     (stroke (width 0) (type default) (color 0 0 0 0))
   )
-  (wire (pts (xy 105.41 43.18) (xy 114.935 43.18))
-    (stroke (width 0) (type default) (color 0 0 0 0))
-  )
   (wire (pts (xy 64.135 59.69) (xy 75.565 59.69))
     (stroke (width 0) (type default) (color 0 0 0 0))
@@
   (wire (pts (xy 129.54 102.87) (xy 151.13 102.87))
     (stroke (width 0) (type default) (color 0 0 0 0))
-  )
-  (text "IGNITION RELAY" (at 118.11 40.64 0)
-    (effects (font (size 1.27 1.27)) (justify left bottom))
   )
   (text "Vo = 1.25V * (1+R1/R2)\n" (at 176.53 86.36 0)
@@
     (pin "2")
   )
-  (symbol (lib_id "power:GND") (at 114.935 46.99 0) (unit 1)
-    (in_bom yes) (on_board yes) (fields_autoplaced)
-    (property "Reference" "#PWR08" (id 0) (at 114.935 53.34 0)
-      (effects (font (size 1.27 1.27)) hide)
-    )
-    (property "Value" "GND" (id 1) (at 114.935 52.07 0))
-    (property "Footprint" "" (id 2) (at 114.935 46.99 0)
-      (effects (font (size 1.27 1.27)) hide)
-    )
-    (property "Datasheet" "" (id 3) (at 114.935 46.99 0)
-      (effects (font (size 1.27 1.27)) hide)
-    )
-    (pin "1")
-  )
   (symbol (lib_id "Device:LED") (at 162.56 88.9 90) (unit 1)
     (in_bom yes) (on_board yes) (fields_autoplaced)
@@
       (effects (font (size 1.27 1.27)) hide)
     )
-    (pin "1")
-    (pin "2")
-  )
-  (symbol (lib_id "Connector:Screw_Terminal_01x02") (at 120.015 43.18 0) (unit 1)
-    (in_bom yes) (on_board yes)
-    (property "Reference" "CON_IGN_12" (id 0) (at 122.555 44.4499 0)
-      (effects (font (size 1.27 1.27)) (justify left))
-    )
-    (property "Value" "Screw_Terminal_01x02" (id 1) (at 122.555 45.7199 0)
-      (effects (font (size 1.27 1.27)) (justify left) hide)
-    )
-    (property "Footprint" "1190363:1190363" (id 2) (at 120.015 43.18 0)
-      (effects (font (size 1.27 1.27)) hide)
-    )
-    (property "Datasheet" "~" (id 3) (at 120.015 43.18 0)
-      (effects (font (size 1.27 1.27)) hide)
-    )
