File: regulators.kicad_sch (KiCad schematic)
At the start: 23 parts, among them J5 Conn_01x04_Female, SW1 S101031MS02Q, SW2 S101031MS02Q, U1 LM1084-ADJ, U2 LM1084-5.0

Commit message: done routing on shrunk board
Connections:
- net FAN_PWR renamed FAN_POW
Changed lines of the file:
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@@
+    (stroke (width 0) (type default) (color 0 0 0 0))
+  )
+  (wire (pts (xy 125.095 27.94) (xy 134.62 27.94))
     (stroke (width 0) (type default) (color 0 0 0 0))
   )
@@
   )
   (wire (pts (xy 92.71 67.31) (xy 92.71 69.85))
-    (stroke (width 0) (type default) (color 0 0 0 0))
-  )
-  (wire (pts (xy 125.095 27.94) (xy 134.62 27.94))
     (stroke (width 0) (type default) (color 0 0 0 0))
   )
@@
     (effects (font (size 1.27 1.27)) (justify left bottom))
   )
+  (label "FAN_POW" (at 127 27.94 0)
+    (effects (font (size 1.27 1.27)) (justify left bottom))
+  )
   (label "10V_FB" (at 133.35 93.98 0)
     (effects (font (size 1.27 1.27)) (justify left bottom))
   )
-  (label "FAN_PWR" (at 125.73 27.94 0)
-    (effects (font (size 1.27 1.27)) (justify left bottom))
-  )

Commit message: done schematiccing after design review
Parts:
- removed J5: Conn_01x04_Female, Connector_PinSocket_2.54mm:PinSocket_1x04_P2.54mm_Vertical, symbol Connector:Conn_01x04_Female
- added TP1, TP2, TP3, TP4, TP5: TestPoint, symbol Connector:TestPoint
- D3, D5: value DO-214AC -> CDBA340-HF; footprint karca_custom_footprints:DO-214AC -> Diode_SMD:D_SMA
Connections:
- net +10V: now also TP4.1
- net +12V: now also TP3.1
- net +5V: now also TP5.1
- net 12V_CON: now also TP1.1
- net 12V_PRERECT: now also TP2.1
Other:
- moved on the sheet: CON_BAT1, SW1

Commit message: cleaned up PT footprint
Parts:
- TP1, TP2, TP3, TP4, TP5: footprint (none) -> TestPoint:TestPoint_Pad_D2.0mm
Changed lines of the file:
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@@
       (effects (font (size 1.27 1.27)) (justify left) hide)
     )
-    (property "Footprint" "" (id 2) (at 151.765 83.82 0)
+    (property "Footprint" "TestPoint:TestPoint_Pad_D2.0mm" (id 2) (at 151.765 83.82 0)
       (effects (font (size 1.27 1.27)) hide)
     )
@@
       (effects (font (size 1.27 1.27)) (justify left) hide)
     )
-    (property "Footprint" "" (id 2) (at 64.135 59.69 0)
+    (property "Footprint" "TestPoint:TestPoint_Pad_D2.0mm" (id 2) (at 64.135 59.69 0)
       (effects (font (size 1.27 1.27)) hide)
     )
@@
       (effects (font (size 1.27 1.27)) (justify left) hide)
     )
-    (property "Footprint" "" (id 2) (at 38.735 59.69 0)
+    (property "Footprint" "TestPoint:TestPoint_Pad_D2.0mm" (id 2) (at 38.735 59.69 0)
       (effects (font (size 1.27 1.27)) hide)
     )
@@
       (effects (font (size 1.27 1.27)) (justify left) hide)
     )
-    (property "Footprint" "" (id 2) (at 103.505 59.69 0)
+    (property "Footprint" "TestPoint:TestPoint_Pad_D2.0mm" (id 2) (at 103.505 59.69 0)
       (effects (font (size 1.27 1.27)) hide)
     )
@@
       (effects (font (size 1.27 1.27)) (justify left) hide)
     )
-    (property "Footprint" "" (id 2) (at 151.765 128.27 0)
-      (effects (font (size 1.27 1.27)) hide)
-    )
+    (property "Footprint" "TestPoint:TestPoint_Pad_D2.0mm" (id 2) (at 151.765 128.27 0)
+      (effects (font (size 1.27 1.27)) hide)
+    )

Commit message: waiting on mouser for footprints
Parts:
- renumbered LED_12V1 to LED13, LED_10V1 to LED14, LED_5V1 to LED15
Changed lines of the file:
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@@
   (symbol (lib_id "Device:LED") (at 92.71 63.5 90) (unit 1)
     (in_bom yes) (on_board yes) (fields_autoplaced)
-    (property "Reference" "LED_12V1" (id 0) (at 96.52 63.8174 90)
+    (property "Reference" "LED13" (id 0) (at 96.52 63.8174 90)
       (effects (font (size 1.27 1.27)) (justify right))
     )
@@
   (symbol (lib_id "Device:LED") (at 162.56 88.9 90) (unit 1)
     (in_bom yes) (on_board yes) (fields_autoplaced)
-    (property "Reference" "LED_10V1" (id 0) (at 166.37 89.2174 90)
+    (property "Reference" "LED14" (id 0) (at 166.37 89.2174 90)
       (effects (font (size 1.27 1.27)) (justify right))
     )
@@
   (symbol (lib_id "Device:LED") (at 151.13 133.35 90) (unit 1)
     (in_bom yes) (on_board yes) (fields_autoplaced)
-    (property "Reference" "LED_5V1" (id 0) (at 154.94 133.6674 90)
-      (effects (font (size 1.27 1.27)) (justify right))
-    )
+    (property "Reference" "LED15" (id 0) (at 154.94 133.6674 90)
+      (effects (font (size 1.27 1.27)) (justify right))
+    )

Commit message: final rev for jlc
Parts:
- R1: value 510 -> 1k
- R3: value 390 -> 820
- R5: value 150 -> 300
Changed lines of the file:
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@@
       (effects (font (size 1.27 1.27)) (justify left))
     )
-    (property "Value" "390" (id 1) (at 165.1 97.7899 0)
+    (property "Value" "820" (id 1) (at 165.1 97.7899 0)
       (effects (font (size 1.27 1.27)) (justify left))
     )
@@
       (effects (font (size 1.27 1.27)) (justify left))
     )
-    (property "Value" "510" (id 1) (at 95.25 74.9299 0)
+    (property "Value" "1k" (id 1) (at 95.25 74.9299 0)
       (effects (font (size 1.27 1.27)) (justify left))
     )
@@
       (effects (font (size 1.27 1.27)) (justify left))
     )
-    (property "Value" "150" (id 1) (at 153.67 142.2399 0)
-      (effects (font (size 1.27 1.27)) (justify left))
-    )
+    (property "Value" "300" (id 1) (at 153.67 142.2399 0)
+      (effects (font (size 1.27 1.27)) (justify left))
+    )

Commit message: started on opamp arrangement
Changed lines of the file:
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@@
       (effects (font (size 1.27 1.27)) hide)
     )
-    (property "Value" "GND" (id 1) (at 129.54 109.22 0))
+    (property "Value" "GND" (id 1) (at 129.54 109.22 0)
+      (effects (font (size 1.27 1.27)) hide)
+    )
     (property "Footprint" "" (id 2) (at 129.54 104.14 0)
       (effects (font (size 1.27 1.27)) hide)
@@
       (effects (font (size 1.27 1.27)) hide)
     )
-    (property "Value" "GND" (id 1) (at 151.13 149.86 0))
+    (property "Value" "GND" (id 1) (at 151.13 149.86 0)
+      (effects (font (size 1.27 1.27)) hide)
+    )
     (property "Footprint" "" (id 2) (at 151.13 144.78 0)
       (effects (font (size 1.27 1.27)) hide)
@@
       (effects (font (size 1.27 1.27)) hide)
     )
-    (property "Value" "GND" (id 1) (at 162.56 105.41 0))
+    (property "Value" "GND" (id 1) (at 162.56 105.41 0)
+      (effects (font (size 1.27 1.27)) hide)
+    )
     (property "Footprint" "" (id 2) (at 162.56 100.33 0)
       (effects (font (size 1.27 1.27)) hide)
@@
       (effects (font (size 1.27 1.27)) hide)
     )
-    (property "Value" "GND" (id 1) (at 114.3 66.04 0))
+    (property "Value" "GND" (id 1) (at 114.3 66.04 0)
+      (effects (font (size 1.27 1.27)) hide)
+    )
     (property "Footprint" "" (id 2) (at 114.3 60.96 0)
       (effects (font (size 1.27 1.27)) hide)
@@
       (effects (font (size 1.27 1.27)) hide)
     )
-    (property "Value" "GND" (id 1) (at 126.365 35.56 0))
+    (property "Value" "GND" (id 1) (at 126.365 35.56 0)
+      (effects (font (size 1.27 1.27)) hide)
+    )
     (property "Footprint" "" (id 2) (at 126.365 30.48 0)
       (effects (font (size 1.27 1.27)) hide)
@@
       (effects (font (size 1.27 1.27)) hide)
     )
-    (property "Value" "GND" (id 1) (at 92.71 82.55 0))
+    (property "Value" "GND" (id 1) (at 92.71 82.55 0)
+      (effects (font (size 1.27 1.27)) hide)
+    )
     (property "Footprint" "" (id 2) (at 92.71 77.47 0)
       (effects (font (size 1.27 1.27)) hide)
@@
       (effects (font (size 1.27 1.27)) hide)
     )
-    (property "Value" "GND" (id 1) (at 129.54 148.59 0))
+    (property "Value" "GND" (id 1) (at 129.54 148.59 0)
+      (effects (font (size 1.27 1.27)) hide)
+    )
     (property "Footprint" "" (id 2) (at 129.54 143.51 0)
       (effects (font (size 1.27 1.27)) hide)
@@
       (effects (font (size 1.27 1.27)) hide)
     )
-    (property "Value" "GND" (id 1) (at 32.385 81.915 0))
+    (property "Value" "GND" (id 1) (at 32.385 81.915 0)
+      (effects (font (size 1.27 1.27)) hide)
+    )
     (property "Footprint" "" (id 2) (at 32.385 77.47 0)
       (effects (font (size 1.27 1.27)) hide)

Commit message: my body is a machine that takes in peanut m&ms and puts out rocket engine controllers
Parts:
- C1, C2, C3, C4: LCSC (none) -> C92797
- D3, D5: LCSC (none) -> C14996
- LED13, LED14, LED15: LCSC (none) -> C84270
- R1: LCSC (none) -> C294117
- R2: LCSC (none) -> C102381
- R3: LCSC (none) -> C229812
- R4: LCSC (none) -> C132649
- R5: LCSC (none) -> C17887
- U1: LCSC (none) -> C259971
- U2: LCSC (none) -> C259973
Changed lines of the file:
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@@
+      (effects (font (size 1.27 1.27)) hide)
+    )
+    (property "LCSC" "C259971" (id 4) (at 129.54 83.82 0)
       (effects (font (size 1.27 1.27)) hide)
     )
@@
       (effects (font (size 1.27 1.27)) hide)
     )
+    (property "LCSC" "C84270" (id 4) (at 92.71 63.5 0)
+      (effects (font (size 1.27 1.27)) hide)
+    )
     (pin "1")
     (pin "2")
@@
     )
     (property "Datasheet" "~" (id 3) (at 115.57 133.35 0)
+      (effects (font (size 1.27 1.27)) hide)
+    )
+    (property "LCSC" "C92797" (id 4) (at 115.57 133.35 0)
       (effects (font (size 1.27 1.27)) hide)
     )
@@
     )
     (property "Datasheet" "~" (id 3) (at 162.56 88.9 0)
+      (effects (font (size 1.27 1.27)) hide)
+    )
+    (property "LCSC" "C84270" (id 4) (at 162.56 88.9 0)
       (effects (font (size 1.27 1.27)) hide)
     )
@@
     )
     (property "Datasheet" "~" (id 3) (at 119.38 88.9 0)
+      (effects (font (size 1.27 1.27)) hide)
+    )
+    (property "LCSC" "C92797" (id 4) (at 119.38 88.9 0)
       (effects (font (size 1.27 1.27)) hide)
     )
@@
       (effects (font (size 1.27 1.27)) hide)
     )
+    (property "LCSC" "C14996" (id 4) (at 129.54 72.39 0)
+      (effects (font (size 1.27 1.27)) hide)
+    )
     (pin "1")
     (pin "2")
@@
       (effects (font (size 1.27 1.27)) hide)
     )
+    (property "LCSC" "C229812" (id 4) (at 162.56 96.52 0)
+      (effects (font (size 1.27 1.27)) hide)
+    )
     (pin "1")
     (pin "2")
@@
     )
     (property "Datasheet" "~" (id 3) (at 92.71 73.66 0)
+      (effects (font (size 1.27 1.27)) hide)
+    )
+    (property "LCSC" "C294117" (id 4) (at 92.71 73.66 0)
       (effects (font (size 1.27 1.27)) hide)
     )
@@
     )
     (property "Datasheet" "~" (id 3) (at 151.13 133.35 0)
+      (effects (font (size 1.27 1.27)) hide)
+    )
+    (property "LCSC" "C84270" (id 4) (at 151.13 133.35 0)
       (effects (font (size 1.27 1.27)) hide)
     )
@@
       (effects (font (size 1.27 1.27)) hide)
     )
+    (property "LCSC" "C259973" (id 4) (at 129.54 128.27 0)
+      (effects (font (size 1.27 1.27)) hide)
+    )
     (pin "1")
     (pin "2")
@@
     )
     (property "Datasheet" "~" (id 3) (at 129.54 97.79 0)
+      (effects (font (size 1.27 1.27)) hide)
+    )
+    (property "LCSC" "C132649" (id 4) (at 129.54 97.79 0)
       (effects (font (size 1.27 1.27)) hide)
     )
@@
     )
     (property "Datasheet" "~" (id 3) (at 129.54 118.11 0)
+      (effects (font (size 1.27 1.27)) hide)
+    )
+    (property "LCSC" "C14996" (id 4) (at 129.54 118.11 0)
       (effects (font (size 1.27 1.27)) hide)
     )
@@
       (effects (font (size 1.27 1.27)) hide)
     )
+    (property "LCSC" "C102381" (id 4) (at 140.97 88.9 0)
+      (effects (font (size 1.27 1.27)) hide)
+    )
     (pin "1")
     (pin "2")
@@
     )
     (property "Datasheet" "~" (id 3) (at 151.13 140.97 0)
+      (effects (font (size 1.27 1.27)) hide)
+    )
+    (property "LCSC" "C17887" (id 4) (at 151.13 140.97 0)
       (effects (font (size 1.27 1.27)) hide)
     )
@@
       (effects (font (size 1.27 1.27)) hide)
     )
+    (property "LCSC" "C92797" (id 4) (at 151.13 88.9 0)
+      (effects (font (size 1.27 1.27)) hide)
+    )
     (pin "1")
     (pin "2")
@@
       (effects (font (size 1.27 1.27)) hide)
     )
+    (property "LCSC" "C92797" (id 4) (at 140.97 133.35 0)
+      (effects (font (size 1.27 1.27)) hide)
+    )
