File: drivers.kicad_sch (KiCad schematic)
At the start: 55 parts

Commit message: secret arca meetings
Parts:
- added J? (x12): Conn_01x01_Male, symbol Connector:Conn_01x01_Male
Connections:
- net DRV_NEG_1: now also J?.1 (Pin_1)
- net DRV_NEG_2: now also J?.1 (Pin_1)
- net DRV_NEG_3: now also J?.1 (Pin_1)
- net DRV_NEG_4: now also J?.1 (Pin_1)
- net DRV_NEG_5: now also J?.1 (Pin_1)
- net DRV_NEG_6: now also J?.1 (Pin_1)
- net DRV_POS_1: now also J?.1 (Pin_1)
- net DRV_POS_2: now also J?.1 (Pin_1)
- net DRV_POS_3: now also J?.1 (Pin_1)
- net DRV_POS_4: now also J?.1 (Pin_1)
- net DRV_POS_5: now also J?.1 (Pin_1)
- net DRV_POS_6: now also J?.1 (Pin_1)
Changed lines of the file:
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@@
+    (pin "1")
+  )
+  (symbol (lib_id "Connector:Conn_01x01_Male") (at 223.52 49.53 0) (unit 1)
+    (in_bom yes) (on_board yes) (fields_autoplaced)
+    (property "Reference" "J?" (id 0) (at 224.155 46.99 0))
+    (property "Value" "Conn_01x01_Male" (id 1) (at 224.155 46.99 0)
+      (effects (font (size 1.27 1.27)) hide)
+    )
+    (property "Footprint" "" (id 2) (at 223.52 49.53 0)
+      (effects (font (size 1.27 1.27)) hide)
+    )
+    (property "Datasheet" "~" (id 3) (at 223.52 49.53 0)
+      (effects (font (size 1.27 1.27)) hide)
+    )
     (pin "1")
   )
@@
     (pin "1")
   )
+  (symbol (lib_id "Connector:Conn_01x01_Male") (at 40.64 121.92 0) (unit 1)
+    (in_bom yes) (on_board yes) (fields_autoplaced)
+    (property "Reference" "J?" (id 0) (at 41.275 119.38 0))
+    (property "Value" "Conn_01x01_Male" (id 1) (at 41.275 119.38 0)
+      (effects (font (size 1.27 1.27)) hide)
+    )
+    (property "Footprint" "" (id 2) (at 40.64 121.92 0)
+      (effects (font (size 1.27 1.27)) hide)
+    )
+    (property "Datasheet" "~" (id 3) (at 40.64 121.92 0)
+      (effects (font (size 1.27 1.27)) hide)
+    )
+    (pin "1")
+  )
   (symbol (lib_id "power:GND") (at 218.44 142.24 0) (unit 1)
     (in_bom yes) (on_board yes) (fields_autoplaced)
@@
     )
     (property "Datasheet" "" (id 3) (at 218.44 142.24 0)
+      (effects (font (size 1.27 1.27)) hide)
+    )
+    (pin "1")
+  )
+  (symbol (lib_id "Connector:Conn_01x01_Male") (at 223.52 105.41 0) (unit 1)
+    (in_bom yes) (on_board yes) (fields_autoplaced)
+    (property "Reference" "J?" (id 0) (at 224.155 102.87 0))
+    (property "Value" "Conn_01x01_Male" (id 1) (at 224.155 102.87 0)
+      (effects (font (size 1.27 1.27)) hide)
+    )
+    (property "Footprint" "" (id 2) (at 223.52 105.41 0)
+      (effects (font (size 1.27 1.27)) hide)
+    )
+    (property "Datasheet" "~" (id 3) (at 223.52 105.41 0)
       (effects (font (size 1.27 1.27)) hide)
     )
@@
     (pin "1")
   )
+  (symbol (lib_id "Connector:Conn_01x01_Male") (at 135.89 104.14 0) (unit 1)
+    (in_bom yes) (on_board yes) (fields_autoplaced)
+    (property "Reference" "J?" (id 0) (at 136.525 101.6 0))
+    (property "Value" "Conn_01x01_Male" (id 1) (at 136.525 101.6 0)
+      (effects (font (size 1.27 1.27)) hide)
+    )
+    (property "Footprint" "" (id 2) (at 135.89 104.14 0)
+      (effects (font (size 1.27 1.27)) hide)
+    )
+    (property "Datasheet" "~" (id 3) (at 135.89 104.14 0)
+      (effects (font (size 1.27 1.27)) hide)
+    )
+    (pin "1")
+  )
   (symbol (lib_id "power:+12V") (at 48.26 24.13 0) (unit 1)
     (in_bom yes) (on_board yes) (fields_autoplaced)
@@
     (pin "1")
   )
+  (symbol (lib_id "Connector:Conn_01x01_Male") (at 39.37 33.02 0) (unit 1)
+    (in_bom yes) (on_board yes) (fields_autoplaced)
+    (property "Reference" "J?" (id 0) (at 40.005 30.48 0))
+    (property "Value" "Conn_01x01_Male" (id 1) (at 40.005 30.48 0)
+      (effects (font (size 1.27 1.27)) hide)
+    )
+    (property "Footprint" "" (id 2) (at 39.37 33.02 0)
+      (effects (font (size 1.27 1.27)) hide)
+    )
+    (property "Datasheet" "~" (id 3) (at 39.37 33.02 0)
+      (effects (font (size 1.27 1.27)) hide)
+    )
+    (pin "1")
+  )
   (symbol (lib_id "Device:Q_NMOS_GDS") (at 46.99 135.89 0) (unit 1)
     (in_bom yes) (on_board yes) (fields_autoplaced)
@@
     (pin "2")
     (pin "3")
+  )
+  (symbol (lib_id "Connector:Conn_01x01_Male") (at 135.89 49.53 0) (unit 1)
+    (in_bom yes) (on_board yes) (fields_autoplaced)
+    (property "Reference" "J?" (id 0) (at 136.525 46.99 0))
+    (property "Value" "Conn_01x01_Male" (id 1) (at 136.525 46.99 0)
+      (effects (font (size 1.27 1.27)) hide)
+    )
+    (property "Footprint" "" (id 2) (at 135.89 49.53 0)
+      (effects (font (size 1.27 1.27)) hide)
+    )
+    (property "Datasheet" "~" (id 3) (at 135.89 49.53 0)
+      (effects (font (size 1.27 1.27)) hide)
+    )
+    (pin "1")
   )
   (symbol (lib_id "power:+5V") (at 130.81 55.88 0) (unit 1)
@@
     )
     (property "Datasheet" "" (id 3) (at 130.81 55.88 0)
+      (effects (font (size 1.27 1.27)) hide)
+    )
+    (pin "1")
+  )
+  (symbol (lib_id "Connector:Conn_01x01_Male") (at 39.37 48.26 0) (unit 1)
+    (in_bom yes) (on_board yes) (fields_autoplaced)
+    (property "Reference" "J?" (id 0) (at 40.005 45.72 0))
+    (property "Value" "Conn_01x01_Male" (id 1) (at 40.005 45.72 0)
+      (effects (font (size 1.27 1.27)) hide)
+    )
+    (property "Footprint" "" (id 2) (at 39.37 48.26 0)
+      (effects (font (size 1.27 1.27)) hide)
+    )
+    (property "Datasheet" "~" (id 3) (at 39.37 48.26 0)
       (effects (font (size 1.27 1.27)) hide)
     )
@@
     (pin "2")
   )
+  (symbol (lib_id "Connector:Conn_01x01_Male") (at 40.64 106.68 0) (unit 1)
+    (in_bom yes) (on_board yes) (fields_autoplaced)
+    (property "Reference" "J?" (id 0) (at 41.275 104.14 0))
+    (property "Value" "Conn_01x01_Male" (id 1) (at 41.275 104.14 0)
+      (effects (font (size 1.27 1.27)) hide)
+    )
+    (property "Footprint" "" (id 2) (at 40.64 106.68 0)
+      (effects (font (size 1.27 1.27)) hide)
+    )
+    (property "Datasheet" "~" (id 3) (at 40.64 106.68 0)
+      (effects (font (size 1.27 1.27)) hide)
+    )
+    (pin "1")
+  )
   (symbol (lib_id "Device:R_US") (at 218.44 138.43 0) (unit 1)
     (in_bom yes) (on_board yes) (fields_autoplaced)
@@
     (pin "2")
   )
+  (symbol (lib_id "Connector:Conn_01x01_Male") (at 135.89 34.29 0) (unit 1)
+    (in_bom yes) (on_board yes) (fields_autoplaced)
+    (property "Reference" "J?" (id 0) (at 136.525 31.75 0))
+    (property "Value" "Conn_01x01_Male" (id 1) (at 136.525 31.75 0)
+      (effects (font (size 1.27 1.27)) hide)
+    )
+    (property "Footprint" "" (id 2) (at 135.89 34.29 0)
+      (effects (font (size 1.27 1.27)) hide)
+    )
+    (property "Datasheet" "~" (id 3) (at 135.89 34.29 0)
+      (effects (font (size 1.27 1.27)) hide)
+    )
+    (pin "1")
+  )
   (symbol (lib_id "Device:R_US") (at 34.29 66.04 0) (unit 1)
     (in_bom yes) (on_board yes) (fields_autoplaced)
@@
     (pin "1")
     (pin "2")
+  )
+  (symbol (lib_id "Connector:Conn_01x01_Male") (at 223.52 120.65 0) (unit 1)
+    (in_bom yes) (on_board yes) (fields_autoplaced)
+    (property "Reference" "J?" (id 0) (at 224.155 118.11 0))
+    (property "Value" "Conn_01x01_Male" (id 1) (at 224.155 118.11 0)
+      (effects (font (size 1.27 1.27)) hide)
+    )
+    (property "Footprint" "" (id 2) (at 223.52 120.65 0)
+      (effects (font (size 1.27 1.27)) hide)
+    )
+    (property "Datasheet" "~" (id 3) (at 223.52 120.65 0)
+      (effects (font (size 1.27 1.27)) hide)
+    )
+    (pin "1")
   )
   (symbol (lib_id "Device:R_US") (at 35.56 139.7 0) (unit 1)
@@
     (pin "2")
   )
+  (symbol (lib_id "Connector:Conn_01x01_Male") (at 135.89 119.38 0) (unit 1)
+    (in_bom yes) (on_board yes) (fields_autoplaced)
+    (property "Reference" "J?" (id 0) (at 136.525 116.84 0))
+    (property "Value" "Conn_01x01_Male" (id 1) (at 136.525 116.84 0)
+      (effects (font (size 1.27 1.27)) hide)
+    )
+    (property "Footprint" "" (id 2) (at 135.89 119.38 0)
+      (effects (font (size 1.27 1.27)) hide)
+    )
+    (property "Datasheet" "~" (id 3) (at 135.89 119.38 0)
+      (effects (font (size 1.27 1.27)) hide)
+    )
+    (pin "1")
+  )
   (symbol (lib_id "Device:D") (at 66.04 114.3 270) (unit 1)
     (in_bom yes) (on_board yes) (fields_autoplaced)
@@
     (pin "2")
   )
+  (symbol (lib_id "Connector:Conn_01x01_Male") (at 223.52 34.29 0) (unit 1)
+    (in_bom yes) (on_board yes) (fields_autoplaced)
+    (property "Reference" "J?" (id 0) (at 224.155 31.75 0))
+    (property "Value" "Conn_01x01_Male" (id 1) (at 224.155 31.75 0)
+      (effects (font (size 1.27 1.27)) hide)
+    )
+    (property "Footprint" "" (id 2) (at 223.52 34.29 0)
+      (effects (font (size 1.27 1.27)) hide)
+    )
+    (property "Datasheet" "~" (id 3) (at 223.52 34.29 0)
+      (effects (font (size 1.27 1.27)) hide)
+    )
+    (pin "1")
+  )
   (symbol (lib_id "Device:R_US") (at 49.53 118.11 0) (unit 1)

Commit message: first revision of full schematic copied over
Parts:
- removed J? (x12): Conn_01x01_Male, symbol Connector:Conn_01x01_Male
- added J? (x6): Conn_01x02_Male, symbol Connector:Conn_01x02_Male
- D?: value YLW -> DRV_STAT_3
- D?: value YLW -> DRV_STAT_5
- D?: value YLW -> DRV_STAT_2
- D?: value YLW -> DRV_STAT_1
- D?: value BLU -> FS_STAT_5
- D?: value BLU -> FS_STAT_1
- D?: value YLW -> DRV_STAT_4
- D?: value YLW -> DRV_STAT_6
- D?: value BLU -> FS_STAT_2
- D?: value BLU -> FS_STAT_6
- D?: value BLU -> FS_STAT_3
- D?: value BLU -> FS_STAT_4
Connections:
- net DRV_NEG_1: now also J?.2 (Pin_2)
- net DRV_NEG_2: now also J?.2 (Pin_2)
- net DRV_NEG_3: now also J?.2 (Pin_2)
- net DRV_NEG_4: now also J?.2 (Pin_2)
- net DRV_NEG_5: now also J?.2 (Pin_2)
- net DRV_NEG_6: now also J?.2 (Pin_2)
- net DRV_POS_1: now also J?.1 (Pin_1)
- net DRV_POS_2: now also J?.1 (Pin_1)
- net DRV_POS_3: now also J?.1 (Pin_1)
- net DRV_POS_4: now also J?.1 (Pin_1)
- net DRV_POS_5: now also J?.1 (Pin_1)
- net DRV_POS_6: now also J?.1 (Pin_1)
- net drv_nc7: now reaches J?.7 (Pin_7)
- net drv_nc8: now reaches J?.8 (Pin_8)
- no-connect marks 0 -> 2
Other:
- note added: "Note: driver 6 used for ignition"
- company: (none) -> Rice Eclipse
- title: (none) -> Drivers
- moved on the sheet: D?

Commit message: added schematic pdf for review
Parts:
- gave numbers to parts that had none: 61

Commit message: added footprints and started schematic review revisions
Parts:
- removed J10, J11, J12, J13, J7, J8: Conn_01x02_Male, symbol Connector:Conn_01x02_Male
- added J10, J11, J12, J13, J7, J8: Conn_01x02_Female, symbol Connector:Conn_01x02_Female
- D10, D15, D16, D21, D22, D9: value D -> SS54; footprint (none) -> karca_custom_footprints:DO-214AC
- D11, D12, D13, D14, D17, D18, D19, D20, D23, D24, D7, D8: footprint (none) -> LED_SMD:LED_1206_3216Metric
- F1, F2, F3, F4, F5, F6: value Fuse -> 3588-20; footprint (none) -> karca_custom_footprints:3588-20 fuse
- Q1, Q2, Q3, Q4, Q5, Q6: footprint (none) -> Package_TO_SOT_THT:TO-220-3_Horizontal_TabDown
- R10, R11, R12, R13, R14, R15, R16, R17, R18, R19, R20, R21, R22, R23, R24, R25, R26, R27, R28, R29, R6, R7, R8, R9: footprint (none) -> Resistor_SMD:R_1206_3216Metric
Connections:
- net DRV_NEG_1: now also J7.2 (Pin_2)
- net DRV_NEG_2: now also J10.2 (Pin_2)
- net DRV_NEG_3: now also J12.2 (Pin_2)
- net DRV_NEG_4: now also J8.2 (Pin_2)
- net DRV_NEG_5: now also J11.2 (Pin_2)
- net DRV_NEG_6: now also J13.2 (Pin_2)
- net DRV_POS_1: now also J7.1 (Pin_1)
- net DRV_POS_2: now also J10.1 (Pin_1)
- net DRV_POS_3: now also J12.1 (Pin_1)
- net DRV_POS_4: now also J8.1 (Pin_1)
- net DRV_POS_5: now also J11.1 (Pin_1)
- net DRV_POS_6: now also J13.1 (Pin_1)

Commit message: schematic editing + creating some footprints
Parts:
- J10, J11, J12, J13, J7, J8: footprint (none) -> Connector_PinHeader_2.54mm:PinHeader_1x02_P2.54mm_Vertical
- J9: symbol Connector:Conn_01x08_Female -> Connector_Generic:Conn_01x08
- Q1, Q2, Q3, Q4, Q5, Q6: footprint Package_TO_SOT_THT:TO-220-3_Horizontal_TabDown -> Package_TO_SOT_THT:TO-220-3_Vertical

Commit message: updated all footprints, resolved most ERC & setup layout
Parts:
- J9: footprint (none) -> Connector_PinSocket_2.54mm:PinSocket_1x08_P2.54mm_Vertical
Changed lines of the file:
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@@
       (effects (font (size 1.27 1.27)) (justify left))
     )
-    (property "Footprint" "" (id 2) (at 41.91 173.99 0)
+    (property "Footprint" "Connector_PinSocket_2.54mm:PinSocket_1x08_P2.54mm_Vertical" (id 2) (at 41.91 173.99 0)
       (effects (font (size 1.27 1.27)) hide)
     )

Commit message: grouped components on PCB
Parts:
- Q1, Q2, Q3, Q4, Q5, Q6: footprint Package_TO_SOT_THT:TO-220-3_Vertical -> Package_TO_SOT_THT:TO-220-3_Horizontal_TabDown
Changed lines of the file:
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@@
       (effects (font (size 1.27 1.27)) (justify left))
     )
-    (property "Footprint" "Package_TO_SOT_THT:TO-220-3_Vertical" (id 2) (at 52.07 133.35 0)
+    (property "Footprint" "Package_TO_SOT_THT:TO-220-3_Horizontal_TabDown" (id 2) (at 52.07 133.35 0)
       (effects (font (size 1.27 1.27)) hide)
     )
@@
       (effects (font (size 1.27 1.27)) (justify left))
     )
-    (property "Footprint" "Package_TO_SOT_THT:TO-220-3_Vertical" (id 2) (at 50.8 59.69 0)
+    (property "Footprint" "Package_TO_SOT_THT:TO-220-3_Horizontal_TabDown" (id 2) (at 50.8 59.69 0)
       (effects (font (size 1.27 1.27)) hide)
     )
@@
   )
   (symbol (lib_id "Device:R_US") (at 35.56 132.08 0) (unit 1)
-    (in_bom yes) (on_board no) (fields_autoplaced)
+    (in_bom yes) (on_board yes) (fields_autoplaced)
     (property "Reference" "R8" (id 0) (at 38.1 130.8099 0)
       (effects (font (size 1.27 1.27)) (justify left))
@@
   )
   (symbol (lib_id "Device:R_US") (at 34.29 58.42 0) (unit 1)
-    (in_bom yes) (on_board no) (fields_autoplaced)
+    (in_bom yes) (on_board yes) (fields_autoplaced)
     (property "Reference" "R6" (id 0) (at 36.83 57.1499 0)
       (effects (font (size 1.27 1.27)) (justify left))
@@
       (effects (font (size 1.27 1.27)) (justify left))
     )
-    (property "Footprint" "Package_TO_SOT_THT:TO-220-3_Vertical" (id 2) (at 147.32 60.96 0)
+    (property "Footprint" "Package_TO_SOT_THT:TO-220-3_Horizontal_TabDown" (id 2) (at 147.32 60.96 0)
       (effects (font (size 1.27 1.27)) hide)
     )
@@
   )
   (symbol (lib_id "Device:R_US") (at 218.44 130.81 0) (unit 1)
-    (in_bom yes) (on_board no) (fields_autoplaced)
+    (in_bom yes) (on_board yes) (fields_autoplaced)
     (property "Reference" "R24" (id 0) (at 220.98 129.5399 0)
       (effects (font (size 1.27 1.27)) (justify left))
@@
       (effects (font (size 1.27 1.27)) (justify left))
     )
-    (property "Footprint" "Package_TO_SOT_THT:TO-220-3_Vertical" (id 2) (at 147.32 130.81 0)
+    (property "Footprint" "Package_TO_SOT_THT:TO-220-3_Horizontal_TabDown" (id 2) (at 147.32 130.81 0)
       (effects (font (size 1.27 1.27)) hide)
     )
@@
   )
   (symbol (lib_id "Device:R_US") (at 130.81 129.54 0) (unit 1)
-    (in_bom yes) (on_board no) (fields_autoplaced)
+    (in_bom yes) (on_board yes) (fields_autoplaced)
     (property "Reference" "R16" (id 0) (at 133.35 128.2699 0)
       (effects (font (size 1.27 1.27)) (justify left))
@@
       (effects (font (size 1.27 1.27)) (justify left))
     )
-    (property "Footprint" "Package_TO_SOT_THT:TO-220-3_Vertical" (id 2) (at 234.95 132.08 0)
+    (property "Footprint" "Package_TO_SOT_THT:TO-220-3_Horizontal_TabDown" (id 2) (at 234.95 132.08 0)
       (effects (font (size 1.27 1.27)) hide)
     )
@@
       (effects (font (size 1.27 1.27)) (justify left))
     )
-    (property "Footprint" "Package_TO_SOT_THT:TO-220-3_Vertical" (id 2) (at 234.95 60.96 0)
+    (property "Footprint" "Package_TO_SOT_THT:TO-220-3_Horizontal_TabDown" (id 2) (at 234.95 60.96 0)
       (effects (font (size 1.27 1.27)) hide)
     )
@@
   )
   (symbol (lib_id "Device:R_US") (at 218.44 59.69 0) (unit 1)
-    (in_bom yes) (on_board no) (fields_autoplaced)
+    (in_bom yes) (on_board yes) (fields_autoplaced)
     (property "Reference" "R22" (id 0) (at 220.98 58.4199 0)
       (effects (font (size 1.27 1.27)) (justify left))
@@
   )
   (symbol (lib_id "Device:R_US") (at 130.81 59.69 0) (unit 1)
-    (in_bom yes) (on_board no) (fields_autoplaced)
+    (in_bom yes) (on_board yes) (fields_autoplaced)
     (property "Reference" "R14" (id 0) (at 133.35 58.4199 0)
       (effects (font (size 1.27 1.27)) (justify left))

Commit message: preliminary layout and started pwr plane config
Parts:
- removed J10, J11, J12, J13, J7, J8: Conn_01x02_Female, Connector_PinHeader_2.54mm:PinHeader_1x02_P2.54mm_Vertical, symbol Connector:Conn_01x02_Female
- removed J9: Conn_01x08_Female, Connector_PinSocket_2.54mm:PinSocket_1x08_P2.54mm_Vertical, symbol Connector_Generic:Conn_01x08
- added J10, J11, J6, J7, J8, J9: Screw_Terminal_01x02, 1190363:1190363, symbol Connector:Screw_Terminal_01x02
- added J12: Conn_01x08_Female, Connector_PinSocket_2.54mm:PinSocket_1x08_P2.54mm_Vertical, symbol Connector:Conn_01x08_Female
- F1, F4: footprint karca_custom_footprints:3588-20 fuse -> 3588-20:358820
- F2: renamed from F3; footprint karca_custom_footprints:3588-20 fuse -> 3588-20:358820
- F3: renamed from F5; footprint karca_custom_footprints:3588-20 fuse -> 3588-20:358820
- F5: renamed from F6; footprint karca_custom_footprints:3588-20 fuse -> 3588-20:358820
- F6: renamed from F2; footprint karca_custom_footprints:3588-20 fuse -> 3588-20:358820
- renumbered D19 to D10, D17 to D11, D23 to D12, D9 to D13, D16 to D14, D21 to D15, D14 to D16, D18 to D17, D20 to D18, D8 to D19, D24 to D20, D12 to D21, D15 to D22, D22 to D23, D10 to D24, D11 to D8, D13 to D9, Q3 to Q2, Q5 to Q3, Q6 to Q5, Q2 to Q6, R20 to R10, R28 to R11, R6 to R12, R14 to R13, R22 to R14, R7 to R15, R15 to R16, R23 to R17, R19 to R18, R27 to R19, R11 to R20, R29 to R22, R13 to R23, R16 to R24, R24 to R25, R8 to R26, R17 to R27, R25 to R28, R9 to R29, R10 to R6, R18 to R7, R26 to R8, R12 to R9
Connections:
- net DRV_CTL_1: now also J12.1 (Pin_1)
- net DRV_CTL_2: now also J12.2 (Pin_2)
- net DRV_CTL_3: now also J12.3 (Pin_3)
- net DRV_CTL_4: now also J12.4 (Pin_4)
- net DRV_CTL_5: now also J12.5 (Pin_5)
- net DRV_CTL_6: now also J12.6 (Pin_6)
- net DRV_NEG_1: now also J6.2 (Pin_2)
- net DRV_NEG_2: now also J7.2 (Pin_2)
- net DRV_NEG_3: now also J8.2 (Pin_2)
- net DRV_NEG_4: now also J11.2 (Pin_2)
- net DRV_NEG_5: now also J9.2 (Pin_2)
- net DRV_NEG_6: now also J10.2 (Pin_2)
- net DRV_POS_1: now also J6.1 (Pin_1)
- net DRV_POS_2: now also J7.1 (Pin_1)
- net DRV_POS_3: now also J8.1 (Pin_1)
- net DRV_POS_4: now also J11.1 (Pin_1)
- net DRV_POS_5: now also J9.1 (Pin_1)
- net DRV_POS_6: now also J10.1 (Pin_1)
- net drv_nc7: now also J12.7 (Pin_7)
- net drv_nc8: now also J12.8 (Pin_8)
