File: drivers.kicad_sch (KiCad schematic)
At the start: 61 parts, among them J12 Conn_01x06_Female, Q1 FQP30N06, Q2 FQP30N06, Q3 FQP30N06, Q4 FQP30N06, Q5 FQP30N06, Q6 FQP30N06

Commit message: enshrinkening of the board
Parts:
- CON_IGN1: renamed from CON_DRV6; footprint 1190363:1190363 -> 1190365:1190365; symbol Connector:Screw_Terminal_01x02 -> Connector:Screw_Terminal_01x04
Connections:
- net +12V: now also CON_IGN1.1 (Pin_1)
- net DRV_NEG_6: now also CON_IGN1.3 (Pin_3); no longer CON_IGN1.2 (Pin_2)
- net DRV_POS_6: now also CON_IGN1.2 (Pin_2); no longer CON_IGN1.1 (Pin_1)
- net GND: now also CON_IGN1.4 (Pin_4)
Changed lines of the file:
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@@
+    (stroke (width 0) (type default) (color 0 0 0 0))
+  )
+  (wire (pts (xy 224.79 99.695) (xy 224.79 102.87))
     (stroke (width 0) (type default) (color 0 0 0 0))
   )
@@
   )
   (wire (pts (xy 218.44 63.5) (xy 224.79 63.5))
+    (stroke (width 0) (type default) (color 0 0 0 0))
+  )
+  (wire (pts (xy 224.79 110.49) (xy 224.79 113.665))
     (stroke (width 0) (type default) (color 0 0 0 0))
   )
@@
     (pin "1")
   )
-  (symbol (lib_name "+12V_1") (lib_id "power:+12V") (at 34.29 54.61 0) (unit 1)
+  (symbol (lib_id "power:+12V") (at 34.29 54.61 0) (unit 1)
     (in_bom yes) (on_board yes) (fields_autoplaced)
     (property "Reference" "#PWR0170" (id 0) (at 34.29 58.42 0)
@@
     (pin "1")
   )
-  (symbol (lib_id "Connector:Screw_Terminal_01x02") (at 219.71 105.41 0) (mirror y) (unit 1)
+  (symbol (lib_id "Connector:Screw_Terminal_01x04") (at 219.71 105.41 0) (mirror y) (unit 1)
     (in_bom yes) (on_board yes)
-    (property "Reference" "CON_DRV6" (id 0) (at 217.17 106.6799 0)
-      (effects (font (size 1.27 1.27)) (justify left))
-    )
-    (property "Value" "Screw_Terminal_01x02" (id 1) (at 217.17 107.9499 0)
+    (property "Reference" "CON_IGN1" (id 0) (at 217.17 106.6799 0)
+      (effects (font (size 1.27 1.27)) (justify left))
+    )
+    (property "Value" "Screw_Terminal_01x02" (id 1) (at 217.17 108.5849 0)
       (effects (font (size 1.27 1.27)) (justify left) hide)
     )
-    (property "Footprint" "1190363:1190363" (id 2) (at 219.71 105.41 0)
+    (property "Footprint" "1190365:1190365" (id 2) (at 219.71 105.41 0)
       (effects (font (size 1.27 1.27)) hide)
     )
@@
     (pin "1")
     (pin "2")
+    (pin "3")
+    (pin "4")
   )
   (symbol (lib_id "Connector:Screw_Terminal_01x02") (at 132.08 34.29 0) (mirror y) (unit 1)
@@
     (pin "1")
   )
-  (symbol (lib_name "+12V_1") (lib_id "power:+12V") (at 130.81 125.73 0) (unit 1)
+  (symbol (lib_id "power:+12V") (at 130.81 125.73 0) (unit 1)
     (in_bom yes) (on_board yes) (fields_autoplaced)
     (property "Reference" "#PWR0168" (id 0) (at 130.81 129.54 0)
@@
     (pin "2")
   )
+  (symbol (lib_id "power:GND") (at 224.79 113.665 0) (unit 1)
+    (in_bom yes) (on_board yes) (fields_autoplaced)
+    (property "Reference" "#PWR0105" (id 0) (at 224.79 120.015 0)
+      (effects (font (size 1.27 1.27)) hide)
+    )
+    (property "Value" "GND" (id 1) (at 224.79 118.745 0))
+    (property "Footprint" "" (id 2) (at 224.79 113.665 0)
+      (effects (font (size 1.27 1.27)) hide)
+    )
+    (property "Datasheet" "" (id 3) (at 224.79 113.665 0)
+      (effects (font (size 1.27 1.27)) hide)
+    )
+    (pin "1")
+  )
   (symbol (lib_id "Device:D") (at 251.46 41.91 270) (unit 1)
     (in_bom yes) (on_board yes) (fields_autoplaced)
@@
     (pin "2")
   )
-  (symbol (lib_name "+12V_1") (lib_id "power:+12V") (at 35.56 128.27 0) (unit 1)
+  (symbol (lib_id "power:+12V") (at 35.56 128.27 0) (unit 1)
     (in_bom yes) (on_board yes) (fields_autoplaced)
     (property "Reference" "#PWR0172" (id 0) (at 35.56 132.08 0)
@@
     (pin "2")
   )
-  (symbol (lib_name "+12V_1") (lib_id "power:+12V") (at 218.44 127 0) (unit 1)
+  (symbol (lib_id "power:+12V") (at 218.44 127 0) (unit 1)
     (in_bom yes) (on_board yes) (fields_autoplaced)
     (property "Reference" "#PWR0169" (id 0) (at 218.44 130.81 0)
@@
     (pin "2")
   )
-  (symbol (lib_name "+12V_1") (lib_id "power:+12V") (at 218.44 55.88 0) (unit 1)
+  (symbol (lib_id "power:+12V") (at 218.44 55.88 0) (unit 1)
     (in_bom yes) (on_board yes) (fields_autoplaced)
     (property "Reference" "#PWR0171" (id 0) (at 218.44 59.69 0)
@@
     (pin "1")
     (pin "2")
+  )
+  (symbol (lib_id "power:+12V") (at 224.79 99.695 0) (unit 1)
+    (in_bom yes) (on_board yes) (fields_autoplaced)
+    (property "Reference" "#PWR0106" (id 0) (at 224.79 103.505 0)
+      (effects (font (size 1.27 1.27)) hide)
+    )
+    (property "Value" "+12V" (id 1) (at 224.79 94.615 0))
+    (property "Footprint" "" (id 2) (at 224.79 99.695 0)
+      (effects (font (size 1.27 1.27)) hide)
+    )
+    (property "Datasheet" "" (id 3) (at 224.79 99.695 0)
+      (effects (font (size 1.27 1.27)) hide)
+    )
+    (pin "1")
   )
   (symbol (lib_id "Connector:Conn_01x06_Female") (at 88.9 168.91 0) (unit 1)
@@
     (pin "2")
   )
-  (symbol (lib_name "+12V_1") (lib_id "power:+12V") (at 130.81 55.88 0) (unit 1)
+  (symbol (lib_id "power:+12V") (at 130.81 55.88 0) (unit 1)
     (in_bom yes) (on_board yes) (fields_autoplaced)
     (property "Reference" "#PWR0173" (id 0) (at 130.81 59.69 0)

Commit message: done schematiccing after design review
Parts:
- removed CON_DRV1, CON_DRV2, CON_DRV3, CON_DRV4, CON_DRV5: Screw_Terminal_01x02, 1190363:1190363, symbol Connector:Screw_Terminal_01x02
- removed CON_IGN1: Screw_Terminal_01x02, 1190365:1190365, symbol Connector:Screw_Terminal_01x04
- removed D14, D15, D22, D23, D24: DO-214AC, karca_custom_footprints:DO-214AC, symbol Device:D
- removed J12: Conn_01x06_Female, Connector_PinSocket_2.54mm:PinSocket_1x06_P2.54mm_Vertical, symbol Connector:Conn_01x06_Female
- added D2, D4, D6, D7, D8: CDBA340-HF, Diode_SMD:D_SMA, symbol Device:D_Schottky
- added J1: Screw_Terminal_01x10, symbol Connector:Screw_Terminal_01x10
- added J2: Screw_Terminal_01x04, symbol Connector:Screw_Terminal_01x04
- added TP10, TP11, TP6, TP7, TP8, TP9: TestPoint, symbol Connector:TestPoint
- D13: value DO-214AC -> CDBA340-HF; footprint karca_custom_footprints:DO-214AC -> Diode_SMD:D_SMA; symbol Device:D -> Device:D_Schottky
- R10, R22, R7: value 510 -> DNP
- R11, R23, R8: value 510 -> 10k
- R14, R25: value DNP -> 10k
- R16, R17, R27, R28, R29: value 10k -> 510
- R26: value DNP -> 510
Connections:
- net +12V: now also R10.1, R22.1, R7.1, J2.1 (Pin_1); no longer R14.1, R25.1, R26.1
- net DRV_CTL_1: now also TP6.1
- net DRV_CTL_2: now also R7.2, R8.1, TP7.1; no longer R13.2, R16.1
- net DRV_CTL_3: now also R10.2, R11.1, TP8.1; no longer R14.2, R17.1
- net DRV_CTL_4: now also R13.2, R14.1, TP9.1; no longer R26.2, R29.1
- net DRV_CTL_5: now also R22.2, R23.1, TP10.1; no longer R24.2, R27.1
- net DRV_CTL_6: now also R24.2, R25.1, TP11.1; no longer R25.2, R28.1
- net GND: now also R14.2, R18.2, R25.2, R26.2, R8.2, J2.4 (Pin_4); no longer R10.2, R21.2, R22.2, R28.2, R29.2
- net at DRV_STAT_3.1 (K): now also R20.1; no longer R8.1
- net at FS_STAT_3.1 (K): now also R17.1; no longer R11.1
- net at R18.1: now also FS_STAT_4.1 (K); no longer DRV_STAT_5.1 (K)
- net at DRV_STAT_2.1 (K): now also R19.1; no longer R7.1
- net at FS_STAT_5.1 (K): now also R26.1; no longer R21.1
- net at DRV_STAT_6.1 (K): now also R29.1; no longer R19.1
- net at FS_STAT_6.1 (K): now also R27.1; no longer R22.1
- net at FS_STAT_2.1 (K): now also R16.1; no longer R10.1
- net at DRV_STAT_4.1 (K): now also R21.1; no longer R20.1
- net DRV_NEG_1 renamed DRV1_NEG
- net DRV1_NEG: now also J1.2 (Pin_2)
- net DRV_NEG_2 renamed DRV2_NEG
- net DRV2_NEG: now also R19.2, D2.2 (A), J1.4 (Pin_4); no longer R7.2
- net DRV_NEG_3 renamed DRV3_NEG
- net DRV3_NEG: now also R20.2, D4.2 (A), J1.6 (Pin_6); no longer R8.2
- net DRV_NEG_4 renamed DRV4_NEG
- net DRV4_NEG: now also R21.2, D6.2 (A), J1.8 (Pin_8); no longer R20.2
- net DRV_NEG_5 renamed DRV5_NEG
- net DRV5_NEG: now also R28.2, D7.2 (A), J1.10 (Pin_10); no longer R18.2
- net DRV_NEG_6 renamed DRV6_NEG
- net DRV6_NEG: now also R29.2, D8.2 (A), J2.3 (Pin_3); no longer R19.2
- net DRV_POS_1 renamed DRV1_POS
- net DRV1_POS: now also J1.1 (Pin_1)
- net DRV_POS_2 renamed DRV2_POS
- net DRV2_POS: now also D2.1 (K), J1.3 (Pin_3)
- net DRV_POS_3 renamed DRV3_POS
- net DRV3_POS: now also D4.1 (K), J1.5 (Pin_5)
- net DRV_POS_4 renamed DRV4_POS
- net DRV4_POS: now also D6.1 (K), J1.7 (Pin_7)
- net DRV_POS_5 renamed DRV5_POS
- net DRV5_POS: now also D7.1 (K), J1.9 (Pin_9)
- net DRV_POS_6 renamed DRV6_POS
- net DRV6_POS: now also D8.1 (K), J2.2 (Pin_2)
- new net: DRV_STAT_5.1 (K), R28.1
Other:
- note added: "Driver 6 is for ignition and has extra connectors for powering the ignition relay."
- note removed: "Driver 1"
- note removed: "Driver 2"
- note removed: "Driver 3"
- note removed: "Driver 4"
- note removed: "Driver 5"
- note removed: "Driver 6"
- note removed: "Note: driver 6 used for ignition"
- moved on the sheet: D13, DRV_STAT_1, F1, FS_STAT_1, Q1, R12, R15, R6, R9

Commit message: cleaned up PT footprint
Parts:
- J2: footprint (none) -> 1190365:1190365
- TP10, TP11, TP6, TP7, TP8, TP9: footprint (none) -> TestPoint:TestPoint_Pad_D2.0mm
Changed lines of the file:
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@@
       (effects (font (size 1.27 1.27)) (justify left) hide)
     )
-    (property "Footprint" "" (id 2) (at 52.07 179.07 0)
+    (property "Footprint" "TestPoint:TestPoint_Pad_D2.0mm" (id 2) (at 52.07 179.07 0)
       (effects (font (size 1.27 1.27)) hide)
     )
@@
       (effects (font (size 1.27 1.27)) (justify left) hide)
     )
-    (property "Footprint" "" (id 2) (at 147.32 97.155 0)
+    (property "Footprint" "TestPoint:TestPoint_Pad_D2.0mm" (id 2) (at 147.32 97.155 0)
       (effects (font (size 1.27 1.27)) hide)
     )
@@
       (effects (font (size 1.27 1.27)) (justify left) hide)
     )
-    (property "Footprint" "" (id 2) (at 52.07 135.255 0)
+    (property "Footprint" "TestPoint:TestPoint_Pad_D2.0mm" (id 2) (at 52.07 135.255 0)
       (effects (font (size 1.27 1.27)) hide)
     )
@@
       (effects (font (size 1.27 1.27)) (justify left) hide)
     )
-    (property "Footprint" "" (id 2) (at 147.32 145.415 0)
+    (property "Footprint" "TestPoint:TestPoint_Pad_D2.0mm" (id 2) (at 147.32 145.415 0)
       (effects (font (size 1.27 1.27)) hide)
     )
@@
       (effects (font (size 1.27 1.27)) (justify left) hide)
     )
-    (property "Footprint" "" (id 2) (at 52.07 90.805 0)
+    (property "Footprint" "TestPoint:TestPoint_Pad_D2.0mm" (id 2) (at 52.07 90.805 0)
       (effects (font (size 1.27 1.27)) hide)
     )
@@
       (effects (font (size 1.27 1.27)) (justify left) hide)
     )
-    (property "Footprint" "" (id 2) (at 52.07 46.99 0)
+    (property "Footprint" "TestPoint:TestPoint_Pad_D2.0mm" (id 2) (at 52.07 46.99 0)
       (effects (font (size 1.27 1.27)) hide)
     )
@@
       (effects (font (size 1.27 1.27)) (justify left))
     )
-    (property "Footprint" "" (id 2) (at 222.885 125.095 0)
-      (effects (font (size 1.27 1.27)) hide)
-    )
+    (property "Footprint" "1190365:1190365" (id 2) (at 222.885 125.095 0)
+      (effects (font (size 1.27 1.27)) hide)
+    )

Commit message: waiting on mouser for footprints
Parts:
- renumbered FS_STAT_1 to LED1, DRV_STAT_5 to LED10, FS_STAT_6 to LED11, DRV_STAT_6 to LED12, DRV_STAT_1 to LED2, FS_STAT_2 to LED3, DRV_STAT_2 to LED4, FS_STAT_3 to LED5, DRV_STAT_3 to LED6, FS_STAT_4 to LED7, DRV_STAT_4 to LED8, FS_STAT_5 to LED9
Changed lines of the file:
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@@
   (symbol (lib_id "Device:LED") (at 74.93 30.48 90) (unit 1)
     (in_bom yes) (on_board yes) (fields_autoplaced)
-    (property "Reference" "DRV_STAT_1" (id 0) (at 78.74 30.7974 90)
+    (property "Reference" "LED2" (id 0) (at 78.74 30.7974 90)
       (effects (font (size 1.27 1.27)) (justify right))
     )
@@
   (symbol (lib_id "Device:LED") (at 74.93 74.295 90) (unit 1)
     (in_bom yes) (on_board yes) (fields_autoplaced)
-    (property "Reference" "DRV_STAT_2" (id 0) (at 78.74 74.6124 90)
+    (property "Reference" "LED4" (id 0) (at 78.74 74.6124 90)
       (effects (font (size 1.27 1.27)) (justify right))
     )
@@
   (symbol (lib_id "Device:LED") (at 68.58 162.56 90) (unit 1)
     (in_bom yes) (on_board yes)
-    (property "Reference" "FS_STAT_4" (id 0) (at 66.675 162.2424 90)
+    (property "Reference" "LED7" (id 0) (at 66.675 162.2424 90)
       (effects (font (size 1.27 1.27)) (justify left))
     )
@@
   (symbol (lib_id "Device:LED") (at 165.1 128.905 90) (unit 1)
     (in_bom yes) (on_board yes)
-    (property "Reference" "FS_STAT_6" (id 0) (at 163.195 128.5874 90)
+    (property "Reference" "LED11" (id 0) (at 163.195 128.5874 90)
       (effects (font (size 1.27 1.27)) (justify left))
     )
@@
   (symbol (lib_id "Device:LED") (at 171.45 128.905 90) (unit 1)
     (in_bom yes) (on_board yes) (fields_autoplaced)
-    (property "Reference" "DRV_STAT_6" (id 0) (at 175.26 129.2224 90)
+    (property "Reference" "LED12" (id 0) (at 175.26 129.2224 90)
       (effects (font (size 1.27 1.27)) (justify right))
     )
@@
   (symbol (lib_id "Device:LED") (at 74.93 118.745 90) (unit 1)
     (in_bom yes) (on_board yes) (fields_autoplaced)
-    (property "Reference" "DRV_STAT_3" (id 0) (at 78.74 119.0624 90)
+    (property "Reference" "LED6" (id 0) (at 78.74 119.0624 90)
       (effects (font (size 1.27 1.27)) (justify right))
     )
@@
   (symbol (lib_id "Device:LED") (at 68.58 30.48 90) (unit 1)
     (in_bom yes) (on_board yes)
-    (property "Reference" "FS_STAT_1" (id 0) (at 66.675 30.1624 90)
+    (property "Reference" "LED1" (id 0) (at 66.675 30.1624 90)
       (effects (font (size 1.27 1.27)) (justify left))
     )
@@
   (symbol (lib_id "Device:LED") (at 74.93 162.56 90) (unit 1)
     (in_bom yes) (on_board yes) (fields_autoplaced)
-    (property "Reference" "DRV_STAT_4" (id 0) (at 78.74 162.8774 90)
+    (property "Reference" "LED8" (id 0) (at 78.74 162.8774 90)
       (effects (font (size 1.27 1.27)) (justify right))
     )
@@
   (symbol (lib_id "Device:LED") (at 68.58 118.745 90) (unit 1)
     (in_bom yes) (on_board yes)
-    (property "Reference" "FS_STAT_3" (id 0) (at 66.675 118.4274 90)
+    (property "Reference" "LED5" (id 0) (at 66.675 118.4274 90)
       (effects (font (size 1.27 1.27)) (justify left))
     )
@@
   (symbol (lib_id "Device:LED") (at 165.1 80.645 90) (unit 1)
     (in_bom yes) (on_board yes)
-    (property "Reference" "FS_STAT_5" (id 0) (at 163.195 80.3274 90)
+    (property "Reference" "LED9" (id 0) (at 163.195 80.3274 90)
       (effects (font (size 1.27 1.27)) (justify left))
     )
@@
   (symbol (lib_id "Device:LED") (at 171.45 80.645 90) (unit 1)
     (in_bom yes) (on_board yes) (fields_autoplaced)
-    (property "Reference" "DRV_STAT_5" (id 0) (at 175.26 80.9624 90)
+    (property "Reference" "LED10" (id 0) (at 175.26 80.9624 90)
       (effects (font (size 1.27 1.27)) (justify right))
     )
@@
   (symbol (lib_id "Device:LED") (at 68.58 74.295 90) (unit 1)
     (in_bom yes) (on_board yes)
-    (property "Reference" "FS_STAT_2" (id 0) (at 66.675 73.9774 90)
-      (effects (font (size 1.27 1.27)) (justify left))
-    )
+    (property "Reference" "LED3" (id 0) (at 66.675 73.9774 90)
+      (effects (font (size 1.27 1.27)) (justify left))
+    )
