File: drivers.kicad_sch (KiCad schematic)
At the start: 62 parts, among them J1 Screw_Terminal_01x10, J2 Screw_Terminal_01x04, Q1 FQP30N06, Q2 FQP30N06, Q3 FQP30N06, Q4 FQP30N06, Q5 FQP30N06, Q6 FQP30N06

Commit message: ready for fab
Parts:
- J1: footprint (none) -> 1190372:1190372
Changed lines of the file:
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@@
       (effects (font (size 1.27 1.27)) (justify left))
     )
-    (property "Footprint" "" (id 2) (at 217.805 36.83 0)
+    (property "Footprint" "1190372:1190372" (id 2) (at 217.805 36.83 0)
       (effects (font (size 1.27 1.27)) hide)
     )

Commit message: final rev for jlc
Parts:
- LED1, LED11, LED3, LED5, LED7, LED9: value BLU -> GRN
- R16, R17, R18, R19, R20, R21, R26, R27, R28, R29, R6, R9: value 510 -> 910
Changed lines of the file:
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@@
       (effects (font (size 1.27 1.27)) (justify left))
     )
-    (property "Value" "510" (id 1) (at 77.47 83.1849 0)
+    (property "Value" "910" (id 1) (at 77.47 83.1849 0)
       (effects (font (size 1.27 1.27)) (justify left))
     )
@@
       (effects (font (size 1.27 1.27)) (justify right))
     )
-    (property "Value" "510" (id 1) (at 67.31 127.6349 0)
+    (property "Value" "910" (id 1) (at 67.31 127.6349 0)
       (effects (font (size 1.27 1.27)) (justify right))
     )
@@
       (effects (font (size 1.27 1.27)) (justify left))
     )
-    (property "Value" "510" (id 1) (at 77.47 127.6349 0)
+    (property "Value" "910" (id 1) (at 77.47 127.6349 0)
       (effects (font (size 1.27 1.27)) (justify left))
     )
@@
       (effects (font (size 1.27 1.27)) (justify left))
     )
-    (property "Value" "BLU" (id 1) (at 66.675 164.7824 90)
+    (property "Value" "GRN" (id 1) (at 66.675 164.7824 90)
       (effects (font (size 1.27 1.27)) (justify left))
     )
@@
       (effects (font (size 1.27 1.27)) (justify left))
     )
-    (property "Value" "BLU" (id 1) (at 163.195 131.1274 90)
+    (property "Value" "GRN" (id 1) (at 163.195 131.1274 90)
       (effects (font (size 1.27 1.27)) (justify left))
     )
@@
       (effects (font (size 1.27 1.27)) (justify right))
     )
-    (property "Value" "510" (id 1) (at 163.83 89.5349 0)
+    (property "Value" "910" (id 1) (at 163.83 89.5349 0)
       (effects (font (size 1.27 1.27)) (justify right))
     )
@@
       (effects (font (size 1.27 1.27)) (justify left))
     )
-    (property "Value" "510" (id 1) (at 77.47 171.4499 0)
+    (property "Value" "910" (id 1) (at 77.47 171.4499 0)
       (effects (font (size 1.27 1.27)) (justify left))
     )
@@
       (effects (font (size 1.27 1.27)) (justify right))
     )
-    (property "Value" "510" (id 1) (at 67.31 171.4499 0)
+    (property "Value" "910" (id 1) (at 67.31 171.4499 0)
       (effects (font (size 1.27 1.27)) (justify right))
     )
@@
       (effects (font (size 1.27 1.27)) (justify right))
     )
-    (property "Value" "510" (id 1) (at 67.31 39.3699 0)
+    (property "Value" "910" (id 1) (at 67.31 39.3699 0)
       (effects (font (size 1.27 1.27)) (justify right))
     )
@@
       (effects (font (size 1.27 1.27)) (justify left))
     )
-    (property "Value" "BLU" (id 1) (at 66.675 32.7024 90)
+    (property "Value" "GRN" (id 1) (at 66.675 32.7024 90)
       (effects (font (size 1.27 1.27)) (justify left))
     )
@@
       (effects (font (size 1.27 1.27)) (justify left))
     )
-    (property "Value" "510" (id 1) (at 173.99 137.7949 0)
+    (property "Value" "910" (id 1) (at 173.99 137.7949 0)
       (effects (font (size 1.27 1.27)) (justify left))
     )
@@
       (effects (font (size 1.27 1.27)) (justify left))
     )
-    (property "Value" "BLU" (id 1) (at 66.675 120.9674 90)
+    (property "Value" "GRN" (id 1) (at 66.675 120.9674 90)
       (effects (font (size 1.27 1.27)) (justify left))
     )
@@
       (effects (font (size 1.27 1.27)) (justify left))
     )
-    (property "Value" "510" (id 1) (at 173.99 89.5349 0)
+    (property "Value" "910" (id 1) (at 173.99 89.5349 0)
       (effects (font (size 1.27 1.27)) (justify left))
     )
@@
       (effects (font (size 1.27 1.27)) (justify left))
     )
-    (property "Value" "BLU" (id 1) (at 163.195 82.8674 90)
+    (property "Value" "GRN" (id 1) (at 163.195 82.8674 90)
       (effects (font (size 1.27 1.27)) (justify left))
     )
@@
       (effects (font (size 1.27 1.27)) (justify right))
     )
-    (property "Value" "510" (id 1) (at 67.31 83.1849 0)
+    (property "Value" "910" (id 1) (at 67.31 83.1849 0)
       (effects (font (size 1.27 1.27)) (justify right))
     )
@@
       (effects (font (size 1.27 1.27)) (justify right))
     )
-    (property "Value" "510" (id 1) (at 163.83 137.7949 0)
+    (property "Value" "910" (id 1) (at 163.83 137.7949 0)
       (effects (font (size 1.27 1.27)) (justify right))
     )
@@
       (effects (font (size 1.27 1.27)) (justify left))
     )
-    (property "Value" "BLU" (id 1) (at 66.675 76.5174 90)
+    (property "Value" "GRN" (id 1) (at 66.675 76.5174 90)
       (effects (font (size 1.27 1.27)) (justify left))
     )
@@
       (effects (font (size 1.27 1.27)) (justify left))
     )
-    (property "Value" "510" (id 1) (at 77.47 39.3699 0)
-      (effects (font (size 1.27 1.27)) (justify left))
-    )
+    (property "Value" "910" (id 1) (at 77.47 39.3699 0)
+      (effects (font (size 1.27 1.27)) (justify left))
+    )

Commit message: my body is a machine that takes in peanut m&ms and puts out rocket engine controllers
Parts:
- D13, D2, D4, D6, D7, D8: LCSC (none) -> C14996
- LED1, LED11, LED3, LED5, LED7, LED9: LCSC (none) -> C499462
- LED10, LED12, LED2, LED4, LED6, LED8: LCSC (none) -> C434441
- R11, R14, R15, R23, R25, R8: LCSC (none) -> C132649
- R16, R17, R18, R19, R20, R21, R26, R27, R28, R29, R6, R9: LCSC (none) -> C429066
Changed lines of the file:
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@@
+      (effects (font (size 1.27 1.27)) hide)
+    )
+    (property "LCSC" "C132649" (id 4) (at 154.94 149.225 0)
       (effects (font (size 1.27 1.27)) hide)
     )
@@
       (effects (font (size 1.27 1.27)) hide)
     )
+    (property "LCSC" "C14996" (id 4) (at 92.71 76.835 0)
+      (effects (font (size 1.27 1.27)) hide)
+    )
     (pin "1")
     (pin "2")
@@
       (effects (font (size 1.27 1.27)) hide)
     )
+    (property "LCSC" "C14996" (id 4) (at 189.23 131.445 0)
+      (effects (font (size 1.27 1.27)) hide)
+    )
     (pin "1")
     (pin "2")
@@
       (effects (font (size 1.27 1.27)) hide)
     )
+    (property "LCSC" "C429066" (id 4) (at 74.93 81.915 0)
+      (effects (font (size 1.27 1.27)) hide)
+    )
     (pin "1")
     (pin "2")
@@
       (effects (font (size 1.27 1.27)) hide)
     )
+    (property "LCSC" "C429066" (id 4) (at 68.58 126.365 0)
+      (effects (font (size 1.27 1.27)) hide)
+    )
     (pin "1")
     (pin "2")
@@
       (effects (font (size 1.27 1.27)) hide)
     )
+    (property "LCSC" "C429066" (id 4) (at 74.93 126.365 0)
+      (effects (font (size 1.27 1.27)) hide)
+    )
     (pin "1")
     (pin "2")
@@
       (effects (font (size 1.27 1.27)) hide)
     )
+    (property "LCSC" "C132649" (id 4) (at 58.42 94.615 0)
+      (effects (font (size 1.27 1.27)) hide)
+    )
     (pin "1")
     (pin "2")
@@
       (effects (font (size 1.27 1.27)) hide)
     )
+    (property "LCSC" "C434441" (id 4) (at 74.93 30.48 0)
+      (effects (font (size 1.27 1.27)) hide)
+    )
     (pin "1")
     (pin "2")
@@
     )
     (property "Datasheet" "~" (id 3) (at 154.94 100.965 0)
+      (effects (font (size 1.27 1.27)) hide)
+    )
+    (property "LCSC" "C132649" (id 4) (at 154.94 100.965 0)
       (effects (font (size 1.27 1.27)) hide)
     )
@@
       (effects (font (size 1.27 1.27)) hide)
     )
+    (property "LCSC" "C434441" (id 4) (at 74.93 74.295 0)
+      (effects (font (size 1.27 1.27)) hide)
+    )
     (pin "1")
     (pin "2")
@@
       (effects (font (size 1.27 1.27)) hide)
     )
+    (property "LCSC" "C14996" (id 4) (at 189.23 83.185 0)
+      (effects (font (size 1.27 1.27)) hide)
+    )
     (pin "1")
     (pin "2")
@@
       (effects (font (size 1.27 1.27)) hide)
     )
+    (property "LCSC" "C499462" (id 4) (at 68.58 162.56 0)
+      (effects (font (size 1.27 1.27)) hide)
+    )
     (pin "1")
     (pin "2")
@@
       (effects (font (size 1.27 1.27)) hide)
     )
+    (property "LCSC" "C499462" (id 4) (at 165.1 128.905 0)
+      (effects (font (size 1.27 1.27)) hide)
+    )
     (pin "1")
     (pin "2")
@@
       (effects (font (size 1.27 1.27)) hide)
     )
+    (property "LCSC" "C429066" (id 4) (at 165.1 88.265 0)
+      (effects (font (size 1.27 1.27)) hide)
+    )
     (pin "1")
     (pin "2")
@@
     )
     (property "Datasheet" "~" (id 3) (at 58.42 182.88 0)
+      (effects (font (size 1.27 1.27)) hide)
+    )
+    (property "LCSC" "C132649" (id 4) (at 58.42 182.88 0)
       (effects (font (size 1.27 1.27)) hide)
     )
@@
       (effects (font (size 1.27 1.27)) hide)
     )
+    (property "LCSC" "C14996" (id 4) (at 92.71 121.285 0)
+      (effects (font (size 1.27 1.27)) hide)
+    )
     (pin "1")
     (pin "2")
@@
       (effects (font (size 1.27 1.27)) hide)
     )
+    (property "LCSC" "C429066" (id 4) (at 74.93 170.18 0)
+      (effects (font (size 1.27 1.27)) hide)
+    )
     (pin "1")
     (pin "2")
@@
     )
     (property "Datasheet" "~" (id 3) (at 68.58 170.18 0)
+      (effects (font (size 1.27 1.27)) hide)
+    )
+    (property "LCSC" "C429066" (id 4) (at 68.58 170.18 0)
       (effects (font (size 1.27 1.27)) hide)
     )
@@
       (effects (font (size 1.27 1.27)) hide)
     )
+    (property "LCSC" "C434441" (id 4) (at 171.45 128.905 0)
+      (effects (font (size 1.27 1.27)) hide)
+    )
     (pin "1")
     (pin "2")
@@
     )
     (property "Datasheet" "~" (id 3) (at 58.42 139.065 0)
+      (effects (font (size 1.27 1.27)) hide)
+    )
+    (property "LCSC" "C132649" (id 4) (at 58.42 139.065 0)
       (effects (font (size 1.27 1.27)) hide)
     )
@@
       (effects (font (size 1.27 1.27)) hide)
     )
+    (property "LCSC" "C434441" (id 4) (at 74.93 118.745 0)
+      (effects (font (size 1.27 1.27)) hide)
+    )
     (pin "1")
     (pin "2")
@@
       (effects (font (size 1.27 1.27)) hide)
     )
+    (property "LCSC" "C429066" (id 4) (at 68.58 38.1 0)
+      (effects (font (size 1.27 1.27)) hide)
+    )
     (pin "1")
     (pin "2")
@@
       (effects (font (size 1.27 1.27)) hide)
     )
+    (property "LCSC" "C499462" (id 4) (at 68.58 30.48 0)
+      (effects (font (size 1.27 1.27)) hide)
+    )
     (pin "1")
     (pin "2")
@@
       (effects (font (size 1.27 1.27)) hide)
     )
+    (property "LCSC" "C429066" (id 4) (at 171.45 136.525 0)
+      (effects (font (size 1.27 1.27)) hide)
+    )
     (pin "1")
     (pin "2")
@@
       (effects (font (size 1.27 1.27)) hide)
     )
+    (property "LCSC" "C434441" (id 4) (at 74.93 162.56 0)
+      (effects (font (size 1.27 1.27)) hide)
+    )
     (pin "1")
     (pin "2")
@@
       (effects (font (size 1.27 1.27)) hide)
     )
+    (property "LCSC" "C132649" (id 4) (at 58.42 50.8 0)
+      (effects (font (size 1.27 1.27)) hide)
+    )
     (pin "1")
     (pin "2")
@@
     )
     (property "Datasheet" "~" (id 3) (at 68.58 118.745 0)
+      (effects (font (size 1.27 1.27)) hide)
+    )
+    (property "LCSC" "C499462" (id 4) (at 68.58 118.745 0)
       (effects (font (size 1.27 1.27)) hide)
     )
@@
       (effects (font (size 1.27 1.27)) hide)
     )
+    (property "LCSC" "C14996" (id 4) (at 92.71 165.1 0)
+      (effects (font (size 1.27 1.27)) hide)
+    )
     (pin "1")
     (pin "2")
@@
       (effects (font (size 1.27 1.27)) hide)
     )
+    (property "LCSC" "C14996" (id 4) (at 92.71 33.02 0)
+      (effects (font (size 1.27 1.27)) hide)
+    )
     (pin "1")
     (pin "2")
@@
       (effects (font (size 1.27 1.27)) hide)
     )
+    (property "LCSC" "C429066" (id 4) (at 171.45 88.265 0)
+      (effects (font (size 1.27 1.27)) hide)
+    )
     (pin "1")
     (pin "2")
@@
     )
     (property "Datasheet" "~" (id 3) (at 165.1 80.645 0)
+      (effects (font (size 1.27 1.27)) hide)
+    )
+    (property "LCSC" "C499462" (id 4) (at 165.1 80.645 0)
       (effects (font (size 1.27 1.27)) hide)
     )
@@
       (effects (font (size 1.27 1.27)) hide)
     )
+    (property "LCSC" "C434441" (id 4) (at 171.45 80.645 0)
+      (effects (font (size 1.27 1.27)) hide)
+    )
     (pin "1")
     (pin "2")
@@
       (effects (font (size 1.27 1.27)) hide)
     )
+    (property "LCSC" "C429066" (id 4) (at 68.58 81.915 0)
+      (effects (font (size 1.27 1.27)) hide)
+    )
     (pin "1")
     (pin "2")
@@
       (effects (font (size 1.27 1.27)) hide)
     )
+    (property "LCSC" "C429066" (id 4) (at 165.1 136.525 0)
+      (effects (font (size 1.27 1.27)) hide)
+    )
     (pin "1")
     (pin "2")
@@
       (effects (font (size 1.27 1.27)) hide)
     )
+    (property "LCSC" "C499462" (id 4) (at 68.58 74.295 0)
+      (effects (font (size 1.27 1.27)) hide)
+    )
     (pin "1")
     (pin "2")
@@
       (effects (font (size 1.27 1.27)) hide)
     )
+    (property "LCSC" "C429066" (id 4) (at 74.93 38.1 0)
+      (effects (font (size 1.27 1.27)) hide)
+    )
