File: adc.kicad_sch (KiCad schematic)
At the start: 0 parts

Commit message: first revision of full schematic copied over
Parts:
- added C? (x3): 100nF, symbol Device:C
- added J? (x3): Conn_01x08_Female, symbol Connector:Conn_01x08_Female
- added R? (x3): 100k, symbol Device:R_US
- added U? (x3): MCP3208, symbol Analog_ADC:MCP3208
Connections:
- new net +5V: C?.2, C?.2, C?.2, R?.2, R?.2, R?.2, U?.15 (Vref), U?.15 (Vref), U?.15 (Vref), U?.16 (Vdd), U?.16 (Vdd), U?.16 (Vdd)
- new net ADC1_CS: R?.1, U?.10 (~{CS}/SHDN)
- new net ADC2_CS: R?.1, U?.10 (~{CS}/SHDN)
- new net ADC3_CS: R?.1, U?.10 (~{CS}/SHDN)
- new net GND: C?.1, C?.1, C?.1, U?.14 (AGND), U?.14 (AGND), U?.14 (AGND), U?.9 (DGND), U?.9 (DGND), U?.9 (DGND)
- new net LC1_CAL: J?.1 (Pin_1), J?.1 (Pin_1), U?.1 (CH0), U?.1 (CH0)
- new net LC2_CAL: J?.2 (Pin_2), J?.2 (Pin_2), U?.2 (CH1), U?.2 (CH1)
- new net LC3_CAL: J?.3 (Pin_3), J?.3 (Pin_3), U?.3 (CH2), U?.3 (CH2)
- new net LC4_CAL: J?.4 (Pin_4), J?.4 (Pin_4), U?.4 (CH3), U?.4 (CH3)
- new net SPI_CLK: U?.13 (CLK), U?.13 (CLK), U?.13 (CLK)
- new net SPI_MISO: U?.12 (Dout), U?.12 (Dout), U?.12 (Dout)
- new net SPI_MOSI: U?.11 (Din), U?.11 (Din), U?.11 (Din)
- new net TC1: J?.1 (Pin_1), U?.1 (CH0)
- new net TC2: J?.2 (Pin_2), U?.2 (CH1)
- new net TC3: J?.3 (Pin_3), U?.3 (CH2)
- new net TC4: J?.4 (Pin_4), U?.4 (CH3)
- new net acd1_nc7: J?.7 (Pin_7), U?.7 (CH6)
- new net adc1_nc5: J?.5 (Pin_5), U?.5 (CH4)
- new net adc1_nc6: J?.6 (Pin_6), U?.6 (CH5)
- new net adc1_nc8: J?.8 (Pin_8), U?.8 (CH7)
- new net adc2_nc5: J?.5 (Pin_5), U?.5 (CH4)
- new net adc2_nc6: J?.6 (Pin_6), U?.6 (CH5)
- new net adc2_nc7: J?.7 (Pin_7), U?.7 (CH6)
- new net adc2_nc8: J?.8 (Pin_8), U?.8 (CH7)
- new net adc3_nc5: J?.5 (Pin_5), U?.5 (CH4)
- new net adc3_nc6: J?.6 (Pin_6), U?.6 (CH5)
- new net adc3_nc7: J?.7 (Pin_7), U?.7 (CH6)
- new net adc3_nc8: J?.8 (Pin_8), U?.8 (CH7)
Other:
- note added: "ADC1 - Load Cells"
- note added: "ADC2 - Pressure Transducers"
- note added: "ADC3 - Thermocouples"
- company: (none) -> Rice Eclipse
- title: (none) -> ADCs

Commit message: added schematic pdf for review
Parts:
- gave numbers to parts that had none: 12
Changed lines of the file:
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@@
   (symbol (lib_id "power:GND") (at 140.97 50.8 0) (unit 1)
     (in_bom yes) (on_board yes) (fields_autoplaced)
-    (property "Reference" "#PWR?" (id 0) (at 140.97 57.15 0)
+    (property "Reference" "#PWR0121" (id 0) (at 140.97 57.15 0)
       (effects (font (size 1.27 1.27)) hide)
     )
@@
   (symbol (lib_id "Connector:Conn_01x08_Female") (at 43.18 107.95 0) (mirror y) (unit 1)
     (in_bom yes) (on_board yes)
-    (property "Reference" "J?" (id 0) (at 38.1 93.98 0))
+    (property "Reference" "J34" (id 0) (at 38.1 93.98 0))
     (property "Value" "Conn_01x08_Female" (id 1) (at 38.1 96.52 0))
     (property "Footprint" "" (id 2) (at 43.18 107.95 0)
@@
   (symbol (lib_id "Device:C") (at 140.97 46.99 180) (unit 1)
     (in_bom yes) (on_board yes) (fields_autoplaced)
-    (property "Reference" "C?" (id 0) (at 144.78 45.7199 0)
+    (property "Reference" "C27" (id 0) (at 144.78 45.7199 0)
       (effects (font (size 1.27 1.27)) (justify right))
     )
@@
   (symbol (lib_id "power:GND") (at 140.97 110.49 0) (unit 1)
     (in_bom yes) (on_board yes) (fields_autoplaced)
-    (property "Reference" "#PWR?" (id 0) (at 140.97 116.84 0)
+    (property "Reference" "#PWR0123" (id 0) (at 140.97 116.84 0)
       (effects (font (size 1.27 1.27)) hide)
     )
@@
   (symbol (lib_id "Analog_ADC:MCP3208") (at 73.66 107.95 0) (unit 1)
     (in_bom yes) (on_board yes)
-    (property "Reference" "U?" (id 0) (at 58.42 91.44 0)
+    (property "Reference" "U10" (id 0) (at 58.42 91.44 0)
       (effects (font (size 1.27 1.27)) (justify left))
     )
@@
   (symbol (lib_id "power:+5V") (at 74.93 95.25 0) (unit 1)
     (in_bom yes) (on_board yes) (fields_autoplaced)
-    (property "Reference" "#PWR?" (id 0) (at 74.93 99.06 0)
+    (property "Reference" "#PWR0113" (id 0) (at 74.93 99.06 0)
       (effects (font (size 1.27 1.27)) hide)
     )
@@
   (symbol (lib_id "power:+5V") (at 114.3 100.33 0) (unit 1)
     (in_bom yes) (on_board yes) (fields_autoplaced)
-    (property "Reference" "#PWR?" (id 0) (at 114.3 104.14 0)
+    (property "Reference" "#PWR0118" (id 0) (at 114.3 104.14 0)
       (effects (font (size 1.27 1.27)) hide)
     )
@@
   (symbol (lib_id "Connector:Conn_01x08_Female") (at 43.18 48.26 0) (mirror y) (unit 1)
     (in_bom yes) (on_board yes)
-    (property "Reference" "J?" (id 0) (at 38.1 34.29 0))
+    (property "Reference" "J33" (id 0) (at 38.1 34.29 0))
     (property "Value" "Conn_01x08_Female" (id 1) (at 38.1 36.83 0))
     (property "Footprint" "" (id 2) (at 43.18 48.26 0)
@@
   (symbol (lib_id "power:GND") (at 74.93 63.5 0) (unit 1)
     (in_bom yes) (on_board yes) (fields_autoplaced)
-    (property "Reference" "#PWR?" (id 0) (at 74.93 69.85 0)
+    (property "Reference" "#PWR0112" (id 0) (at 74.93 69.85 0)
       (effects (font (size 1.27 1.27)) hide)
     )
@@
   (symbol (lib_id "Device:C") (at 140.97 106.68 180) (unit 1)
     (in_bom yes) (on_board yes) (fields_autoplaced)
-    (property "Reference" "C?" (id 0) (at 144.78 105.4099 0)
+    (property "Reference" "C28" (id 0) (at 144.78 105.4099 0)
       (effects (font (size 1.27 1.27)) (justify right))
     )
@@
   (symbol (lib_id "power:+5V") (at 74.93 154.94 0) (unit 1)
     (in_bom yes) (on_board yes) (fields_autoplaced)
-    (property "Reference" "#PWR?" (id 0) (at 74.93 158.75 0)
+    (property "Reference" "#PWR0115" (id 0) (at 74.93 158.75 0)
       (effects (font (size 1.27 1.27)) hide)
     )
@@
   (symbol (lib_id "power:GND") (at 74.93 123.19 0) (unit 1)
     (in_bom yes) (on_board yes) (fields_autoplaced)
-    (property "Reference" "#PWR?" (id 0) (at 74.93 129.54 0)
+    (property "Reference" "#PWR0114" (id 0) (at 74.93 129.54 0)
       (effects (font (size 1.27 1.27)) hide)
     )
@@
   (symbol (lib_id "Device:R_US") (at 114.3 44.45 180) (unit 1)
     (in_bom yes) (on_board yes) (fields_autoplaced)
-    (property "Reference" "R?" (id 0) (at 116.84 43.1799 0)
+    (property "Reference" "R74" (id 0) (at 116.84 43.1799 0)
       (effects (font (size 1.27 1.27)) (justify right))
     )
@@
   (symbol (lib_id "power:+5V") (at 114.3 160.02 0) (unit 1)
     (in_bom yes) (on_board yes) (fields_autoplaced)
-    (property "Reference" "#PWR?" (id 0) (at 114.3 163.83 0)
+    (property "Reference" "#PWR0119" (id 0) (at 114.3 163.83 0)
       (effects (font (size 1.27 1.27)) hide)
     )
@@
   (symbol (lib_id "Device:C") (at 140.97 166.37 180) (unit 1)
     (in_bom yes) (on_board yes) (fields_autoplaced)
-    (property "Reference" "C?" (id 0) (at 144.78 165.0999 0)
+    (property "Reference" "C29" (id 0) (at 144.78 165.0999 0)
       (effects (font (size 1.27 1.27)) (justify right))
     )
@@
   (symbol (lib_id "power:+5V") (at 140.97 43.18 0) (unit 1)
     (in_bom yes) (on_board yes) (fields_autoplaced)
-    (property "Reference" "#PWR?" (id 0) (at 140.97 46.99 0)
+    (property "Reference" "#PWR0120" (id 0) (at 140.97 46.99 0)
       (effects (font (size 1.27 1.27)) hide)
     )
@@
   (symbol (lib_id "Device:R_US") (at 114.3 104.14 180) (unit 1)
     (in_bom yes) (on_board yes) (fields_autoplaced)
-    (property "Reference" "R?" (id 0) (at 116.84 102.8699 0)
+    (property "Reference" "R75" (id 0) (at 116.84 102.8699 0)
       (effects (font (size 1.27 1.27)) (justify right))
     )
@@
   (symbol (lib_id "Analog_ADC:MCP3208") (at 73.66 48.26 0) (unit 1)
     (in_bom yes) (on_board yes)
-    (property "Reference" "U?" (id 0) (at 58.42 31.75 0)
+    (property "Reference" "U9" (id 0) (at 58.42 31.75 0)
       (effects (font (size 1.27 1.27)) (justify left))
     )
@@
   (symbol (lib_id "power:GND") (at 74.93 182.88 0) (unit 1)
     (in_bom yes) (on_board yes) (fields_autoplaced)
-    (property "Reference" "#PWR?" (id 0) (at 74.93 189.23 0)
+    (property "Reference" "#PWR0116" (id 0) (at 74.93 189.23 0)
       (effects (font (size 1.27 1.27)) hide)
     )
@@
   (symbol (lib_id "power:+5V") (at 114.3 40.64 0) (unit 1)
     (in_bom yes) (on_board yes) (fields_autoplaced)
-    (property "Reference" "#PWR?" (id 0) (at 114.3 44.45 0)
+    (property "Reference" "#PWR0117" (id 0) (at 114.3 44.45 0)
       (effects (font (size 1.27 1.27)) hide)
     )
@@
   (symbol (lib_id "power:+5V") (at 140.97 162.56 0) (unit 1)
     (in_bom yes) (on_board yes) (fields_autoplaced)
-    (property "Reference" "#PWR?" (id 0) (at 140.97 166.37 0)
+    (property "Reference" "#PWR0124" (id 0) (at 140.97 166.37 0)
       (effects (font (size 1.27 1.27)) hide)
     )
@@
   (symbol (lib_id "power:+5V") (at 74.93 35.56 0) (unit 1)
     (in_bom yes) (on_board yes) (fields_autoplaced)
-    (property "Reference" "#PWR?" (id 0) (at 74.93 39.37 0)
+    (property "Reference" "#PWR0111" (id 0) (at 74.93 39.37 0)
       (effects (font (size 1.27 1.27)) hide)
     )
@@
   (symbol (lib_id "Analog_ADC:MCP3208") (at 73.66 167.64 0) (unit 1)
     (in_bom yes) (on_board yes)
-    (property "Reference" "U?" (id 0) (at 58.42 151.13 0)
+    (property "Reference" "U11" (id 0) (at 58.42 151.13 0)
       (effects (font (size 1.27 1.27)) (justify left))
     )
@@
   (symbol (lib_id "power:+5V") (at 140.97 102.87 0) (unit 1)
     (in_bom yes) (on_board yes) (fields_autoplaced)
-    (property "Reference" "#PWR?" (id 0) (at 140.97 106.68 0)
+    (property "Reference" "#PWR0122" (id 0) (at 140.97 106.68 0)
       (effects (font (size 1.27 1.27)) hide)
     )
@@
   (symbol (lib_id "Device:R_US") (at 114.3 163.83 180) (unit 1)
     (in_bom yes) (on_board yes) (fields_autoplaced)
-    (property "Reference" "R?" (id 0) (at 116.84 162.5599 0)
+    (property "Reference" "R76" (id 0) (at 116.84 162.5599 0)
       (effects (font (size 1.27 1.27)) (justify right))
     )
@@
   (symbol (lib_id "power:GND") (at 140.97 170.18 0) (unit 1)
     (in_bom yes) (on_board yes) (fields_autoplaced)
-    (property "Reference" "#PWR?" (id 0) (at 140.97 176.53 0)
+    (property "Reference" "#PWR0125" (id 0) (at 140.97 176.53 0)
       (effects (font (size 1.27 1.27)) hide)
     )
@@
   (symbol (lib_id "Connector:Conn_01x08_Female") (at 43.18 167.64 0) (mirror y) (unit 1)
     (in_bom yes) (on_board yes)
-    (property "Reference" "J?" (id 0) (at 38.1 153.67 0))
+    (property "Reference" "J35" (id 0) (at 38.1 153.67 0))
     (property "Value" "Conn_01x08_Female" (id 1) (at 38.1 156.21 0))
     (property "Footprint" "" (id 2) (at 43.18 167.64 0)

Commit message: added footprints and started schematic review revisions
Parts:
- C27, C28, C29: footprint (none) -> Capacitor_SMD:C_1206_3216Metric
- R74, R75, R76: footprint (none) -> Resistor_SMD:R_1206_3216Metric
- U10, U11, U9: value MCP3208 -> MCP3208-CI/SL; footprint (none) -> Package_SO:SOIC-16_3.9x9.9mm_P1.27mm
Changed lines of the file:
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@@
       (effects (font (size 1.27 1.27)) (justify right))
     )
-    (property "Footprint" "" (id 2) (at 140.0048 43.18 0)
+    (property "Footprint" "Capacitor_SMD:C_1206_3216Metric" (id 2) (at 140.0048 43.18 0)
       (effects (font (size 1.27 1.27)) hide)
     )
@@
       (effects (font (size 1.27 1.27)) (justify left))
     )
-    (property "Value" "MCP3208" (id 1) (at 58.42 93.98 0)
-      (effects (font (size 1.27 1.27)) (justify left))
-    )
-    (property "Footprint" "" (id 2) (at 76.2 105.41 0)
-      (effects (font (size 1.27 1.27)) hide)
-    )
-    (property "Datasheet" "http://ww1.microchip.com/downloads/en/DeviceDoc/21298c.pdf" (id 3) (at 76.2 105.41 0)
+    (property "Value" "MCP3208-CI/SL" (id 1) (at 58.42 93.98 0)
+      (effects (font (size 1.27 1.27)) (justify left))
+    )
+    (property "Footprint" "Package_SO:SOIC-16_3.9x9.9mm_P1.27mm" (id 2) (at 76.2 105.41 0)
+      (effects (font (size 1.27 1.27)) hide)
+    )
+    (property "Datasheet" "https://www.mouser.com/datasheet/2/268/21298e-1101808.pdf" (id 3) (at 76.2 105.41 0)
       (effects (font (size 1.27 1.27)) hide)
     )
@@
       (effects (font (size 1.27 1.27)) (justify right))
     )
-    (property "Footprint" "" (id 2) (at 140.0048 102.87 0)
+    (property "Footprint" "Capacitor_SMD:C_1206_3216Metric" (id 2) (at 140.0048 102.87 0)
       (effects (font (size 1.27 1.27)) hide)
     )
@@
       (effects (font (size 1.27 1.27)) (justify right))
     )
-    (property "Footprint" "" (id 2) (at 113.284 44.196 90)
+    (property "Footprint" "Resistor_SMD:R_1206_3216Metric" (id 2) (at 113.284 44.196 90)
       (effects (font (size 1.27 1.27)) hide)
     )
@@
       (effects (font (size 1.27 1.27)) (justify right))
     )
-    (property "Footprint" "" (id 2) (at 140.0048 162.56 0)
+    (property "Footprint" "Capacitor_SMD:C_1206_3216Metric" (id 2) (at 140.0048 162.56 0)
       (effects (font (size 1.27 1.27)) hide)
     )
@@
       (effects (font (size 1.27 1.27)) (justify right))
     )
-    (property "Footprint" "" (id 2) (at 113.284 103.886 90)
+    (property "Footprint" "Resistor_SMD:R_1206_3216Metric" (id 2) (at 113.284 103.886 90)
       (effects (font (size 1.27 1.27)) hide)
     )
@@
       (effects (font (size 1.27 1.27)) (justify left))
     )
-    (property "Value" "MCP3208" (id 1) (at 58.42 34.29 0)
-      (effects (font (size 1.27 1.27)) (justify left))
-    )
-    (property "Footprint" "" (id 2) (at 76.2 45.72 0)
-      (effects (font (size 1.27 1.27)) hide)
-    )
-    (property "Datasheet" "http://ww1.microchip.com/downloads/en/DeviceDoc/21298c.pdf" (id 3) (at 76.2 45.72 0)
+    (property "Value" "MCP3208-CI/SL" (id 1) (at 58.42 34.29 0)
+      (effects (font (size 1.27 1.27)) (justify left))
+    )
+    (property "Footprint" "Package_SO:SOIC-16_3.9x9.9mm_P1.27mm" (id 2) (at 76.2 45.72 0)
+      (effects (font (size 1.27 1.27)) hide)
+    )
+    (property "Datasheet" "https://www.mouser.com/datasheet/2/268/21298e-1101808.pdf" (id 3) (at 76.2 45.72 0)
       (effects (font (size 1.27 1.27)) hide)
     )
@@
       (effects (font (size 1.27 1.27)) (justify left))
     )
-    (property "Value" "MCP3208" (id 1) (at 58.42 153.67 0)
-      (effects (font (size 1.27 1.27)) (justify left))
-    )
-    (property "Footprint" "" (id 2) (at 76.2 165.1 0)
-      (effects (font (size 1.27 1.27)) hide)
-    )
-    (property "Datasheet" "http://ww1.microchip.com/downloads/en/DeviceDoc/21298c.pdf" (id 3) (at 76.2 165.1 0)
+    (property "Value" "MCP3208-CI/SL" (id 1) (at 58.42 153.67 0)
+      (effects (font (size 1.27 1.27)) (justify left))
+    )
+    (property "Footprint" "Package_SO:SOIC-16_3.9x9.9mm_P1.27mm" (id 2) (at 76.2 165.1 0)
+      (effects (font (size 1.27 1.27)) hide)
+    )
+    (property "Datasheet" "https://www.mouser.com/datasheet/2/268/21298e-1101808.pdf" (id 3) (at 76.2 165.1 0)
       (effects (font (size 1.27 1.27)) hide)
     )
@@
       (effects (font (size 1.27 1.27)) (justify right))
     )
-    (property "Footprint" "" (id 2) (at 113.284 163.576 90)
-      (effects (font (size 1.27 1.27)) hide)
-    )
+    (property "Footprint" "Resistor_SMD:R_1206_3216Metric" (id 2) (at 113.284 163.576 90)
+      (effects (font (size 1.27 1.27)) hide)
+    )

Commit message: schematic editing + creating some footprints
Parts:
- J33, J34, J35: symbol Connector:Conn_01x08_Female -> Connector_Generic:Conn_01x08
Changed lines of the file:
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@@
     (pin "1")
   )
-  (symbol (lib_id "Connector:Conn_01x08_Female") (at 43.18 107.95 0) (mirror y) (unit 1)
+  (symbol (lib_id "Connector_Generic:Conn_01x08") (at 43.18 107.95 0) (mirror y) (unit 1)
     (in_bom yes) (on_board yes)
     (property "Reference" "J34" (id 0) (at 38.1 93.98 0))
@@
     (pin "1")
   )
-  (symbol (lib_id "Connector:Conn_01x08_Female") (at 43.18 48.26 0) (mirror y) (unit 1)
+  (symbol (lib_id "Connector_Generic:Conn_01x08") (at 43.18 48.26 0) (mirror y) (unit 1)
     (in_bom yes) (on_board yes)
     (property "Reference" "J33" (id 0) (at 38.1 34.29 0))
@@
     (pin "1")
   )
-  (symbol (lib_id "Connector:Conn_01x08_Female") (at 43.18 167.64 0) (mirror y) (unit 1)
+  (symbol (lib_id "Connector_Generic:Conn_01x08") (at 43.18 167.64 0) (mirror y) (unit 1)
     (in_bom yes) (on_board yes)
     (property "Reference" "J35" (id 0) (at 38.1 153.67 0))

Commit message: updated all footprints, resolved most ERC & setup layout
Parts:
- J33, J34, J35: footprint (none) -> Connector_PinSocket_2.54mm:PinSocket_1x08_P2.54mm_Vertical
Changed lines of the file:
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@@
     (property "Reference" "J34" (id 0) (at 38.1 93.98 0))
     (property "Value" "Conn_01x08_Female" (id 1) (at 38.1 96.52 0))
-    (property "Footprint" "" (id 2) (at 43.18 107.95 0)
+    (property "Footprint" "Connector_PinSocket_2.54mm:PinSocket_1x08_P2.54mm_Vertical" (id 2) (at 43.18 107.95 0)
       (effects (font (size 1.27 1.27)) hide)
     )
@@
     (property "Reference" "J33" (id 0) (at 38.1 34.29 0))
     (property "Value" "Conn_01x08_Female" (id 1) (at 38.1 36.83 0))
-    (property "Footprint" "" (id 2) (at 43.18 48.26 0)
+    (property "Footprint" "Connector_PinSocket_2.54mm:PinSocket_1x08_P2.54mm_Vertical" (id 2) (at 43.18 48.26 0)
       (effects (font (size 1.27 1.27)) hide)
     )
@@
     (property "Reference" "J35" (id 0) (at 38.1 153.67 0))
     (property "Value" "Conn_01x08_Female" (id 1) (at 38.1 156.21 0))
-    (property "Footprint" "" (id 2) (at 43.18 167.64 0)
-      (effects (font (size 1.27 1.27)) hide)
-    )
+    (property "Footprint" "Connector_PinSocket_2.54mm:PinSocket_1x08_P2.54mm_Vertical" (id 2) (at 43.18 167.64 0)
+      (effects (font (size 1.27 1.27)) hide)
+    )

Commit message: preliminary layout and started pwr plane config
Parts:
- renumbered C27 to C34, C28 to C35, C29 to C36, J33 to J30, J34 to J31, J35 to J32, R74 to R86, R75 to R87, R76 to R88, U9 to U12, U10 to U13, U11 to U14
Connections:
- net LC1_CAL: no longer J31.1 (Pin_1), U13.1 (CH0)
- net LC2_CAL: no longer J31.2 (Pin_2), U13.2 (CH1)
- net LC3_CAL: no longer J31.3 (Pin_3), U13.3 (CH2)
- net LC4_CAL: no longer J31.4 (Pin_4), U13.4 (CH3)
- net adc1_nc5 renamed LC5_CAL
- net adc1_nc6 renamed LC6_CAL
- new net PT1_CAL: J31.1 (Pin_1), U13.1 (CH0)
- new net PT2_CAL: J31.2 (Pin_2), U13.2 (CH1)
- new net PT3_CAL: J31.3 (Pin_3), U13.3 (CH2)
- new net PT4_CAL: J31.4 (Pin_4), U13.4 (CH3)

Commit message: some minor schematic cleanup
Parts:
- C34, C35, C36: value 100nF -> 100n
- J30, J31, J32: symbol Connector_Generic:Conn_01x08 -> Connector:Conn_01x08_Female
Other:
- moved on the sheet: R86, R87
