File: adc.kicad_sch (KiCad schematic)
At the start: 12 parts, among them J30 Conn_01x08_Female, J31 Conn_01x08_Female, J32 Conn_01x08_Female, U12 MCP3208-CI/SL, U13 MCP3208-CI/SL, U14 MCP3208-CI/SL

Commit message: shuffle around some parts
Parts:
- removed R86, R87, R88: 100k, Resistor_SMD:R_1206_3216Metric, symbol Device:R_US
Other:
- moved on the sheet: J30, J31

Commit message: enshrinkening of the board
Connections:
- net LC5_CAL: no longer names the net of J30.5 (Pin_5), U12.5 (CH4)
- net LC6_CAL: no longer names the net of J30.6 (Pin_6), U12.6 (CH5)
Other:
- moved on the sheet: J30

Commit message: done routing on shrunk board
Parts:
- renumbered U12 to ADC1, U13 to ADC2, U14 to ADC3
Changed lines of the file:
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@@
   (symbol (lib_id "Analog_ADC:MCP3208") (at 73.66 107.95 0) (unit 1)
     (in_bom yes) (on_board yes)
-    (property "Reference" "U13" (id 0) (at 57.15 91.44 0)
+    (property "Reference" "ADC2" (id 0) (at 57.15 91.44 0)
       (effects (font (size 1.27 1.27)) (justify left))
     )
@@
   (symbol (lib_id "Analog_ADC:MCP3208") (at 73.66 48.26 0) (unit 1)
     (in_bom yes) (on_board yes)
-    (property "Reference" "U12" (id 0) (at 57.15 31.75 0)
+    (property "Reference" "ADC1" (id 0) (at 57.15 31.75 0)
       (effects (font (size 1.27 1.27)) (justify left))
     )
@@
   (symbol (lib_id "Analog_ADC:MCP3208") (at 73.66 167.64 0) (unit 1)
     (in_bom yes) (on_board yes)
-    (property "Reference" "U14" (id 0) (at 57.15 151.13 0)
-      (effects (font (size 1.27 1.27)) (justify left))
-    )
+    (property "Reference" "ADC3" (id 0) (at 57.15 151.13 0)
+      (effects (font (size 1.27 1.27)) (justify left))
+    )

Commit message: done schematiccing after design review
Parts:
- removed ADC1, ADC2, ADC3: MCP3208-CI/SL, Package_SO:SOIC-16_3.9x9.9mm_P1.27mm, symbol Analog_ADC:MCP3208
- removed C34, C35, C36: 100n, Capacitor_SMD:C_1206_3216Metric, symbol Device:C
- removed J30, J31, J32: Conn_01x08_Female, Connector_PinSocket_2.54mm:PinSocket_1x08_P2.54mm_Vertical, symbol Connector:Conn_01x08_Female
