File: lc_inamps.kicad_sch (KiCad schematic)
At the start: 0 parts

Commit message: secret arca meetings
Parts:
- added C? (x4): 1uF, symbol Device:C_Polarized
- added F? (x4): Fuse, symbol Device:Fuse
- added J? (x16): Conn_01x01_Male, symbol Connector:Conn_01x01_Male
- added J?: Conn_01x04, symbol Connector_Generic:Conn_01x04
- added J?: Conn_01x08, symbol Connector_Generic:Conn_01x08
- added R? (x4): 20K, symbol Device:R_US
- added R? (x4): 200, symbol Device:R_US
- added RV? (x4): 30k, symbol Device:R_Potentiometer
- added U? (x4): MCP6N11R, symbol karca_custom_components:MCP6N11R
Connections:
- new net: R?.1, U?.1 (Vfg) (x4)
- new net: R?.1, RV?.2, U?.5 (Vref) (x4)
- new net: F?.2, J?.1 (Pin_1) (x4)
- new net +5V: C?.1, C?.1, C?.1, C?.1, F?.1, F?.1, F?.1, F?.1, RV?.1, RV?.1, RV?.1, RV?.1, U?.7 (Vdd), U?.7 (Vdd), U?.7 (Vdd), U?.7 (Vdd), U?.8 (EN/nCAL), U?.8 (EN/nCAL), U?.8 (EN/nCAL), U?.8 (EN/nCAL)
- new net GND: C?.2, C?.2, C?.2, C?.2, J?.1 (Pin_1), J?.1 (Pin_1), J?.1 (Pin_1), J?.1 (Pin_1), RV?.3, RV?.3, RV?.3, RV?.3, U?.4 (Vss), U?.4 (Vss), U?.4 (Vss), U?.4 (Vss)
- new net LC1+: J?.1 (Pin_1), J?.1 (Pin_1), U?.3 (Vip)
- new net LC1-: J?.1 (Pin_1), J?.2 (Pin_2), U?.2 (Vim)
- new net LC1_PREC: J?.1 (Pin_1), R?.2, R?.2, U?.6 (Vout)
- new net LC2+: J?.1 (Pin_1), J?.3 (Pin_3), U?.3 (Vip)
- new net LC2-: J?.1 (Pin_1), J?.4 (Pin_4), U?.2 (Vim)
- new net LC2_PREC: J?.2 (Pin_2), R?.2, R?.2, U?.6 (Vout)
- new net LC3+: J?.1 (Pin_1), J?.5 (Pin_5), U?.3 (Vip)
- new net LC3-: J?.1 (Pin_1), J?.6 (Pin_6), U?.2 (Vim)
- new net LC3_PREC: J?.3 (Pin_3), R?.2, R?.2, U?.6 (Vout)
- new net LC4+: J?.1 (Pin_1), J?.7 (Pin_7), U?.3 (Vip)
- new net LC4-: J?.1 (Pin_1), J?.8 (Pin_8), U?.2 (Vim)
- new net LC4_PREC: J?.4 (Pin_4), R?.2, R?.2, U?.6 (Vout)
Other:
- note added: "Inamp 1"
- note added: "Inamp 2"
- note added: "Inamp 3"
- note added: "Inamp 4"

Commit message: first revision of full schematic copied over
Parts:
- removed C? (x4): 1uF, symbol Device:C_Polarized
- removed F? (x3): Fuse, symbol Device:Fuse
- removed J? (x16): Conn_01x01_Male, symbol Connector:Conn_01x01_Male
- removed R? (x3): 20K, symbol Device:R_US
- removed R? (x3): 200, symbol Device:R_US
- removed RV? (x3): 30k, symbol Device:R_Potentiometer
- removed U? (x3): MCP6N11R, symbol karca_custom_components:MCP6N11R
- added C? (x4): 1uF, symbol Device:C
- added F? (x3): Fuse, symbol Device:Fuse
- added J? (x4): Conn_01x04_Male, symbol Connector:Conn_01x04_Male
- added R? (x3): 200, symbol Device:R_US
- added R? (x3): 20K, symbol Device:R_US
- added RV? (x3): 30k, symbol Device:R_Potentiometer
- added U? (x3): MCP6N11R, symbol karca_custom_components:MCP6N11R
Connections:
- net +5V: now also C?.1, C?.1, C?.1, C?.1, F?.1, F?.1, F?.1, RV?.1, RV?.1, RV?.1, U?.7 (Vdd), U?.7 (Vdd), U?.7 (Vdd), U?.8 (EN/nCAL), U?.8 (EN/nCAL), U?.8 (EN/nCAL)
- net GND: now also C?.2, C?.2, C?.2, C?.2, J?.4 (Pin_4), J?.4 (Pin_4), J?.4 (Pin_4), J?.4 (Pin_4), RV?.3, RV?.3, RV?.3, U?.4 (Vss), U?.4 (Vss), U?.4 (Vss)
- net LC1+: now also J?.3 (Pin_3), U?.3 (Vip)
- net LC1-: now also J?.2 (Pin_2), U?.2 (Vim)
- net LC1_PREC: now also R?.1, R?.2, U?.6 (Vout)
- net LC2+: now also J?.3 (Pin_3), U?.3 (Vip)
- net LC2-: now also J?.2 (Pin_2), U?.2 (Vim)
- net LC2_PREC: now also R?.1, R?.2, U?.6 (Vout)
- net LC3+: now also J?.3 (Pin_3)
- net LC3-: now also J?.2 (Pin_2)
- net LC3_PREC: now also R?.1; no longer R?.2
- net LC4+: now also J?.3 (Pin_3), U?.3 (Vip)
- net LC4-: now also J?.2 (Pin_2), U?.2 (Vim)
- net LC4_PREC: now also R?.1, R?.2, U?.6 (Vout)
- net at U?.1 (Vfg): now also R?.2; no longer R?.1
- net at F?.2: now also J?.1 (Pin_1)
- new net: F?.2, J?.1 (Pin_1) (x3)
- new net: R?.1, RV?.2, U?.5 (Vref) (x3)
- new net: R?.2, U?.1 (Vfg) (x3)
Other:
- company: (none) -> Rice Eclipse
- title: (none) -> Load Cell InAmps
- moved on the sheet: F?, R?, RV?, U?

Commit message: added schematic pdf for review
Parts:
- gave numbers to parts that had none: 30

Commit message: added footprints and started schematic review revisions
Parts:
- C5, C6, C7, C8: footprint (none) -> Capacitor_SMD:C_1206_3216Metric
- F10, F7, F8, F9: value Fuse -> 3588-20; footprint (none) -> karca_custom_footprints:3588-20 fuse
- R30, R31, R32, R33, R34, R35, R36, R37, RV1, RV2, RV3, RV4: footprint (none) -> Resistor_SMD:R_1206_3216Metric
- U3, U4, U5, U6: value MCP6N11R -> MCP6N11T-001E; footprint (none) -> Package_DFN_QFN:TDFN-8-1EP_3x2mm_P0.5mm_EP1.80x1.65mm
Other:
- moved on the sheet: C5, C6, C7, C8, F10, F7, F8, F9, J14, J15, J18, J19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

Commit message: schematic editing + creating some footprints
Parts:
- removed J14, J15, J18, J19: Conn_01x04_Male, symbol Connector:Conn_01x04_Male
- removed J16: Conn_01x04, symbol Connector_Generic:Conn_01x04
- removed J17: Conn_01x08, symbol Connector_Generic:Conn_01x08
- added J14, J17, J18, J6: Conn_01x04_Female, karca_custom_footprints:LPTA-4pos, symbol Connector:Conn_01x04_Female
- added J15: Conn_01x04_Female, Connector_PinHeader_2.54mm:PinHeader_1x04_P2.54mm_Vertical, symbol Connector:Conn_01x04_Female
- added J16: Conn_01x08_Female, symbol Connector:Conn_01x08_Female
Connections:
- net GND: now also J14.4 (Pin_4), J17.4 (Pin_4), J18.4 (Pin_4), J6.4 (Pin_4)
- net LC1+: now also J14.3 (Pin_3), J16.1 (Pin_1)
- net LC1-: now also J14.2 (Pin_2), J16.2 (Pin_2)
- net LC1_PREC: now also J15.1 (Pin_1)
- net LC2+: now also J16.3 (Pin_3), J17.3 (Pin_3)
- net LC2-: now also J16.4 (Pin_4), J17.2 (Pin_2)
- net LC2_PREC: now also J15.2 (Pin_2)
- net LC3+: now also J16.5 (Pin_5), J6.3 (Pin_3)
- net LC3-: now also J16.6 (Pin_6), J6.2 (Pin_2)
- net LC3_PREC: now also J15.3 (Pin_3)
- net LC4+: now also J16.7 (Pin_7), J18.3 (Pin_3)
- net LC4-: now also J16.8 (Pin_8), J18.2 (Pin_2)
- net LC4_PREC: now also J15.4 (Pin_4)
- net at F10.2: now also J18.1 (Pin_1)
- net at F7.2: now also J14.1 (Pin_1)
- net at F8.2: now also J6.1 (Pin_1)
- net at F9.2: now also J17.1 (Pin_1)

Commit message: updated all footprints, resolved most ERC & setup layout
Parts:
- J16: footprint (none) -> Connector_PinSocket_2.54mm:PinSocket_1x08_P2.54mm_Vertical
- RV1, RV2, RV3, RV4: footprint Resistor_SMD:R_1206_3216Metric -> 3296W-1-303LF:TRIM_3296W-1-303LF
Connections:
- net GND: now also U3.9 (PAD), U4.9 (PAD), U5.9 (PAD), U6.9 (PAD)
Changed lines of the file:
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@@
       (effects (font (size 1.27 1.27)) (justify right))
     )
-    (property "Footprint" "Resistor_SMD:R_1206_3216Metric" (id 2) (at 83.82 132.08 0)
+    (property "Footprint" "3296W-1-303LF:TRIM_3296W-1-303LF" (id 2) (at 83.82 132.08 0)
       (effects (font (size 1.27 1.27)) hide)
     )
@@
       (effects (font (size 1.27 1.27)) (justify right))
     )
-    (property "Footprint" "Resistor_SMD:R_1206_3216Metric" (id 2) (at 193.04 66.04 0)
+    (property "Footprint" "3296W-1-303LF:TRIM_3296W-1-303LF" (id 2) (at 193.04 66.04 0)
       (effects (font (size 1.27 1.27)) hide)
     )
@@
     (pin "1")
   )
-  (symbol (lib_id "karca_custom_components:MCP6N11R") (at 48.26 113.03 0) (unit 1)
+  (symbol (lib_name "MCP6N11R_3") (lib_id "karca_custom_components:MCP6N11R") (at 48.26 113.03 0) (unit 1)
     (in_bom yes) (on_board yes) (fields_autoplaced)
     (property "Reference" "U4" (id 0) (at 55.245 113.03 0))
@@
     (pin "7")
     (pin "8")
+    (pin "9")
   )
   (symbol (lib_id "power:+5V") (at 146.05 44.45 0) (unit 1)
@@
       (effects (font (size 1.27 1.27)) (justify right))
     )
-    (property "Footprint" "Resistor_SMD:R_1206_3216Metric" (id 2) (at 88.9 62.23 0)
+    (property "Footprint" "3296W-1-303LF:TRIM_3296W-1-303LF" (id 2) (at 88.9 62.23 0)
       (effects (font (size 1.27 1.27)) hide)
     )
@@
     (pin "1")
     (pin "2")
+  )
+  (symbol (lib_id "power:GND") (at 163.83 133.35 0) (unit 1)
+    (in_bom yes) (on_board yes) (fields_autoplaced)
+    (property "Reference" "#PWR0132" (id 0) (at 163.83 139.7 0)
+      (effects (font (size 1.27 1.27)) hide)
+    )
+    (property "Value" "GND" (id 1) (at 163.83 138.43 0))
+    (property "Footprint" "" (id 2) (at 163.83 133.35 0)
+      (effects (font (size 1.27 1.27)) hide)
+    )
+    (property "Datasheet" "" (id 3) (at 163.83 133.35 0)
+      (effects (font (size 1.27 1.27)) hide)
+    )
+    (pin "1")
   )
   (symbol (lib_id "Connector:Conn_01x04_Female") (at 38.1 53.34 0) (mirror y) (unit 1)
@@
     (pin "4")
   )
+  (symbol (lib_id "power:GND") (at 162.56 64.77 0) (unit 1)
+    (in_bom yes) (on_board yes) (fields_autoplaced)
+    (property "Reference" "#PWR0131" (id 0) (at 162.56 71.12 0)
+      (effects (font (size 1.27 1.27)) hide)
+    )
+    (property "Value" "GND" (id 1) (at 162.56 69.85 0))
+    (property "Footprint" "" (id 2) (at 162.56 64.77 0)
+      (effects (font (size 1.27 1.27)) hide)
+    )
+    (property "Datasheet" "" (id 3) (at 162.56 64.77 0)
+      (effects (font (size 1.27 1.27)) hide)
+    )
+    (pin "1")
+  )
   (symbol (lib_id "Device:R_US") (at 180.34 114.3 180) (unit 1)
     (in_bom yes) (on_board yes)
@@
       (effects (font (size 1.27 1.27)) (justify right))
     )
-    (property "Footprint" "Resistor_SMD:R_1206_3216Metric" (id 2) (at 193.04 134.62 0)
+    (property "Footprint" "3296W-1-303LF:TRIM_3296W-1-303LF" (id 2) (at 193.04 134.62 0)
       (effects (font (size 1.27 1.27)) hide)
     )
@@
     )
     (property "Datasheet" "" (id 3) (at 85.09 107.95 0)
+      (effects (font (size 1.27 1.27)) hide)
+    )
+    (pin "1")
+  )
+  (symbol (lib_id "power:GND") (at 59.69 62.23 0) (unit 1)
+    (in_bom yes) (on_board yes) (fields_autoplaced)
+    (property "Reference" "#PWR0129" (id 0) (at 59.69 68.58 0)
+      (effects (font (size 1.27 1.27)) hide)
+    )
+    (property "Value" "GND" (id 1) (at 59.69 67.31 0))
+    (property "Footprint" "" (id 2) (at 59.69 62.23 0)
+      (effects (font (size 1.27 1.27)) hide)
+    )
+    (property "Datasheet" "" (id 3) (at 59.69 62.23 0)
       (effects (font (size 1.27 1.27)) hide)
     )
@@
     (pin "7")
     (pin "8")
+    (pin "9")
   )
   (symbol (lib_id "Connector:Conn_01x04_Female") (at 33.02 121.92 0) (mirror y) (unit 1)
@@
       (effects (font (size 1.27 1.27)) (justify left))
     )
-    (property "Footprint" "" (id 2) (at 110.49 167.64 0)
+    (property "Footprint" "Connector_PinSocket_2.54mm:PinSocket_1x08_P2.54mm_Vertical" (id 2) (at 110.49 167.64 0)
       (effects (font (size 1.27 1.27)) hide)
     )
@@
     (pin "1")
   )
-  (symbol (lib_id "karca_custom_components:MCP6N11R") (at 53.34 44.45 0) (unit 1)
+  (symbol (lib_name "MCP6N11R_2") (lib_id "karca_custom_components:MCP6N11R") (at 53.34 44.45 0) (unit 1)
     (in_bom yes) (on_board yes) (fields_autoplaced)
     (property "Reference" "U3" (id 0) (at 60.325 44.45 0))
@@
     (pin "7")
     (pin "8")
+    (pin "9")
   )
   (symbol (lib_id "Device:R_US") (at 180.34 124.46 180) (unit 1)
@@
     (pin "3")
     (pin "4")
+  )
+  (symbol (lib_id "power:GND") (at 54.61 130.81 0) (unit 1)
+    (in_bom yes) (on_board yes) (fields_autoplaced)
+    (property "Reference" "#PWR0130" (id 0) (at 54.61 137.16 0)
+      (effects (font (size 1.27 1.27)) hide)
+    )
+    (property "Value" "GND" (id 1) (at 54.61 135.89 0))
+    (property "Footprint" "" (id 2) (at 54.61 130.81 0)
+      (effects (font (size 1.27 1.27)) hide)
+    )
+    (property "Datasheet" "" (id 3) (at 54.61 130.81 0)
+      (effects (font (size 1.27 1.27)) hide)
+    )
+    (pin "1")
   )
   (symbol (lib_id "karca_custom_components:MCP6N11R") (at 157.48 115.57 0) (unit 1)
@@
     (pin "7")
     (pin "8")
+    (pin "9")
   )
   (symbol (lib_id "power:GND") (at 151.13 63.5 0) (unit 1)

Commit message: preliminary layout and started pwr plane config
Parts:
- removed J14, J17, J18, J6: Conn_01x04_Female, karca_custom_footprints:LPTA-4pos, symbol Connector:Conn_01x04_Female
- removed J15: Conn_01x04_Female, Connector_PinHeader_2.54mm:PinHeader_1x04_P2.54mm_Vertical, symbol Connector:Conn_01x04_Female
- removed J16: Conn_01x08_Female, Connector_PinSocket_2.54mm:PinSocket_1x08_P2.54mm_Vertical, symbol Connector:Conn_01x08_Female
- added C7, C9: 1uF, Capacitor_SMD:C_1206_3216Metric, symbol Device:C
- added F12, F9: 3588-20, 3588-20:358820, symbol Device:Fuse
- added J13, J14, J15, J16, J17, J18: Screw_Terminal_01x04, 1190365:1190365, symbol Connector:Screw_Terminal_01x04
- added J19: Conn_01x06_Female, Connector_PinSocket_2.54mm:PinSocket_1x06_P2.54mm_Vertical, symbol Connector:Conn_01x06_Female
- added J20: Conn_02x06_Odd_Even, Connector_PinSocket_2.54mm:PinSocket_2x06_P2.54mm_Vertical, symbol Connector_Generic:Conn_02x06_Odd_Even
- added R32, R38: 20K, Resistor_SMD:R_1206_3216Metric, symbol Device:R_US
- added R35, R41: 200, Resistor_SMD:R_1206_3216Metric, symbol Device:R_US
- added RV3, RV6: 30k, 3296W-1-303LF:TRIM_3296W-1-303LF, symbol Device:R_Potentiometer
- added U5, U8: MCP6N11T-001E, Package_DFN_QFN:TDFN-8-1EP_3x2mm_P0.5mm_EP1.80x1.65mm, symbol karca_custom_components:MCP6N11R
- F10: renamed from F8; footprint karca_custom_footprints:3588-20 fuse -> 3588-20:358820
- F11: renamed from F10; footprint karca_custom_footprints:3588-20 fuse -> 3588-20:358820
- F7: footprint karca_custom_footprints:3588-20 fuse -> 3588-20:358820
- F8: renamed from F9; footprint karca_custom_footprints:3588-20 fuse -> 3588-20:358820
- renumbered C6 to C10, C7 to C6, R34 to R31, R31 to R33, R35 to R34, R32 to R36, R36 to R37, R33 to R39, R37 to R40, RV3 to RV2, RV2 to RV4, RV4 to RV5, U5 to U4, U4 to U6, U6 to U7
Connections:
- net +5V: now also C7.1, C9.1, F12.1, F9.1, RV3.1, RV6.1, U5.7 (Vdd), U5.8 (EN/nCAL), U8.7 (Vdd), U8.8 (EN/nCAL)
- net GND: now also C7.2, C9.2, J13.4 (Pin_4), J14.4 (Pin_4), J15.4 (Pin_4), J16.4 (Pin_4), J17.4 (Pin_4), J18.4 (Pin_4), RV3.3, RV6.3, U5.4 (Vss), U5.9 (PAD), U8.4 (Vss), U8.9 (PAD)
- net LC1+: now also J13.3 (Pin_3), J20.1 (Pin_1)
- net LC1-: now also J13.2 (Pin_2), J20.2 (Pin_2)
- net LC1_PREC: now also J19.1 (Pin_1)
- net LC2+: now also J14.3 (Pin_3), J20.3 (Pin_3)
- net LC2-: now also J14.2 (Pin_2), J20.4 (Pin_4)
- net LC2_PREC: now also J19.2 (Pin_2)
- net LC3+: now also J15.3 (Pin_3), J20.5 (Pin_5), U5.3 (Vip); no longer U6.3 (Vip)
- net LC3-: now also J15.2 (Pin_2), J20.6 (Pin_6), U5.2 (Vim); no longer U6.2 (Vim)
- net LC3_PREC: now also J19.3 (Pin_3), R32.1, R35.2, U5.6 (Vout); no longer R36.1, R39.2, U6.6 (Vout)
- net LC4+: now also U6.3 (Vip), J16.3 (Pin_3), J20.7 (Pin_7); no longer U7.3 (Vip)
- net LC4-: now also U6.2 (Vim), J16.2 (Pin_2), J20.8 (Pin_8); no longer U7.2 (Vim)
- net LC4_PREC: now also R36.1, R39.2, U6.6 (Vout), J19.4 (Pin_4); no longer R37.1, R40.2, U7.6 (Vout)
- net at F7.2: now also J13.1 (Pin_1)
- net at F11.2: now also J17.1 (Pin_1)
- net at F10.2: now also J16.1 (Pin_1)
- net at F8.2: now also J14.1 (Pin_1)
- new net: R32.2, U5.1 (Vfg)
- new net: R35.1, RV3.2, U5.5 (Vref)
- new net: F12.2, J18.1 (Pin_1)
- new net: R38.2, U8.1 (Vfg)
- new net: R41.1, RV6.2, U8.5 (Vref)
- new net: F9.2, J15.1 (Pin_1)
- new net LC5+: J17.3 (Pin_3), J20.9 (Pin_9), U7.3 (Vip)
- new net LC5-: J17.2 (Pin_2), J20.10 (Pin_10), U7.2 (Vim)
- new net LC5_PREC: J19.5 (Pin_5), R37.1, R40.2, U7.6 (Vout)
- new net LC6+: J18.3 (Pin_3), J20.11 (Pin_11), U8.3 (Vip)
- new net LC6-: J18.2 (Pin_2), J20.12 (Pin_12), U8.2 (Vim)
- new net LC6_PREC: J19.6 (Pin_6), R38.1, R41.2, U8.6 (Vout)
Other:
- note added: "Inamp 5"
- note added: "Inamp 6"
- moved on the sheet: C5, C6, C8, F11, F7, F8, R30, R31, R33, R34, R37, R40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

Commit message: some minor schematic cleanup
Parts:
- C10, C5, C6, C7, C8, C9: value 1uF -> 1u
