File: lc_inamps.kicad_sch (KiCad schematic)
At the start: 39 parts, among them J13 Conn_01x02_Female, J19 Conn_01x06_Female, J20 Conn_02x06_Odd_Even, U3 MCP6N11, U4 MCP6N11, U5 MCP6N11, U6 MCP6N11, U7 MCP6N11, U8 MCP6N11

Commit message: mostly finished routing
Connections:
- net +10V is gone; now on net +5V: RV1.1, RV2.1, RV3.1, RV4.1, RV5.1, RV6.1
Changed lines of the file:
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@@
-    (pin "1")
-  )
-  (symbol (lib_id "power:+10V") (at 259.08 128.27 0) (unit 1)
-    (in_bom yes) (on_board yes) (fields_autoplaced)
-    (property "Reference" "#PWR0164" (id 0) (at 259.08 132.08 0)
-      (effects (font (size 1.27 1.27)) hide)
-    )
-    (property "Value" "+10V" (id 1) (at 259.08 123.19 0))
-    (property "Footprint" "" (id 2) (at 259.08 128.27 0)
-      (effects (font (size 1.27 1.27)) hide)
-    )
-    (property "Datasheet" "" (id 3) (at 259.08 128.27 0)
-      (effects (font (size 1.27 1.27)) hide)
-    )
     (pin "1")
   )
@@
     (pin "3")
     (pin "4")
+  )
+  (symbol (lib_id "power:+5V") (at 171.45 58.42 0) (unit 1)
+    (in_bom yes) (on_board yes)
+    (property "Reference" "#PWR0163" (id 0) (at 171.45 62.23 0)
+      (effects (font (size 1.27 1.27)) hide)
+    )
+    (property "Value" "+5V" (id 1) (at 171.45 54.61 0))
+    (property "Footprint" "" (id 2) (at 171.45 58.42 0)
+      (effects (font (size 1.27 1.27)) hide)
+    )
+    (property "Datasheet" "" (id 3) (at 171.45 58.42 0)
+      (effects (font (size 1.27 1.27)) hide)
+    )
+    (pin "1")
   )
   (symbol (lib_id "power:+5V") (at 212.09 118.11 0) (unit 1)
@@
     (pin "1")
   )
-  (symbol (lib_id "power:+10V") (at 82.55 57.15 0) (unit 1)
-    (in_bom yes) (on_board yes) (fields_autoplaced)
-    (property "Reference" "#PWR0167" (id 0) (at 82.55 60.96 0)
-      (effects (font (size 1.27 1.27)) hide)
-    )
-    (property "Value" "+10V" (id 1) (at 82.55 52.07 0))
-    (property "Footprint" "" (id 2) (at 82.55 57.15 0)
-      (effects (font (size 1.27 1.27)) hide)
-    )
-    (property "Datasheet" "" (id 3) (at 82.55 57.15 0)
-      (effects (font (size 1.27 1.27)) hide)
-    )
-    (pin "1")
-  )
   (symbol (lib_id "Device:R_US") (at 246.38 111.76 180) (unit 1)
     (in_bom yes) (on_board yes)
@@
     (pin "1")
     (pin "2")
+  )
+  (symbol (lib_id "power:+5V") (at 259.08 58.42 0) (unit 1)
+    (in_bom yes) (on_board yes)
+    (property "Reference" "#PWR0165" (id 0) (at 259.08 62.23 0)
+      (effects (font (size 1.27 1.27)) hide)
+    )
+    (property "Value" "+5V" (id 1) (at 259.08 54.61 0))
+    (property "Footprint" "" (id 2) (at 259.08 58.42 0)
+      (effects (font (size 1.27 1.27)) hide)
+    )
+    (property "Datasheet" "" (id 3) (at 259.08 58.42 0)
+      (effects (font (size 1.27 1.27)) hide)
+    )
+    (pin "1")
   )
   (symbol (lib_id "power:+5V") (at 240.03 114.3 0) (unit 1)
@@
     )
     (property "Datasheet" "" (id 3) (at 171.45 66.04 0)
-      (effects (font (size 1.27 1.27)) hide)
-    )
-    (pin "1")
-  )
-  (symbol (lib_id "power:+10V") (at 171.45 58.42 0) (unit 1)
-    (in_bom yes) (on_board yes) (fields_autoplaced)
-    (property "Reference" "#PWR0163" (id 0) (at 171.45 62.23 0)
-      (effects (font (size 1.27 1.27)) hide)
-    )
-    (property "Value" "+10V" (id 1) (at 171.45 53.34 0))
-    (property "Footprint" "" (id 2) (at 171.45 58.42 0)
-      (effects (font (size 1.27 1.27)) hide)
-    )
-    (property "Datasheet" "" (id 3) (at 171.45 58.42 0)
-      (effects (font (size 1.27 1.27)) hide)
-    )
-    (pin "1")
-  )
-  (symbol (lib_id "power:+10V") (at 171.45 128.27 0) (unit 1)
-    (in_bom yes) (on_board yes) (fields_autoplaced)
-    (property "Reference" "#PWR0162" (id 0) (at 171.45 132.08 0)
-      (effects (font (size 1.27 1.27)) hide)
-    )
-    (property "Value" "+10V" (id 1) (at 171.45 123.19 0))
-    (property "Footprint" "" (id 2) (at 171.45 128.27 0)
-      (effects (font (size 1.27 1.27)) hide)
-    )
-    (property "Datasheet" "" (id 3) (at 171.45 128.27 0)
       (effects (font (size 1.27 1.27)) hide)
     )
@@
     (pin "1")
     (pin "2")
-  )
-  (symbol (lib_id "power:+10V") (at 259.08 58.42 0) (unit 1)
-    (in_bom yes) (on_board yes) (fields_autoplaced)
-    (property "Reference" "#PWR0165" (id 0) (at 259.08 62.23 0)
-      (effects (font (size 1.27 1.27)) hide)
-    )
-    (property "Value" "+10V" (id 1) (at 259.08 53.34 0))
-    (property "Footprint" "" (id 2) (at 259.08 58.42 0)
-      (effects (font (size 1.27 1.27)) hide)
-    )
-    (property "Datasheet" "" (id 3) (at 259.08 58.42 0)
-      (effects (font (size 1.27 1.27)) hide)
-    )
-    (pin "1")
   )
   (symbol (lib_id "Device:R_US") (at 71.12 121.92 180) (unit 1)
@@
     (pin "1")
   )
+  (symbol (lib_id "power:+5V") (at 82.55 57.15 0) (unit 1)
+    (in_bom yes) (on_board yes)
+    (property "Reference" "#PWR0167" (id 0) (at 82.55 60.96 0)
+      (effects (font (size 1.27 1.27)) hide)
+    )
+    (property "Value" "+5V" (id 1) (at 82.55 53.34 0))
+    (property "Footprint" "" (id 2) (at 82.55 57.15 0)
+      (effects (font (size 1.27 1.27)) hide)
+    )
+    (property "Datasheet" "" (id 3) (at 82.55 57.15 0)
+      (effects (font (size 1.27 1.27)) hide)
+    )
+    (pin "1")
+  )
   (symbol (lib_name "MCP6N11R_3") (lib_id "karca_custom_components:MCP6N11R") (at 53.34 53.34 0) (unit 1)
     (in_bom yes) (on_board yes)
@@
     (pin "8")
   )
+  (symbol (lib_id "power:+5V") (at 83.82 128.27 0) (unit 1)
+    (in_bom yes) (on_board yes)
+    (property "Reference" "#PWR0166" (id 0) (at 83.82 132.08 0)
+      (effects (font (size 1.27 1.27)) hide)
+    )
+    (property "Value" "+5V" (id 1) (at 83.82 124.46 0))
+    (property "Footprint" "" (id 2) (at 83.82 128.27 0)
+      (effects (font (size 1.27 1.27)) hide)
+    )
+    (property "Datasheet" "" (id 3) (at 83.82 128.27 0)
+      (effects (font (size 1.27 1.27)) hide)
+    )
+    (pin "1")
+  )
+  (symbol (lib_id "power:+5V") (at 259.08 128.27 0) (unit 1)
+    (in_bom yes) (on_board yes)
+    (property "Reference" "#PWR0164" (id 0) (at 259.08 132.08 0)
+      (effects (font (size 1.27 1.27)) hide)
+    )
+    (property "Value" "+5V" (id 1) (at 259.08 124.46 0))
+    (property "Footprint" "" (id 2) (at 259.08 128.27 0)
+      (effects (font (size 1.27 1.27)) hide)
+    )
+    (property "Datasheet" "" (id 3) (at 259.08 128.27 0)
+      (effects (font (size 1.27 1.27)) hide)
+    )
+    (pin "1")
+  )
   (symbol (lib_id "Connector:Screw_Terminal_01x04") (at 118.11 52.07 0) (mirror y) (unit 1)
     (in_bom yes) (on_board yes)
@@
     (pin "1")
   )
+  (symbol (lib_id "power:+5V") (at 171.45 128.27 0) (unit 1)
+    (in_bom yes) (on_board yes)
+    (property "Reference" "#PWR0162" (id 0) (at 171.45 132.08 0)
+      (effects (font (size 1.27 1.27)) hide)
+    )
+    (property "Value" "+5V" (id 1) (at 171.45 124.46 0))
+    (property "Footprint" "" (id 2) (at 171.45 128.27 0)
+      (effects (font (size 1.27 1.27)) hide)
+    )
+    (property "Datasheet" "" (id 3) (at 171.45 128.27 0)
+      (effects (font (size 1.27 1.27)) hide)
+    )
+    (pin "1")
+  )
   (symbol (lib_id "power:GND") (at 259.08 135.89 0) (unit 1)
     (in_bom yes) (on_board yes) (fields_autoplaced)
@@
     (pin "2")
   )
-  (symbol (lib_id "power:+10V") (at 83.82 128.27 0) (unit 1)
-    (in_bom yes) (on_board yes) (fields_autoplaced)
-    (property "Reference" "#PWR0166" (id 0) (at 83.82 132.08 0)
-      (effects (font (size 1.27 1.27)) hide)
-    )
-    (property "Value" "+10V" (id 1) (at 83.82 123.19 0))
-    (property "Footprint" "" (id 2) (at 83.82 128.27 0)
-      (effects (font (size 1.27 1.27)) hide)
-    )
-    (property "Datasheet" "" (id 3) (at 83.82 128.27 0)
-      (effects (font (size 1.27 1.27)) hide)
-    )
-    (pin "1")
-  )
   (symbol (lib_id "power:+5V") (at 64.77 114.3 0) (unit 1)
