File: lc_inamps.kicad_sch (KiCad schematic)
At the start: 39 parts, among them J13 Conn_01x02_Female, J19 Conn_01x06_Female, J20 Conn_02x06_Odd_Even, U3 MCP6N11, U4 MCP6N11, U5 MCP6N11, U6 MCP6N11, U7 MCP6N11, U8 MCP6N11

Commit message: not sure if anything has changed but this is the last commit before moving to two LCs
Parts:
- J13: footprint Connector_PinHeader_2.54mm:PinHeader_1x02_P2.54mm_Vertical -> Connector_PinSocket_2.54mm:PinSocket_1x02_P2.54mm_Vertical
- J19: footprint Connector_PinSocket_2.54mm:PinSocket_1x06_P2.54mm_Vertical -> Connector_PinSocket_2.54mm:PinSocket_1x04_P2.54mm_Vertical
Changed lines of the file:
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@@
       (effects (font (size 1.27 1.27)) (justify left) hide)
     )
-    (property "Footprint" "Connector_PinSocket_2.54mm:PinSocket_1x06_P2.54mm_Vertical" (id 2) (at 71.12 167.64 0)
+    (property "Footprint" "Connector_PinSocket_2.54mm:PinSocket_1x04_P2.54mm_Vertical" (id 2) (at 71.12 167.64 0)
       (effects (font (size 1.27 1.27)) hide)
     )
@@
       (effects (font (size 1.27 1.27)) (justify left))
     )
-    (property "Footprint" "Connector_PinHeader_2.54mm:PinHeader_1x02_P2.54mm_Vertical" (id 2) (at 71.12 179.07 0)
-      (effects (font (size 1.27 1.27)) hide)
-    )
+    (property "Footprint" "Connector_PinSocket_2.54mm:PinSocket_1x02_P2.54mm_Vertical" (id 2) (at 71.12 179.07 0)
+      (effects (font (size 1.27 1.27)) hide)
+    )

Commit message: enshrinkening of the board
Parts:
- removed C8, C9: 1u, Capacitor_SMD:C_1206_3216Metric, symbol Device:C
- removed CON_LC5, CON_LC6: Screw_Terminal_01x04, 1190365:1190365, symbol Connector:Screw_Terminal_01x04
- removed J13: Conn_01x02_Female, Connector_PinSocket_2.54mm:PinSocket_1x02_P2.54mm_Vertical, symbol Connector:Conn_01x02_Female
- removed R37, R38: 20K, Resistor_SMD:R_1206_3216Metric, symbol Device:R_US
- removed R40, R41: 200, Resistor_SMD:R_1206_3216Metric, symbol Device:R_US
- removed RV5, RV6: 30k, Potentiometer_THT:Potentiometer_Bourns_3296W_Vertical, symbol Device:R_Potentiometer
- removed U7, U8: MCP6N11, Package_SO:SOIC-8_3.9x4.9mm_P1.27mm, symbol karca_custom_components:MCP6N11R
- J20: footprint Connector_PinSocket_2.54mm:PinSocket_2x06_P2.54mm_Vertical -> Connector_PinSocket_2.54mm:PinSocket_2x04_P2.54mm_Vertical; symbol Connector_Generic:Conn_02x06_Odd_Even -> Connector_Generic:Conn_02x04_Odd_Even
Connections:
- removed net LC5+: J20.9 (Pin_9)
- removed net LC5-: J20.10 (Pin_10)
- removed net LC6+: J20.11 (Pin_11)
- removed net LC6-: J20.12 (Pin_12)
Other:
- note removed: "Inamp 5"
- note removed: "Inamp 6"

Commit message: done schematiccing after design review
Parts:
- removed CON_LC1, CON_LC2, CON_LC3, CON_LC4: Screw_Terminal_01x04, 1190365:1190365, symbol Connector:Screw_Terminal_01x04
- removed J19: Conn_01x06_Female, Connector_PinSocket_2.54mm:PinSocket_1x04_P2.54mm_Vertical, symbol Connector:Conn_01x04_Female
- removed J20: Conn_02x06_Odd_Even, Connector_PinSocket_2.54mm:PinSocket_2x04_P2.54mm_Vertical, symbol Connector_Generic:Conn_02x04_Odd_Even
- added ADC1: MCP3208-CI/SL, Package_SO:SOIC-16_3.9x9.9mm_P1.27mm, symbol Analog_ADC:MCP3208
- added C11, C12, C14, C15, C16, C17, C8, C9: 1n, Capacitor_SMD:C_1206_3216Metric, symbol Device:C
- added C13, C18: 100n, Capacitor_SMD:C_1206_3216Metric, symbol Device:C
- added D14, D15, D17, D18, D19, D20, D21, D22, D23, D24, D25, D26, D27, D28, D29, D30, D31, D32, D33, D9: CDBA340-HF, Diode_SMD:D_SMA, symbol Device:D_Schottky
- added J3, J4: Screw_Terminal_01x08, symbol Connector:Screw_Terminal_01x08
- added J5: Conn_01x08_Female, Connector_PinSocket_2.54mm:PinSocket_1x08_P2.54mm_Vertical, symbol Connector:Conn_01x08_Female
- added R37, R38, R40, R41, R42, R43, R44, R45: 68k, Resistor_SMD:R_1206_3216Metric, symbol Device:R_US
- added R46, R48, R50, R52: 15k, Resistor_SMD:R_1206_3216Metric, symbol Device:R_US
- added R47, R49, R51, R53: 10k, Resistor_SMD:R_1206_3216Metric, symbol Device:R_US
- added TP12: LC1-, symbol Connector:TestPoint
- added TP13: LC1+, symbol Connector:TestPoint
- added TP14: LC2+, symbol Connector:TestPoint
- added TP15: LC2-, symbol Connector:TestPoint
- added TP16, TP17, TP18, TP19: TestPoint, symbol Connector:TestPoint
- added TP20: LC1_PREC, symbol Connector:TestPoint
- added TP21: LC2_PREC, symbol Connector:TestPoint
- added TP22: LC3_PREC, symbol Connector:TestPoint
- added TP23: LC4_PREC, symbol Connector:TestPoint
- added U7, U9: LM324DT, Package_SO:SOIC-14_3.9x8.7mm_P1.27mm, symbol Amplifier_Operational:LM324
Connections:
- net +5V: now also ADC1.15 (Vref), ADC1.16 (Vdd), C18.2, D15.1 (K), D18.1 (K), D20.1 (K), D22.1 (K), D24.1 (K), D26.1 (K), D28.1 (K), D30.1 (K), D31.1 (K), D32.1 (K), D33.1 (K), D9.1 (K), J3.1 (Pin_1), J3.5 (Pin_5), J4.1 (Pin_1), J4.5 (Pin_5)
- net GND: now also ADC1.14 (AGND), ADC1.9 (DGND), C11.2, C12.2, C13.2, C18.1, C8.2, C9.2, D14.2 (A), D17.2 (A), D19.2 (A), D21.2 (A), D23.2 (A), D25.2 (A), D27.2 (A), D29.2 (A), J3.4 (Pin_4), J3.8 (Pin_8), J4.4 (Pin_4), J4.8 (Pin_8), R47.2, R49.2, R51.2, R53.2, U9.11 (V-)
- net LC1+: now also D22.2 (A), D23.1 (K), J3.3 (Pin_3), TP13.1
- net LC1-: now also D14.1 (K), D9.2 (A), J3.2 (Pin_2), TP12.1
- net LC1_PREC: now also R37.1, TP20.1
- net LC2+: now also D24.2 (A), D25.1 (K), J3.7 (Pin_7), TP15.1
- net LC2-: now also D15.2 (A), D17.1 (K), J3.6 (Pin_6), TP14.1
- net LC2_PREC: now also R38.1, TP21.1
- net LC3+: now also D26.2 (A), D27.1 (K), J4.3 (Pin_3), TP17.1
- net LC3-: now also D18.2 (A), D19.1 (K), J4.2 (Pin_2), TP16.1
- net LC3_PREC: now also R40.1, TP22.1
- net LC4+: now also D28.2 (A), D29.1 (K), J4.7 (Pin_7), TP19.1
- net LC4-: now also D20.2 (A), D21.1 (K), J4.6 (Pin_6), TP18.1
- net LC4_PREC: now also R41.1, TP23.1
- new net: ADC1.1 (CH0), C14.2, D30.2 (A), J5.1 (Pin_1), R46.1, U7.1
- new net: ADC1.2 (CH1), C15.2, D31.2 (A), J5.2 (Pin_2), R48.1, U7.7
- new net: ADC1.3 (CH2), C16.2, D32.2 (A), J5.3 (Pin_3), R50.1, U7.14
- new net: ADC1.4 (CH3), C17.2, D33.2 (A), J5.4 (Pin_4), R52.1, U7.8
- new net: ADC1.5 (CH4), J5.5 (Pin_5)
- new net: ADC1.6 (CH5), J5.6 (Pin_6)
- new net: ADC1.7 (CH6), J5.7 (Pin_7)
- new net: ADC1.8 (CH7), J5.8 (Pin_8)
- new net: C9.1, R43.2, U7.5 (+)
- new net: R48.2, R49.1, U7.6 (-)
- new net: R52.2, R53.1, U7.9 (-)
- new net: C15.1, R38.2, R43.1
- new net: R46.2, R47.1, U7.2 (-)
- new net: C8.1, R42.2, U7.3 (+)
- new net: C14.1, R37.2, R42.1
- new net: R50.2, R51.1, U7.13 (-)
- new net: C16.1, R40.2, R44.1
- new net: C11.1, R44.2, U7.12 (+)
- new net: C17.1, R41.2, R45.1
- new net: C12.1, R45.2, U7.10 (+)
- new net +10V: C13.1, U9.4 (V+)
- new net CS: ADC1.10 (~{CS}/SHDN)
- new net SPI_CLK: ADC1.13 (CLK)
- new net SPI_MISO: ADC1.12 (Dout)
- new net SPI_MOSI: ADC1.11 (Din)
Other:
- note added: "Anti-aliasing"
- note added: "Instrumentation amps"
- note removed: "Inamp 1"
- note removed: "Inamp 2"
- note removed: "Inamp 3"
- note removed: "Inamp 4"
- title: Load Cell InAmps -> Load Cells
- moved on the sheet: C10, C5, C6, C7, R30, R31, R32, R33, R34, R35, R36, R39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

Commit message: cleaned up PT footprint
Parts:
- J3, J4: footprint (none) -> 1190370:1190370
- TP12: value LC1- -> TestPoint; footprint (none) -> TestPoint:TestPoint_Pad_D2.0mm
- TP13: value LC1+ -> TestPoint; footprint (none) -> TestPoint:TestPoint_Pad_D2.0mm
- TP14: value LC2+ -> TestPoint; footprint (none) -> TestPoint:TestPoint_Pad_D2.0mm
- TP15: value LC2- -> TestPoint; footprint (none) -> TestPoint:TestPoint_Pad_D2.0mm
- TP16, TP17, TP18, TP19: footprint (none) -> TestPoint:TestPoint_Pad_D2.0mm
- TP20: value LC1_PREC -> TestPoint; footprint (none) -> TestPoint:TestPoint_Pad_D2.0mm
- TP21: value LC2_PREC -> TestPoint; footprint (none) -> TestPoint:TestPoint_Pad_D2.0mm
- TP22: value LC3_PREC -> TestPoint; footprint (none) -> TestPoint:TestPoint_Pad_D2.0mm
- TP23: value LC4_PREC -> TestPoint; footprint (none) -> TestPoint:TestPoint_Pad_D2.0mm
- renumbered U9 to U7
Connections:
- net LC1_CAL: now reaches ADC1.1 (CH0), C14.2, D30.2 (A), J5.1 (Pin_1), R46.1, U7.1
- net LC2_CAL: now reaches ADC1.2 (CH1), C15.2, D31.2 (A), J5.2 (Pin_2), R48.1, U7.7
- net LC3_CAL: now reaches ADC1.3 (CH2), C16.2, D32.2 (A), J5.3 (Pin_3), R50.1, U7.14
- net LC4_CAL: now reaches ADC1.4 (CH3), C17.2, D33.2 (A), J5.4 (Pin_4), R52.1, U7.8
Changed lines of the file:
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@@
+    (effects (font (size 1.27 1.27)) (justify left bottom))
+  )
+  (label "LC3_CAL" (at 205.74 95.885 0)
     (effects (font (size 1.27 1.27)) (justify left bottom))
   )
@@
     (effects (font (size 1.27 1.27)) (justify left bottom))
   )
+  (label "LC4_CAL" (at 205.74 98.425 0)
+    (effects (font (size 1.27 1.27)) (justify left bottom))
+  )
   (label "LC3-" (at 64.77 113.03 0)
     (effects (font (size 1.27 1.27)) (justify left bottom))
   )
+  (label "LC2_CAL" (at 205.74 93.345 0)
+    (effects (font (size 1.27 1.27)) (justify left bottom))
+  )
   (label "LC1_PREC" (at 107.315 27.305 0)
     (effects (font (size 1.27 1.27)) (justify left bottom))
@@
   )
   (label "LC4_PREC" (at 107.95 145.415 0)
+    (effects (font (size 1.27 1.27)) (justify left bottom))
+  )
+  (label "LC1_CAL" (at 205.74 90.805 0)
     (effects (font (size 1.27 1.27)) (justify left bottom))
   )
@@
       (effects (font (size 1.27 1.27)) (justify left) hide)
     )
-    (property "Footprint" "" (id 2) (at 50.165 153.035 0)
+    (property "Footprint" "TestPoint:TestPoint_Pad_D2.0mm" (id 2) (at 50.165 153.035 0)
       (effects (font (size 1.27 1.27)) hide)
     )
@@
       (effects (font (size 1.27 1.27)) hide)
     )
-    (property "Footprint" "" (id 2) (at 18.415 118.11 0)
+    (property "Footprint" "1190370:1190370" (id 2) (at 18.415 118.11 0)
       (effects (font (size 1.27 1.27)) hide)
     )
@@
       (effects (font (size 1.27 1.27)) (justify left))
     )
-    (property "Value" "LC2_PREC" (id 1) (at 107.95 62.7379 0)
-      (effects (font (size 1.27 1.27)) (justify left) hide)
-    )
-    (property "Footprint" "" (id 2) (at 110.49 64.77 0)
+    (property "Value" "TestPoint" (id 1) (at 107.95 62.7379 0)
+      (effects (font (size 1.27 1.27)) (justify left) hide)
+    )
+    (property "Footprint" "TestPoint:TestPoint_Pad_D2.0mm" (id 2) (at 110.49 64.77 0)
       (effects (font (size 1.27 1.27)) hide)
     )
@@
       (effects (font (size 1.27 1.27)) (justify left))
     )
-    (property "Value" "LC2+" (id 1) (at 47.625 67.8179 0)
-      (effects (font (size 1.27 1.27)) (justify left) hide)
-    )
-    (property "Footprint" "" (id 2) (at 50.165 69.85 0)
+    (property "Value" "TestPoint" (id 1) (at 47.625 67.8179 0)
+      (effects (font (size 1.27 1.27)) (justify left) hide)
+    )
+    (property "Footprint" "TestPoint:TestPoint_Pad_D2.0mm" (id 2) (at 50.165 69.85 0)
       (effects (font (size 1.27 1.27)) hide)
     )
@@
       (effects (font (size 1.27 1.27)) (justify left))
     )
-    (property "Value" "LC1_PREC" (id 1) (at 107.95 25.2729 0)
-      (effects (font (size 1.27 1.27)) (justify left) hide)
-    )
-    (property "Footprint" "" (id 2) (at 110.49 27.305 0)
+    (property "Value" "TestPoint" (id 1) (at 107.95 25.2729 0)
+      (effects (font (size 1.27 1.27)) (justify left) hide)
+    )
+    (property "Footprint" "TestPoint:TestPoint_Pad_D2.0mm" (id 2) (at 110.49 27.305 0)
       (effects (font (size 1.27 1.27)) hide)
     )
@@
       (effects (font (size 1.27 1.27)) (justify left) hide)
     )
-    (property "Footprint" "" (id 2) (at 50.165 113.03 0)
+    (property "Footprint" "TestPoint:TestPoint_Pad_D2.0mm" (id 2) (at 50.165 113.03 0)
       (effects (font (size 1.27 1.27)) hide)
     )
@@
       (effects (font (size 1.27 1.27)) (justify left))
     )
-    (property "Value" "LC4_PREC" (id 1) (at 107.95 143.3829 0)
-      (effects (font (size 1.27 1.27)) (justify left) hide)
-    )
-    (property "Footprint" "" (id 2) (at 110.49 145.415 0)
+    (property "Value" "TestPoint" (id 1) (at 107.95 143.3829 0)
+      (effects (font (size 1.27 1.27)) (justify left) hide)
+    )
+    (property "Footprint" "TestPoint:TestPoint_Pad_D2.0mm" (id 2) (at 110.49 145.415 0)
       (effects (font (size 1.27 1.27)) hide)
     )
@@
   (symbol (lib_id "Amplifier_Operational:LM324") (at 160.655 173.99 0) (unit 5)
     (in_bom yes) (on_board yes) (fields_autoplaced)
-    (property "Reference" "U9" (id 0) (at 159.385 172.7199 0)
-      (effects (font (size 1.27 1.27)) (justify left))
-    )
-    (property "Value" "LM324DT" (id 1) (at 159.385 175.2599 0)
+    (property "Reference" "U7" (id 0) (at 158.75 172.7199 0)
+      (effects (font (size 1.27 1.27)) (justify left))
+    )
+    (property "Value" "LM324DT" (id 1) (at 158.75 175.2599 0)
       (effects (font (size 1.27 1.27)) (justify left))
     )
@@
       (effects (font (size 1.27 1.27)) (justify left) hide)
     )
-    (property "Footprint" "" (id 2) (at 50.165 115.57 0)
+    (property "Footprint" "TestPoint:TestPoint_Pad_D2.0mm" (id 2) (at 50.165 115.57 0)
       (effects (font (size 1.27 1.27)) hide)
     )
@@
       (effects (font (size 1.27 1.27)) (justify left))
     )
-    (property "Value" "LC2-" (id 1) (at 47.625 74.4221 0)
-      (effects (font (size 1.27 1.27)) (justify left) hide)
-    )
-    (property "Footprint" "" (id 2) (at 50.165 72.39 0)
+    (property "Value" "TestPoint" (id 1) (at 47.625 74.4221 0)
+      (effects (font (size 1.27 1.27)) (justify left) hide)
+    )
+    (property "Footprint" "TestPoint:TestPoint_Pad_D2.0mm" (id 2) (at 50.165 72.39 0)
       (effects (font (size 1.27 1.27)) hide)
     )
@@
       (effects (font (size 1.27 1.27)) (justify left))
     )
-    (property "Value" "LC1+" (id 1) (at 47.625 36.9571 0)
-      (effects (font (size 1.27 1.27)) (justify left) hide)
-    )
-    (property "Footprint" "" (id 2) (at 50.165 34.925 0)
+    (property "Value" "TestPoint" (id 1) (at 47.625 36.9571 0)
+      (effects (font (size 1.27 1.27)) (justify left) hide)
+    )
+    (property "Footprint" "TestPoint:TestPoint_Pad_D2.0mm" (id 2) (at 50.165 34.925 0)
       (effects (font (size 1.27 1.27)) hide)
     )
@@
       (effects (font (size 1.27 1.27)) (justify left) hide)
     )
-    (property "Footprint" "" (id 2) (at 50.165 150.495 0)
+    (property "Footprint" "TestPoint:TestPoint_Pad_D2.0mm" (id 2) (at 50.165 150.495 0)
       (effects (font (size 1.27 1.27)) hide)
     )
@@
       (effects (font (size 1.27 1.27)) (justify left))
     )
-    (property "Value" "LC3_PREC" (id 1) (at 107.95 105.9179 0)
-      (effects (font (size 1.27 1.27)) (justify left) hide)
-    )
-    (property "Footprint" "" (id 2) (at 110.49 107.95 0)
+    (property "Value" "TestPoint" (id 1) (at 107.95 105.9179 0)
+      (effects (font (size 1.27 1.27)) (justify left) hide)
+    )
+    (property "Footprint" "TestPoint:TestPoint_Pad_D2.0mm" (id 2) (at 110.49 107.95 0)
       (effects (font (size 1.27 1.27)) hide)
     )
@@
       (effects (font (size 1.27 1.27)) hide)
     )
-    (property "Footprint" "" (id 2) (at 18.415 37.465 0)
+    (property "Footprint" "1190370:1190370" (id 2) (at 18.415 37.465 0)
       (effects (font (size 1.27 1.27)) hide)
     )
@@
       (effects (font (size 1.27 1.27)) (justify left))
     )
-    (property "Value" "LC1-" (id 1) (at 47.625 30.3529 0)
-      (effects (font (size 1.27 1.27)) (justify left) hide)
-    )
-    (property "Footprint" "" (id 2) (at 50.165 32.385 0)
-      (effects (font (size 1.27 1.27)) hide)
-    )
+    (property "Value" "TestPoint" (id 1) (at 47.625 30.3529 0)
+      (effects (font (size 1.27 1.27)) (justify left) hide)
+    )
+    (property "Footprint" "TestPoint:TestPoint_Pad_D2.0mm" (id 2) (at 50.165 32.385 0)
+      (effects (font (size 1.27 1.27)) hide)
+    )

Commit message: waiting on mouser for footprints
Connections:
- net LC3_CAL: now also U7.8; no longer U7.14
- net LC4_CAL: now also U7.14; no longer U7.8
- net at R52.2, R53.1: now also U7.13 (-); no longer U7.9 (-)
- net at R50.2, R51.1: now also U7.9 (-); no longer U7.13 (-)
- net at C11.1, R44.2: now also U7.10 (+); no longer U7.12 (+)
- net at C12.1, R45.2: now also U7.12 (+); no longer U7.10 (+)
Other:
- moved on the sheet: U7C, U7D
Changed lines of the file:
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@@
     (pin "1")
   )
-  (symbol (lib_id "Amplifier_Operational:LM324") (at 160.02 147.955 0) (unit 3)
-    (in_bom yes) (on_board yes) (fields_autoplaced)
-    (property "Reference" "U7" (id 0) (at 160.02 137.795 0))
-    (property "Value" "LM324DT" (id 1) (at 160.02 140.335 0))
-    (property "Footprint" "Package_SO:SOIC-14_3.9x8.7mm_P1.27mm" (id 2) (at 158.75 145.415 0)
-      (effects (font (size 1.27 1.27)) hide)
-    )
-    (property "Datasheet" "http://www.ti.com/lit/ds/symlink/lm2902-n.pdf" (id 3) (at 161.29 142.875 0)
+  (symbol (lib_id "Amplifier_Operational:LM324") (at 160.02 110.49 0) (unit 3)
+    (in_bom yes) (on_board yes) (fields_autoplaced)
+    (property "Reference" "U7" (id 0) (at 160.02 100.33 0))
+    (property "Value" "LM324DT" (id 1) (at 160.02 102.87 0))
+    (property "Footprint" "Package_SO:SOIC-14_3.9x8.7mm_P1.27mm" (id 2) (at 158.75 107.95 0)
+      (effects (font (size 1.27 1.27)) hide)
+    )
+    (property "Datasheet" "http://www.ti.com/lit/ds/symlink/lm2902-n.pdf" (id 3) (at 161.29 105.41 0)
       (effects (font (size 1.27 1.27)) hide)
     )
@@
     (pin "2")
   )
-  (symbol (lib_id "Amplifier_Operational:LM324") (at 160.02 110.49 0) (unit 4)
-    (in_bom yes) (on_board yes) (fields_autoplaced)
-    (property "Reference" "U7" (id 0) (at 160.02 100.33 0))
-    (property "Value" "LM324DT" (id 1) (at 160.02 102.87 0))
-    (property "Footprint" "Package_SO:SOIC-14_3.9x8.7mm_P1.27mm" (id 2) (at 158.75 107.95 0)
-      (effects (font (size 1.27 1.27)) hide)
-    )
-    (property "Datasheet" "http://www.ti.com/lit/ds/symlink/lm2902-n.pdf" (id 3) (at 161.29 105.41 0)
-      (effects (font (size 1.27 1.27)) hide)
-    )
+  (symbol (lib_id "Amplifier_Operational:LM324") (at 160.02 147.955 0) (unit 4)
+    (in_bom yes) (on_board yes) (fields_autoplaced)
+    (property "Reference" "U7" (id 0) (at 160.02 137.795 0))
+    (property "Value" "LM324DT" (id 1) (at 160.02 140.335 0))
+    (property "Footprint" "Package_SO:SOIC-14_3.9x8.7mm_P1.27mm" (id 2) (at 158.75 145.415 0)
+      (effects (font (size 1.27 1.27)) hide)
+    )
+    (property "Datasheet" "http://www.ti.com/lit/ds/symlink/lm2902-n.pdf" (id 3) (at 161.29 142.875 0)
+      (effects (font (size 1.27 1.27)) hide)
+    )

Commit message: possible fix for output impedance on load cell reference voltage; not yet in PCB
Parts:
- added C21: 100n, Capacitor_SMD:C_1206_3216Metric, symbol Device:C
- added U8: LM324, Package_SO:SOIC-14_3.9x8.7mm_P1.27mm, symbol Amplifier_Operational:LM324
Connections:
- net +5V: now also C21.1, U8.4 (V+)
- net GND: now also C21.2, U8.11 (V-)
- net LC3_REF: now reaches R35.1, U5.5 (Vref)
- net LC3_REF: now also U8.8, U8.9 (-); no longer RV3.2
- net LC4_REF: now reaches R39.1, U6.5 (Vref)
- net LC4_REF: now also U8.13 (-), U8.14; no longer RV4.2
- net LC2_REF: now reaches R34.1, U4.5 (Vref)
- net LC2_REF: now also U8.6 (-), U8.7; no longer RV2.2
- net LC1_REF: now reaches R33.1, U3.5 (Vref)
- net LC1_REF: now also U8.1, U8.2 (-); no longer RV1.2
- new net: RV4.2, U8.12 (+)
- new net: RV2.2, U8.5 (+)
- new net: RV1.2, U8.3 (+)
- new net: RV3.2, U8.10 (+)
Other:
- moved on the sheet: RV1, RV2, RV3, RV4

Commit message: started on opamp arrangement
Other:
- note added: "Reference voltage buffering"
Changed lines of the file:
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@@
+    (effects (font (size 1.27 1.27)) (justify left bottom))
+  )
+  (text "Reference voltage buffering" (at 95.885 196.215 0)
     (effects (font (size 1.27 1.27)) (justify left bottom))
   )

Commit message: my body is a machine that takes in peanut m&ms and puts out rocket engine controllers
Parts:
- ADC1: LCSC (none) -> C16939
- C10, C5, C6, C7: LCSC (none) -> C85867
- C11, C12, C14, C15, C16, C17, C8, C9: LCSC (none) -> C1845
- C13, C18, C21: LCSC (none) -> C377067
- D14, D15, D17, D18, D19, D20, D21, D22, D23, D24, D25, D26, D27, D28, D29, D30, D31, D32, D33, D9: LCSC (none) -> C14996
- R30, R31, R32, R36: LCSC (none) -> C114940
- R33, R34, R35, R39: LCSC (none) -> C114939
- R37, R38, R40, R41, R42, R43, R44, R45: LCSC (none) -> C102381
- R46, R48, R50, R52: LCSC (none) -> C1493
- R47, R49, R51, R53: LCSC (none) -> C132649
- U7: value LM324DT -> LM324; LCSC (none) -> C71035
- U8: LCSC (none) -> C71035
