File: pi.kicad_sch (KiCad schematic)
At the start: 0 parts

Commit message: first revision of full schematic copied over
Parts:
- added D?: HBT, symbol Device:LED
- added J?: 2540-5, symbol Connector_Generic:Conn_02x20_Odd_Even
- added R?: 150, symbol Device:R_US
Connections:
- new net: D?.2 (A), R?.1
- new net +5V: J?.2 (Pin_2), J?.4 (Pin_4)
- new net ADC1_CS: J?.22 (Pin_22)
- new net ADC2_CS: J?.24 (Pin_24)
- new net ADC3_CS: J?.26 (Pin_26)
- new net DRV_CTL_1: J?.11 (Pin_11)
- new net DRV_CTL_2: J?.13 (Pin_13)
- new net DRV_CTL_3: J?.15 (Pin_15)
- new net DRV_CTL_4: J?.18 (Pin_18)
- new net DRV_CTL_5: J?.33 (Pin_33)
- new net DRV_CTL_6: J?.32 (Pin_32)
- new net GND: D?.1 (K), J?.14 (Pin_14), J?.20 (Pin_20), J?.25 (Pin_25), J?.30 (Pin_30), J?.34 (Pin_34), J?.39 (Pin_39), J?.6 (Pin_6), J?.9 (Pin_9)
- new net HBT: J?.29 (Pin_29), R?.2
- new net SPI_CLK: J?.23 (Pin_23)
- new net SPI_MISO: J?.21 (Pin_21)
- new net SPI_MOSI: J?.19 (Pin_19)
- new net nc1: J?.1 (Pin_1)
- new net nc10: J?.10 (Pin_10)
- new net nc12: J?.12 (Pin_12)
- new net nc16: J?.16 (Pin_16)
- new net nc17: J?.17 (Pin_17)
- new net nc27: J?.27 (Pin_27)
- new net nc28: J?.28 (Pin_28)
- new net nc3: J?.3 (Pin_3)
- new net nc31: J?.31 (Pin_31)
- new net nc35: J?.35 (Pin_35)
- new net nc36: J?.36 (Pin_36)
- new net nc37: J?.37 (Pin_37)
- new net nc38: J?.38 (Pin_38)
- new net nc40: J?.40 (Pin_40)
- new net nc5: J?.5 (Pin_5)
- new net nc7: J?.7 (Pin_7)
- new net nc8: J?.8 (Pin_8)
- no-connect marks 0 -> 17
Other:
- company: (none) -> Rice Eclipse
- title: (none) -> Raspberry Pi Interface

Commit message: added schematic pdf for review
Parts:
- gave numbers to parts that had none: 3
Changed lines of the file:
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@@
   (symbol (lib_id "power:+5V") (at 121.92 62.23 0) (unit 1)
     (in_bom yes) (on_board yes) (fields_autoplaced)
-    (property "Reference" "#PWR?" (id 0) (at 121.92 66.04 0)
+    (property "Reference" "#PWR0127" (id 0) (at 121.92 66.04 0)
       (effects (font (size 1.27 1.27)) hide)
     )
@@
   (symbol (lib_id "power:GND") (at 68.58 110.49 0) (unit 1)
     (in_bom yes) (on_board yes) (fields_autoplaced)
-    (property "Reference" "#PWR?" (id 0) (at 68.58 116.84 0)
+    (property "Reference" "#PWR0126" (id 0) (at 68.58 116.84 0)
       (effects (font (size 1.27 1.27)) hide)
     )
@@
   (symbol (lib_id "Device:R_US") (at 82.55 97.79 90) (unit 1)
     (in_bom yes) (on_board yes)
-    (property "Reference" "R?" (id 0) (at 82.55 95.25 90))
+    (property "Reference" "R77" (id 0) (at 82.55 95.25 90))
     (property "Value" "150" (id 1) (at 82.55 100.33 90))
     (property "Footprint" "" (id 2) (at 82.804 96.774 90)
@@
   (symbol (lib_id "power:GND") (at 144.78 102.87 0) (unit 1)
     (in_bom yes) (on_board yes) (fields_autoplaced)
-    (property "Reference" "#PWR?" (id 0) (at 144.78 109.22 0)
+    (property "Reference" "#PWR0128" (id 0) (at 144.78 109.22 0)
       (effects (font (size 1.27 1.27)) hide)
     )
@@
   (symbol (lib_id "Connector_Generic:Conn_02x20_Odd_Even") (at 104.14 85.09 0) (unit 1)
     (in_bom yes) (on_board yes) (fields_autoplaced)
-    (property "Reference" "J?" (id 0) (at 105.41 55.88 0))
+    (property "Reference" "J36" (id 0) (at 105.41 55.88 0))
     (property "Value" "2540-5" (id 1) (at 105.41 58.42 0))
     (property "Footprint" "" (id 2) (at 104.14 85.09 0)
@@
   (symbol (lib_id "Device:LED") (at 73.66 97.79 0) (unit 1)
     (in_bom yes) (on_board yes)
-    (property "Reference" "D?" (id 0) (at 73.66 95.25 0))
+    (property "Reference" "D25" (id 0) (at 73.66 95.25 0))
     (property "Value" "HBT" (id 1) (at 73.66 100.33 0))
     (property "Footprint" "" (id 2) (at 73.66 97.79 0)

Commit message: added footprints and started schematic review revisions
Parts:
- D25: footprint (none) -> LED_SMD:LED_1206_3216Metric
- R77: footprint (none) -> Resistor_SMD:R_1206_3216Metric
Changed lines of the file:
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@@
     (property "Reference" "R77" (id 0) (at 82.55 95.25 90))
     (property "Value" "150" (id 1) (at 82.55 100.33 90))
-    (property "Footprint" "" (id 2) (at 82.804 96.774 90)
+    (property "Footprint" "Resistor_SMD:R_1206_3216Metric" (id 2) (at 82.804 96.774 90)
       (effects (font (size 1.27 1.27)) hide)
     )
@@
     (property "Reference" "D25" (id 0) (at 73.66 95.25 0))
     (property "Value" "HBT" (id 1) (at 73.66 100.33 0))
-    (property "Footprint" "" (id 2) (at 73.66 97.79 0)
+    (property "Footprint" "LED_SMD:LED_1206_3216Metric" (id 2) (at 73.66 97.79 0)
       (effects (font (size 1.27 1.27)) hide)
     )
-    (property "Datasheet" "~" (id 3) (at 73.66 97.79 0)
+    (property "Datasheet" "https://datasheet.lcsc.com/lcsc/1912111437_MEIHUA-MHT150UBCT_C404273.pdf" (id 3) (at 73.66 97.79 0)
       (effects (font (size 1.27 1.27)) hide)
     )

Commit message: schematic editing + creating some footprints
Connections:
- net nc1: no longer names the net of J36.1 (Pin_1)
- net nc10: no longer names the net of J36.10 (Pin_10)
- net nc12: no longer names the net of J36.12 (Pin_12)
- net nc16: no longer names the net of J36.16 (Pin_16)
- net nc17: no longer names the net of J36.17 (Pin_17)
- net nc27: no longer names the net of J36.27 (Pin_27)
- net nc28: no longer names the net of J36.28 (Pin_28)
- net nc3: no longer names the net of J36.3 (Pin_3)
- net nc31: no longer names the net of J36.31 (Pin_31)
- net nc35: no longer names the net of J36.35 (Pin_35)
- net nc36: no longer names the net of J36.36 (Pin_36)
- net nc37: no longer names the net of J36.37 (Pin_37)
- net nc38: no longer names the net of J36.38 (Pin_38)
- net nc40: no longer names the net of J36.40 (Pin_40)
- net nc5: no longer names the net of J36.5 (Pin_5)
- net nc7: no longer names the net of J36.7 (Pin_7)
- net nc8: no longer names the net of J36.8 (Pin_8)

Commit message: updated all footprints, resolved most ERC & setup layout
Parts:
- J36: footprint (none) -> Connector_PinHeader_2.54mm:PinHeader_2x20_P2.54mm_Horizontal
Changed lines of the file:
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@@
     (property "Reference" "J36" (id 0) (at 105.41 55.88 0))
     (property "Value" "2540-5" (id 1) (at 105.41 58.42 0))
-    (property "Footprint" "" (id 2) (at 104.14 85.09 0)
+    (property "Footprint" "Connector_PinHeader_2.54mm:PinHeader_2x20_P2.54mm_Horizontal" (id 2) (at 104.14 85.09 0)
       (effects (font (size 1.27 1.27)) hide)
     )

Commit message: preliminary layout and started pwr plane config
Parts:
- renumbered J36 to J33, R77 to R89
Changed lines of the file:
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@@
   (symbol (lib_id "power:+5V") (at 121.92 62.23 0) (unit 1)
     (in_bom yes) (on_board yes) (fields_autoplaced)
-    (property "Reference" "#PWR0127" (id 0) (at 121.92 66.04 0)
+    (property "Reference" "#PWR0152" (id 0) (at 121.92 66.04 0)
       (effects (font (size 1.27 1.27)) hide)
     )
@@
   (symbol (lib_id "power:GND") (at 68.58 110.49 0) (unit 1)
     (in_bom yes) (on_board yes) (fields_autoplaced)
-    (property "Reference" "#PWR0126" (id 0) (at 68.58 116.84 0)
+    (property "Reference" "#PWR0154" (id 0) (at 68.58 116.84 0)
       (effects (font (size 1.27 1.27)) hide)
     )
@@
   (symbol (lib_id "Device:R_US") (at 82.55 97.79 90) (unit 1)
     (in_bom yes) (on_board yes)
-    (property "Reference" "R77" (id 0) (at 82.55 95.25 90))
+    (property "Reference" "R89" (id 0) (at 82.55 95.25 90))
     (property "Value" "150" (id 1) (at 82.55 100.33 90))
     (property "Footprint" "Resistor_SMD:R_1206_3216Metric" (id 2) (at 82.804 96.774 90)
@@
   (symbol (lib_id "power:GND") (at 138.43 102.87 0) (unit 1)
     (in_bom yes) (on_board yes) (fields_autoplaced)
-    (property "Reference" "#PWR0128" (id 0) (at 138.43 109.22 0)
+    (property "Reference" "#PWR0153" (id 0) (at 138.43 109.22 0)
       (effects (font (size 1.27 1.27)) hide)
     )
@@
   (symbol (lib_id "Connector_Generic:Conn_02x20_Odd_Even") (at 104.14 85.09 0) (unit 1)
     (in_bom yes) (on_board yes) (fields_autoplaced)
-    (property "Reference" "J36" (id 0) (at 105.41 55.88 0))
+    (property "Reference" "J33" (id 0) (at 105.41 55.88 0))
     (property "Value" "2540-5" (id 1) (at 105.41 58.42 0))
     (property "Footprint" "Connector_PinHeader_2.54mm:PinHeader_2x20_P2.54mm_Horizontal" (id 2) (at 104.14 85.09 0)

Commit message: shuffle around some parts
Parts:
- HBT1: renamed from D25; value HBT -> BLU
Other:
- moved on the sheet: HBT1, R89
Changed lines of the file:
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@@
     (company "Rice Eclipse")
   )
-  (junction (at 68.58 92.71) (diameter 0) (color 0 0 0 0)
+  (junction (at 76.2 92.71) (diameter 0) (color 0 0 0 0)
   )
   (junction (at 127 97.79) (diameter 0) (color 0 0 0 0)
@@
   (junction (at 114.3 62.23) (diameter 0) (color 0 0 0 0)
   )
-  (junction (at 68.58 97.79) (diameter 0) (color 0 0 0 0)
+  (junction (at 76.2 97.79) (diameter 0) (color 0 0 0 0)
   )
   (junction (at 127 77.47) (diameter 0) (color 0 0 0 0)
   )
-  (junction (at 68.58 110.49) (diameter 0) (color 0 0 0 0)
+  (junction (at 76.2 110.49) (diameter 0) (color 0 0 0 0)
   )
   (junction (at 127 85.09) (diameter 0) (color 0 0 0 0)
@@
     (stroke (width 0) (type default) (color 0 0 0 0))
   )
-  (wire (pts (xy 68.58 110.49) (xy 68.58 111.76))
+  (wire (pts (xy 76.2 110.49) (xy 76.2 111.76))
     (stroke (width 0) (type default) (color 0 0 0 0))
   )
@@
     (stroke (width 0) (type default) (color 0 0 0 0))
   )
-  (wire (pts (xy 77.47 97.79) (xy 78.74 97.79))
-    (stroke (width 0) (type default) (color 0 0 0 0))
-  )
-  (wire (pts (xy 68.58 72.39) (xy 99.06 72.39))
-    (stroke (width 0) (type default) (color 0 0 0 0))
-  )
-  (wire (pts (xy 68.58 110.49) (xy 99.06 110.49))
+  (wire (pts (xy 76.2 72.39) (xy 99.06 72.39))
+    (stroke (width 0) (type default) (color 0 0 0 0))
+  )
+  (wire (pts (xy 76.2 110.49) (xy 99.06 110.49))
     (stroke (width 0) (type default) (color 0 0 0 0))
   )
@@
     (stroke (width 0) (type default) (color 0 0 0 0))
   )
-  (wire (pts (xy 68.58 97.79) (xy 69.85 97.79))
+  (wire (pts (xy 76.2 97.79) (xy 79.375 97.79))
     (stroke (width 0) (type default) (color 0 0 0 0))
   )
@@
     (stroke (width 0) (type default) (color 0 0 0 0))
   )
-  (wire (pts (xy 68.58 92.71) (xy 99.06 92.71))
-    (stroke (width 0) (type default) (color 0 0 0 0))
-  )
-  (wire (pts (xy 68.58 97.79) (xy 68.58 110.49))
+  (wire (pts (xy 76.2 92.71) (xy 99.06 92.71))
+    (stroke (width 0) (type default) (color 0 0 0 0))
+  )
+  (wire (pts (xy 76.2 97.79) (xy 76.2 110.49))
     (stroke (width 0) (type default) (color 0 0 0 0))
   )
@@
     (stroke (width 0) (type default) (color 0 0 0 0))
   )
-  (wire (pts (xy 86.36 97.79) (xy 99.06 97.79))
+  (wire (pts (xy 94.615 97.79) (xy 99.06 97.79))
     (stroke (width 0) (type default) (color 0 0 0 0))
   )
@@
     (stroke (width 0) (type default) (color 0 0 0 0))
   )
-  (wire (pts (xy 68.58 72.39) (xy 68.58 92.71))
-    (stroke (width 0) (type default) (color 0 0 0 0))
-  )
-  (wire (pts (xy 68.58 92.71) (xy 68.58 97.79))
+  (wire (pts (xy 76.2 72.39) (xy 76.2 92.71))
+    (stroke (width 0) (type default) (color 0 0 0 0))
+  )
+  (wire (pts (xy 76.2 92.71) (xy 76.2 97.79))
     (stroke (width 0) (type default) (color 0 0 0 0))
   )
@@
     (pin "1")
   )
-  (symbol (lib_id "power:GND") (at 68.58 110.49 0) (unit 1)
-    (in_bom yes) (on_board yes) (fields_autoplaced)
-    (property "Reference" "#PWR0154" (id 0) (at 68.58 116.84 0)
-      (effects (font (size 1.27 1.27)) hide)
-    )
-    (property "Value" "GND" (id 1) (at 68.58 115.57 0))
-    (property "Footprint" "" (id 2) (at 68.58 110.49 0)
-      (effects (font (size 1.27 1.27)) hide)
-    )
-    (property "Datasheet" "" (id 3) (at 68.58 110.49 0)
-      (effects (font (size 1.27 1.27)) hide)
-    )
-    (pin "1")
-  )
-  (symbol (lib_id "Device:R_US") (at 82.55 97.79 90) (unit 1)
+  (symbol (lib_id "power:GND") (at 76.2 110.49 0) (unit 1)
+    (in_bom yes) (on_board yes) (fields_autoplaced)
+    (property "Reference" "#PWR0154" (id 0) (at 76.2 116.84 0)
+      (effects (font (size 1.27 1.27)) hide)
+    )
+    (property "Value" "GND" (id 1) (at 76.2 115.57 0))
+    (property "Footprint" "" (id 2) (at 76.2 110.49 0)
+      (effects (font (size 1.27 1.27)) hide)
+    )
+    (property "Datasheet" "" (id 3) (at 76.2 110.49 0)
+      (effects (font (size 1.27 1.27)) hide)
+    )
+    (pin "1")
+  )
+  (symbol (lib_id "Device:R_US") (at 90.805 97.79 90) (unit 1)
     (in_bom yes) (on_board yes)
-    (property "Reference" "R89" (id 0) (at 82.55 95.25 90))
-    (property "Value" "150" (id 1) (at 82.55 100.33 90))
-    (property "Footprint" "Resistor_SMD:R_1206_3216Metric" (id 2) (at 82.804 96.774 90)
-      (effects (font (size 1.27 1.27)) hide)
-    )
-    (property "Datasheet" "~" (id 3) (at 82.55 97.79 0)
+    (property "Reference" "R89" (id 0) (at 90.805 95.25 90))
+    (property "Value" "150" (id 1) (at 90.805 100.33 90))
+    (property "Footprint" "Resistor_SMD:R_1206_3216Metric" (id 2) (at 91.059 96.774 90)
+      (effects (font (size 1.27 1.27)) hide)
+    )
+    (property "Datasheet" "~" (id 3) (at 90.805 97.79 0)
       (effects (font (size 1.27 1.27)) hide)
     )
@@
     (pin "9")
   )
-  (symbol (lib_id "Device:LED") (at 73.66 97.79 0) (unit 1)
+  (symbol (lib_id "Device:LED") (at 83.185 97.79 0) (unit 1)
     (in_bom yes) (on_board yes)
-    (property "Reference" "D25" (id 0) (at 73.66 95.25 0))
-    (property "Value" "HBT" (id 1) (at 73.66 100.33 0))
-    (property "Footprint" "LED_SMD:LED_1206_3216Metric" (id 2) (at 73.66 97.79 0)
-      (effects (font (size 1.27 1.27)) hide)
-    )
-    (property "Datasheet" "~" (id 3) (at 73.66 97.79 0)
-      (effects (font (size 1.27 1.27)) hide)
-    )
+    (property "Reference" "HBT1" (id 0) (at 83.185 95.25 0))
+    (property "Value" "BLU" (id 1) (at 83.185 100.33 0))
+    (property "Footprint" "LED_SMD:LED_1206_3216Metric" (id 2) (at 83.185 97.79 0)
+      (effects (font (size 1.27 1.27)) hide)
+    )
+    (property "Datasheet" "~" (id 3) (at 83.185 97.79 0)
+      (effects (font (size 1.27 1.27)) hide)
+    )
