File: karca.kicad_pcb (KiCad board)
At the start: 2 copper layers, 9 parts, among them U1 LM1084-ADJ

Commit message: schematic editing + creating some footprints
Parts:
- added C1: 10uF, Capacitor_SMD:C_1206_3216Metric, F.Cu at (132.1, -55.9)
- added C10: 1nF, Capacitor_SMD:C_1206_3216Metric, F.Cu at (175.4, -105.9)
- added C11: 1nF, Capacitor_SMD:C_1206_3216Metric, F.Cu at (183.9, -116.1)
- added C12: 1nF, Capacitor_SMD:C_1206_3216Metric, F.Cu at (183.9, -119.5)
- added C13: 1nF, Capacitor_SMD:C_1206_3216Metric, F.Cu at (175.4, -109.3)
- added C14: 1nF, Capacitor_SMD:C_1206_3216Metric, F.Cu at (181.1, -112.6)
- added C15: 1nF, Capacitor_SMD:C_1206_3216Metric, F.Cu at (181.1, -109.3)
- added C16: 1nF, Capacitor_SMD:C_1206_3216Metric, F.Cu at (175.4, -112.6)
- added C17: 1nF, Capacitor_SMD:C_1206_3216Metric, F.Cu at (189.5, -122.8)
- added C18: 1nF, Capacitor_SMD:C_1206_3216Metric, F.Cu at (122.0, -89.5)
- added C19: 1nF, Capacitor_SMD:C_1206_3216Metric, F.Cu at (152.9, -119.5)
- added C2: 10uF, Capacitor_SMD:C_1206_3216Metric, F.Cu at (132.1, -59.2)
- added C20: 1nF, Capacitor_SMD:C_1206_3216Metric, F.Cu at (149.2, -115.6)
- added C21: 1nF, Capacitor_SMD:C_1206_3216Metric, F.Cu at (125.6, -93.4)
- added C22: 100nF, Capacitor_SMD:C_1206_3216Metric, F.Cu at (143.6, -115.6)
- added C23: 1nF, Capacitor_SMD:C_1206_3216Metric, F.Cu at (125.6, -96.7)
- added C24: 1nF, Capacitor_SMD:C_1206_3216Metric, F.Cu at (143.6, -112.3)
- added C25: 1nF, Capacitor_SMD:C_1206_3216Metric, F.Cu at (152.9, -122.8)
- added C26: 1nF, Capacitor_SMD:C_1206_3216Metric, F.Cu at (116.3, -89.5)
- added C27: 100nF, Capacitor_SMD:C_1206_3216Metric, F.Cu at (149.6, -69.5)
- added C28: 100nF, Capacitor_SMD:C_1206_3216Metric, F.Cu at (155.2, -69.5)
- added C29: 100nF, Capacitor_SMD:C_1206_3216Metric, F.Cu at (149.6, -66.1)
- added C3: 10uF, Capacitor_SMD:C_1206_3216Metric, F.Cu at (109.3, -38.1)
- added C4: 10uF, Capacitor_SMD:C_1206_3216Metric, F.Cu at (116.7, -43.2)
- added C5: 1uF, Capacitor_SMD:C_1206_3216Metric, F.Cu at (-1.26, -14.2)
- added C6: 1uF, Capacitor_SMD:C_1206_3216Metric, F.Cu at (10.0, -17.5)
- added C7: 1uF, Capacitor_SMD:C_1206_3216Metric, F.Cu at (-1.26, -17.5)
- added C8: 1uF, Capacitor_SMD:C_1206_3216Metric, F.Cu at (4.39, -17.5)
- added C9: 100nF, Capacitor_SMD:C_1206_3216Metric, F.Cu at (183.9, -122.8)
- added D1: 1N5822RLG, Diode_THT:D_DO-201AD_P15.24mm_Horizontal, F.Cu at (94.0, -61.0)
- added D10: SS54, karca_custom_footprints:DO-214AC, F.Cu at (20.8, -84.2)
- added D11: FS_STAT_1, LED_SMD:LED_1206_3216Metric, F.Cu at (70.8, -109.8)
- added D12: FS_STAT_4, LED_SMD:LED_1206_3216Metric, F.Cu at (43.8, -82.3)
- added D13: DRV_STAT_2, LED_SMD:LED_1206_3216Metric, F.Cu at (70.8, -106.4)
- added D14: DRV_STAT_5, LED_SMD:LED_1206_3216Metric, F.Cu at (43.8, -78.9)
- added D15: SS54, karca_custom_footprints:DO-214AC, F.Cu at (28.1, -87.7)
- added D16: SS54, karca_custom_footprints:DO-214AC, F.Cu at (28.1, -84.2)
- added D17: FS_STAT_2, LED_SMD:LED_1206_3216Metric, F.Cu at (65.1, -109.8)
- added D18: FS_STAT_5, LED_SMD:LED_1206_3216Metric, F.Cu at (56.0, -93.3)
- added D19: DRV_STAT_3, LED_SMD:LED_1206_3216Metric, F.Cu at (39.1, -73.5)
- added D2: PWR_12V, LED_SMD:LED_1206_3216Metric, F.Cu at (126.1, -50.4)
- added D20: DRV_STAT_6, LED_SMD:LED_1206_3216Metric, F.Cu at (56.0, -96.7)
- added D21: SS54, karca_custom_footprints:DO-214AC, F.Cu at (20.8, -87.7)
- added D22: SS54, karca_custom_footprints:DO-214AC, F.Cu at (35.4, -87.7)
- added D23: FS_STAT_3, LED_SMD:LED_1206_3216Metric, F.Cu at (65.1, -103.0)
- added D24: FS_STAT_6, LED_SMD:LED_1206_3216Metric, F.Cu at (65.1, -106.4)
- added D25: HBT, LED_SMD:LED_1206_3216Metric, F.Cu at (-1.24, -7.62)
- added D3: SS54, karca_custom_footprints:DO-214AC, F.Cu at (131.0, -62.7)
- added D4: SS54, karca_custom_footprints:DO-214AC, F.Cu at (102.6, -43.6)
- added D5: PWR_5V, LED_SMD:LED_1206_3216Metric, F.Cu at (103.7, -40.1)
- added D6: PWR_10V, LED_SMD:LED_1206_3216Metric, F.Cu at (139.4, -62.7)
- added D7: DRV_STAT_1, LED_SMD:LED_1206_3216Metric, F.Cu at (65.1, -99.6)
- added D8: DRV_STAT_4, LED_SMD:LED_1206_3216Metric, F.Cu at (85.3, -122.8)
- added D9: SS54, karca_custom_footprints:DO-214AC, F.Cu at (35.4, -84.2)
- added F1: 3588-20, karca_custom_footprints:3588-20 fuse, F.Cu at (67.4, -113.5)
- added F10: 3588-20, karca_custom_footprints:3588-20 fuse, F.Cu at (63.1, -53.4)
- added F11: 3588-20, karca_custom_footprints:3588-20 fuse, F.Cu at (125.7, -113.5)
- added F12: 3588-20, karca_custom_footprints:3588-20 fuse, F.Cu at (125.7, -100.5)
- added F13: 3588-20, karca_custom_footprints:3588-20 fuse, F.Cu at (105.5, -100.5)
- added F14: 3588-20, karca_custom_footprints:3588-20 fuse, F.Cu at (105.5, -113.5)
- added F15: 3588-20, karca_custom_footprints:3588-20 fuse, F.Cu at (116.9, -21.1)
- added F16: 3588-20, karca_custom_footprints:3588-20 fuse, F.Cu at (116.9, -8.05)
- added F17: 3588-20, karca_custom_footprints:3588-20 fuse, F.Cu at (96.7, -21.1)
- added F18: 3588-20, karca_custom_footprints:3588-20 fuse, F.Cu at (96.7, -8.05)
- added F2: 3588-20, karca_custom_footprints:3588-20 fuse, F.Cu at (47.3, -113.5)
- added F3: 3588-20, karca_custom_footprints:3588-20 fuse, F.Cu at (21.2, -69.5)
- added F4: 3588-20, karca_custom_footprints:3588-20 fuse, F.Cu at (24.2, -91.5)
- added F5: 3588-20, karca_custom_footprints:3588-20 fuse, F.Cu at (47.3, -100.5)
- added F6: 3588-20, karca_custom_footprints:3588-20 fuse, F.Cu at (1.05, -69.5)
- added F7: 3588-20, karca_custom_footprints:3588-20 fuse, F.Cu at (21.7, -17.8)
- added F8: 3588-20, karca_custom_footprints:3588-20 fuse, F.Cu at (21.7, -30.8)
- added F9: 3588-20, karca_custom_footprints:3588-20 fuse, F.Cu at (41.9, -30.8)
- added J1: Conn_01x02_Female, Connector_PinHeader_2.54mm:PinHeader_1x02_P2.54mm_Vertical, F.Cu at (120.9, -49.8)
- added J10: Conn_01x02_Female, Connector_PinHeader_2.54mm:PinHeader_1x02_P2.54mm_Vertical, F.Cu at (43.3, -88.9)
- added J11: Conn_01x02_Female, Connector_PinHeader_2.54mm:PinHeader_1x02_P2.54mm_Vertical, F.Cu at (50.8, -96.1)
- added J12: Conn_01x02_Female, Connector_PinHeader_2.54mm:PinHeader_1x02_P2.54mm_Vertical, F.Cu at (38.6, -80.1)
- added J13: Conn_01x02_Female, Connector_PinHeader_2.54mm:PinHeader_1x02_P2.54mm_Vertical, F.Cu at (48.0, -88.9)
- added J14: Conn_01x04_Female, karca_custom_footprints:LPTA-4pos, F.Cu at (3.98, -30.5)
- added J15: Conn_01x04_Female, Connector_PinHeader_2.54mm:PinHeader_1x04_P2.54mm_Vertical, F.Cu at (39.1, -26.4)
- added J17: Conn_01x04_Female, karca_custom_footprints:LPTA-4pos, F.Cu at (3.98, -52.7)
- added J18: Conn_01x04_Female, karca_custom_footprints:LPTA-4pos, F.Cu at (45.3, -52.7)
- added J19: Conn_01x04_Female, Connector_PinHeader_2.54mm:PinHeader_1x04_P2.54mm_Vertical, F.Cu at (102.7, -96.1)
- added J2: Conn_01x02_Female, Connector_PinHeader_2.54mm:PinHeader_1x03_P2.54mm_Vertical, F.Cu at (93.9, -43.0)
- added J20: Conn_01x02_Female, Connector_PinHeader_2.54mm:PinHeader_1x02_P2.54mm_Vertical, F.Cu at (143.1, -122.2)
- added J21: Conn_01x02_Female, Connector_PinHeader_2.54mm:PinHeader_1x02_P2.54mm_Vertical, F.Cu at (147.7, -122.2)
- added J22: Conn_01x02_Female, Connector_PinHeader_2.54mm:PinHeader_1x02_P2.54mm_Vertical, F.Cu at (120.5, -96.1)
- added J23: Conn_01x02_Female, Connector_PinHeader_2.54mm:PinHeader_1x02_P2.54mm_Vertical, F.Cu at (115.8, -96.1)
- added J3: Conn_01x02_Female, Connector_PinHeader_2.54mm:PinHeader_1x02_P2.54mm_Vertical, F.Cu at (116.2, -49.8)
- added J4: Conn_01x04_Female, Connector_PinHeader_2.54mm:PinHeader_1x04_P2.54mm_Vertical, F.Cu at (111.6, -49.8)
- added J5: Conn_01x02_Female, Connector_PinHeader_2.54mm:PinHeader_1x03_P2.54mm_Vertical, F.Cu at (98.5, -43.0)
- added J6: Conn_01x04_Female, karca_custom_footprints:LPTA-4pos, F.Cu at (24.6, -52.7)
- added J7: Conn_01x02_Female, Connector_PinHeader_2.54mm:PinHeader_1x02_P2.54mm_Vertical, F.Cu at (46.2, -96.1)
- added J8: Conn_01x02_Female, Connector_PinHeader_2.54mm:PinHeader_1x02_P2.54mm_Vertical, F.Cu at (41.5, -96.1)
- added Q1: FQP30N06, Package_TO_SOT_THT:TO-220-3_Vertical, F.Cu at (-0.85, -104.3)
- added Q2: FQP30N06, Package_TO_SOT_THT:TO-220-3_Horizontal_TabDown, F.Cu at (10.7, -82.3)
- added Q2: FQP30N06, Package_TO_SOT_THT:TO-220-3_Vertical, F.Cu at (76.2, -83.8)
- added Q3: FQP30N06, Package_TO_SOT_THT:TO-220-3_Vertical, F.Cu at (76.2, -77.9)
- added Q3: FQP30N06, Package_TO_SOT_THT:TO-220-3_Horizontal_TabDown, F.Cu at (10.7, -104.3)
- added Q4: FQP30N06, Package_TO_SOT_THT:TO-220-3_Horizontal_TabDown, F.Cu at (22.2, -104.3)
- added Q4: FQP30N06, Package_TO_SOT_THT:TO-220-3_Vertical, F.Cu at (87.8, -83.8)
- added Q5: FQP30N06, Package_TO_SOT_THT:TO-220-3_Horizontal_TabDown, F.Cu at (-0.85, -82.3)
- added Q5: FQP30N06, Package_TO_SOT_THT:TO-220-3_Vertical, F.Cu at (87.8, -77.9)
- added Q6: FQP30N06, Package_TO_SOT_THT:TO-220-3_Vertical, F.Cu at (76.2, -71.9)
- added Q6: FQP30N06, Package_TO_SOT_THT:TO-220-3_Horizontal_TabDown, F.Cu at (33.8, -104.3)
- added R1: 510, Resistor_SMD:R_1206_3216Metric, F.Cu at (103.7, -36.8)
- added R10: 510, Resistor_SMD:R_1206_3216Metric, F.Cu at (85.3, -119.5)
- added R11: 510, Resistor_SMD:R_1206_3216Metric, F.Cu at (70.7, -103.0)
- added R12: 510, Resistor_SMD:R_1206_3216Metric, F.Cu at (90.9, -119.5)
- added R13: 510, Resistor_SMD:R_1206_3216Metric, F.Cu at (61.6, -93.0)
- added R15: 10k, Resistor_SMD:R_1206_3216Metric, F.Cu at (53.1, -89.5)
- added R17: 10k, Resistor_SMD:R_1206_3216Metric, F.Cu at (90.9, -122.9)
- added R18: 510, Resistor_SMD:R_1206_3216Metric, F.Cu at (76.4, -109.8)
- added R19: 510, Resistor_SMD:R_1206_3216Metric, F.Cu at (44.7, -75.6)
- added R2: 10k, Resistor_SMD:R_1206_3216Metric, F.Cu at (116.7, -39.9)
- added R20: 510, Resistor_SMD:R_1206_3216Metric, F.Cu at (70.7, -99.7)
- added R21: 510, Resistor_SMD:R_1206_3216Metric, F.Cu at (58.7, -89.7)
- added R23: 10k, Resistor_SMD:R_1206_3216Metric, F.Cu at (49.4, -82.3)
- added R25: 10k, Resistor_SMD:R_1206_3216Metric, F.Cu at (61.6, -96.2)
- added R26: 510, Resistor_SMD:R_1206_3216Metric, F.Cu at (85.3, -116.2)
- added R27: 510, Resistor_SMD:R_1206_3216Metric, F.Cu at (67.2, -96.2)
- added R28: 510, Resistor_SMD:R_1206_3216Metric, F.Cu at (53.1, -86.2)
- added R29: 510, Resistor_SMD:R_1206_3216Metric, F.Cu at (39.1, -70.2)
- added R3: 68k, Resistor_SMD:R_1206_3216Metric, F.Cu at (126.0, -47.0)
- added R30: 20K, Resistor_SMD:R_1206_3216Metric, F.Cu at (80.9, -62.8)
- added R31: 200, Resistor_SMD:R_1206_3216Metric, F.Cu at (26.8, -14.0)
- added R32: 20K, Resistor_SMD:R_1206_3216Metric, F.Cu at (44.2, -27.1)
- added R33: 200, Resistor_SMD:R_1206_3216Metric, F.Cu at (60.7, -49.7)
- added R34: 20K, Resistor_SMD:R_1206_3216Metric, F.Cu at (15.6, -14.0)
- added R35: 200, Resistor_SMD:R_1206_3216Metric, F.Cu at (9.98, -14.2)
- added R36: 20K, Resistor_SMD:R_1206_3216Metric, F.Cu at (59.7, -40.2)
- added R37: 200, Resistor_SMD:R_1206_3216Metric, F.Cu at (21.2, -14.0)
- added R38: 68k, Resistor_SMD:R_1206_3216Metric, F.Cu at (195.2, -119.6)
- added R39: 68k, Resistor_SMD:R_1206_3216Metric, F.Cu at (195.2, -122.9)
- added R4: 150, Resistor_SMD:R_1206_3216Metric, F.Cu at (137.7, -59.3)
- added R40: 68k, Resistor_SMD:R_1206_3216Metric, F.Cu at (186.7, -106.0)
- added R41: 68k, Resistor_SMD:R_1206_3216Metric, F.Cu at (189.5, -119.5)
- added R42: 15k, Resistor_SMD:R_1206_3216Metric, F.Cu at (192.3, -109.6)
- added R43: 10k, Resistor_SMD:R_1206_3216Metric, F.Cu at (181.1, -106.0)
- added R44: 15k, Resistor_SMD:R_1206_3216Metric, F.Cu at (186.7, -109.5)
- added R45: 10k, Resistor_SMD:R_1206_3216Metric, F.Cu at (206.4, -122.9)
- added R46: 68k, Resistor_SMD:R_1206_3216Metric, F.Cu at (197.9, -113.0)
- added R47: 68k, Resistor_SMD:R_1206_3216Metric, F.Cu at (192.3, -112.9)
- added R48: 68k, Resistor_SMD:R_1206_3216Metric, F.Cu at (200.8, -122.9)
- added R49: 68k, Resistor_SMD:R_1206_3216Metric, F.Cu at (195.1, -116.3)
- added R5: 390, Resistor_SMD:R_1206_3216Metric, F.Cu at (122.4, -43.2)
- added R50: 15k, Resistor_SMD:R_1206_3216Metric, F.Cu at (189.5, -116.2)
- added R51: 10k, Resistor_SMD:R_1206_3216Metric, F.Cu at (186.7, -112.8)
- added R52: 15k, Resistor_SMD:R_1206_3216Metric, F.Cu at (200.8, -119.6)
- added R53: 10k, Resistor_SMD:R_1206_3216Metric, F.Cu at (200.7, -116.3)
- added R54: 22, Resistor_SMD:R_1206_3216Metric, F.Cu at (127.6, -90.0)
- added R55: 22, Resistor_SMD:R_1206_3216Metric, F.Cu at (131.3, -93.5)
- added R56: 68k, Resistor_SMD:R_1206_3216Metric, F.Cu at (143.6, -105.7)
- added R57: 68k, Resistor_SMD:R_1206_3216Metric, F.Cu at (133.2, -90.2)
- added R58: 68k, Resistor_SMD:R_1206_3216Metric, F.Cu at (154.8, -116.2)
- added R59: 68k, Resistor_SMD:R_1206_3216Metric, F.Cu at (149.2, -109.0)
- added R60: 47k, Resistor_SMD:R_1206_3216Metric, F.Cu at (149.2, -105.7)
- added R61: 5.1k, Resistor_SMD:R_1206_3216Metric, F.Cu at (143.6, -109.0)
- added R62: 47k, Resistor_SMD:R_1206_3216Metric, F.Cu at (158.5, -122.9)
- added R63: 5.1k, Resistor_SMD:R_1206_3216Metric, F.Cu at (164.1, -119.6)
- added R64: 22, Resistor_SMD:R_1206_3216Metric, F.Cu at (154.8, -112.3)
- added R65: 22, Resistor_SMD:R_1206_3216Metric, F.Cu at (136.9, -96.7)
- added R66: 68k, Resistor_SMD:R_1206_3216Metric, F.Cu at (131.3, -96.7)
- added R67: 68k, Resistor_SMD:R_1206_3216Metric, F.Cu at (158.5, -119.6)
- added R68: 68k, Resistor_SMD:R_1206_3216Metric, F.Cu at (143.6, -102.4)
- added R69: 68k, Resistor_SMD:R_1206_3216Metric, F.Cu at (136.9, -93.5)
- added R7: 10k, Resistor_SMD:R_1206_3216Metric, F.Cu at (49.4, -79.0)
- added R70: 47k, Resistor_SMD:R_1206_3216Metric, F.Cu at (164.1, -122.9)
- added R71: 5.1k, Resistor_SMD:R_1206_3216Metric, F.Cu at (143.6, -99.1)
- added R72: 47k, Resistor_SMD:R_1206_3216Metric, F.Cu at (149.2, -112.3)
- added R73: 5.1k, Resistor_SMD:R_1206_3216Metric, F.Cu at (160.5, -116.3)
- added R74: 100k, Resistor_SMD:R_1206_3216Metric, F.Cu at (160.8, -69.5)
- added R75: 100k, Resistor_SMD:R_1206_3216Metric, F.Cu at (155.2, -66.1)
- added R76: 100k, Resistor_SMD:R_1206_3216Metric, F.Cu at (149.5, -62.8)
- added R77: 150, Resistor_SMD:R_1206_3216Metric, F.Cu at (4.37, -7.67)
- added R9: 10k, Resistor_SMD:R_1206_3216Metric, F.Cu at (76.4, -106.5)
- added RV1: 30k, Resistor_SMD:R_1206_3216Metric, F.Cu at (66.3, -49.7)
- added RV2: 30k, Resistor_SMD:R_1206_3216Metric, F.Cu at (39.6, -14.8)
- added RV3: 30k, Resistor_SMD:R_1206_3216Metric, F.Cu at (60.7, -46.4)
- added RV4: 30k, Resistor_SMD:R_1206_3216Metric, F.Cu at (4.37, -14.2)
- added U1: LM1084-ADJ, Package_TO_SOT_SMD:TO-263-3_TabPin2, F.Cu at (100.4, -51.5)
- added U10: MCP3208-CI/SL, Package_SO:SOIC-16_3.9x9.9mm_P1.27mm, F.Cu at (151.0, -76.9)
- added U11: MCP3208-CI/SL, Package_SO:SOIC-16_3.9x9.9mm_P1.27mm, F.Cu at (167.9, -76.9)
- added U2: LM1084-5.0, Package_TO_SOT_SMD:TO-263-3_TabPin2, F.Cu at (120.4, -58.2)
- added U3: MCP6N11T-001E, Package_DFN_QFN:TDFN-8-1EP_3x2mm_P0.5mm_EP1.80x1.65mm, F.Cu at (49.7, -27.0)
- added U4: MCP6N11T-001E, Package_DFN_QFN:TDFN-8-1EP_3x2mm_P0.5mm_EP1.80x1.65mm, F.Cu at (66.2, -46.3)
- added U5: MCP6N11T-001E, Package_DFN_QFN:TDFN-8-1EP_3x2mm_P0.5mm_EP1.80x1.65mm, F.Cu at (80.8, -59.4)
- added U6: MCP6N11T-001E, Package_DFN_QFN:TDFN-8-1EP_3x2mm_P0.5mm_EP1.80x1.65mm, F.Cu at (44.1, -23.7)
- added U7: LM324DT, Package_SO:SOIC-14_3.9x8.7mm_P1.27mm, F.Cu at (176.8, -119.4)
- added U8: LM324DT, Package_SO:SOIC-14_3.9x8.7mm_P1.27mm, F.Cu at (109.3, -93.3)
- added U9: MCP3208-CI/SL, Package_SO:SOIC-16_3.9x9.9mm_P1.27mm, F.Cu at (159.4, -76.9)

Commit message: updated all footprints, resolved most ERC & setup layout
Parts:
- added J16: Conn_01x08_Female, Connector_PinSocket_2.54mm:PinSocket_1x08_P2.54mm_Vertical, F.Cu at (347.8, 66.0)
- added J29: Conn_01x03_Female, Connector_PinSocket_2.54mm:PinSocket_1x03_P2.54mm_Vertical, F.Cu at (327.8, 95.5)
- added J30: Conn_01x03_Female, Connector_PinSocket_2.54mm:PinSocket_1x03_P2.54mm_Vertical, F.Cu at (323.1, 95.5)
- added J31: Conn_01x03_Female, Connector_PinSocket_2.54mm:PinSocket_1x03_P2.54mm_Vertical, F.Cu at (332.4, 95.5)
- added J32: Conn_01x03_Female, Connector_PinSocket_2.54mm:PinSocket_1x03_P2.54mm_Vertical, F.Cu at (323.1, 105.2)
- added J33: Conn_01x08_Female, Connector_PinSocket_2.54mm:PinSocket_1x08_P2.54mm_Vertical, F.Cu at (348.6, 95.5)
- added J34: Conn_01x08_Female, Connector_PinSocket_2.54mm:PinSocket_1x08_P2.54mm_Vertical, F.Cu at (344.0, 95.5)
- added J35: Conn_01x08_Female, Connector_PinSocket_2.54mm:PinSocket_1x08_P2.54mm_Vertical, F.Cu at (353.2, 95.5)
- added J36: 2540-5, Connector_PinHeader_2.54mm:PinHeader_2x20_P2.54mm_Horizontal, F.Cu at (286.6, 66.0)
- added J9: Conn_01x08_Female, Connector_PinSocket_2.54mm:PinSocket_1x08_P2.54mm_Vertical, F.Cu at (365.8, 66.0)
- added SW1: 1101M2S3CQE2, 1101M2S3CQE2:SW_1101M2S3CQE2, F.Cu at (326.0, 70.8)
- added SW2: 1101M2S3CQE2, 1101M2S3CQE2:SW_1101M2S3CQE2, F.Cu at (335.3, 70.8)
- J2, J5: footprint Connector_PinHeader_2.54mm:PinHeader_1x03_P2.54mm_Vertical -> Connector_PinHeader_2.54mm:PinHeader_1x02_P2.54mm_Vertical
- RV1, RV2, RV3, RV4: footprint Resistor_SMD:R_1206_3216Metric -> 3296W-1-303LF:TRIM_3296W-1-303LF
- moved U1 23.1 mm to (110.9, 76.2)
Other:
- board outline added: 355.6 x 152.4 mm
- copper layers 2 -> 4

Commit message: grouped components on PCB
Parts:
- removed the C1 at (109.2, 58.4)
- removed the C2 at (101.6, 28.8)
- removed the C2 at (132.1, -59.2)
- removed the C3 at (107.2, 25.4)
- removed the C4 at (134.6, 58.4)
- removed the Q2 at (10.7, -82.3)
- removed the Q3 at (10.7, -104.3)
- removed the Q4 at (22.2, -104.3)
- removed the Q4 at (87.8, -83.8)
- removed the Q5 at (-0.85, -82.3)
- removed the Q6 at (76.2, -71.9)
- removed the Q6 at (33.8, -104.3)
- removed the R1 at (116.8, 43.2)
- removed the R2 at (116.8, 48.3)
- removed the R3 at (109.2, 33.0)
- removed the R4 at (114.3, 33.0)
- removed the R4 at (137.7, -59.3)
- removed the U1 at (110.9, 76.2)
- removed the U1 at (100.4, -51.5)
- added C2: 10uF, Capacitor_SMD:C_1206_3216Metric, F.Cu at (269.2, -38.1)
- added Q4: FQP30N06, Package_TO_SOT_THT:TO-220-3_Horizontal_TabDown, F.Cu at (-101.6, -84.8)
- added Q6: FQP30N06, Package_TO_SOT_THT:TO-220-3_Horizontal_TabDown, F.Cu at (-195.6, -74.6)
- added R14: DNP, Resistor_SMD:R_1206_3216Metric, F.Cu at (-186.9, -114.3)
- added R16: DNP, Resistor_SMD:R_1206_3216Metric, F.Cu at (-87.9, -75.7)
- added R22: DNP, Resistor_SMD:R_1206_3216Metric, F.Cu at (-103.1, -116.8)
- added R24: DNP, Resistor_SMD:R_1206_3216Metric, F.Cu at (-176.7, -71.1)
- added R4: 150, Resistor_SMD:R_1206_3216Metric, F.Cu at (269.2, -73.7)
- added R6: DNP, Resistor_SMD:R_1206_3216Metric, F.Cu at (-193.0, -165.1)
- added R8: DNP, Resistor_SMD:R_1206_3216Metric, F.Cu at (-121.9, -172.7)
- added U1: LM1084-ADJ, Package_TO_SOT_SMD:TO-263-3_TabPin2, F.Cu at (284.5, -33.0)
- Q1, Q2, Q3, Q5: footprint Package_TO_SOT_THT:TO-220-3_Vertical -> Package_TO_SOT_THT:TO-220-3_Horizontal_TabDown
- moved J9 630.9 mm to (-231.1, -138.4)
- moved J16 566.4 mm to (-218.4, 53.3)
- moved R30 403.5 mm to (-304.8, 55.9)
- moved RV1 375.4 mm to (-294.6, 53.3)
- moved U3 362.4 mm to (-304.8, 48.3)
- moved F7 355.4 mm to (-325.0, 60.3)
- moved R31 340.0 mm to (-304.8, 61.0)
- moved U4 321.3 mm to (-205.9, 124.6)
- moved J6 317.5 mm to (-246.5, 112.4), turned to 90 degrees
- moved R33 309.9 mm to (-203.3, 112.4)
- moved C5 305.3 mm to (-297.2, 61.0), turned to 90 degrees
- moved J29 301.9 mm to (45.7, 203.2)
- moved RV2 301.5 mm to (-226.2, 127.6)
- moved U5 294.6 mm to (-191.5, 53.3)
- moved J14 292.9 mm to (-274.3, 61.0)
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Connections:
- U3 pad 9: (no net) -> GND
- U4 pad 9: (no net) -> GND
- U5 pad 9: (no net) -> GND
- U6 pad 9: (no net) -> GND

Commit message: preliminary layout and started pwr plane config
Parts:
- removed the J30 at (67.0, 205.7)
- removed the J31 at (104.1, 203.2)
- removed the J32 at (61.0, 228.6)
- added C20: 1nF, Capacitor_SMD:C_1206_3216Metric, F.Cu at (267.5, 76.3)
- added C21: 100nF, Capacitor_SMD:C_1206_3216Metric, F.Cu at (242.6, 90.2)
- added C22: 1nF, Capacitor_SMD:C_1206_3216Metric, F.Cu at (233.2, 77.6)
- added C23: 1nF, Capacitor_SMD:C_1206_3216Metric, F.Cu at (262.4, 76.3)
- added C24: 1nF, Capacitor_SMD:C_1206_3216Metric, F.Cu at (226.6, 77.6)
- added C7: 1uF, Capacitor_SMD:C_1206_3216Metric, F.Cu at (180.9, 57.1)
- added C9: 1uF, Capacitor_SMD:C_1206_3216Metric, F.Cu at (266.0, 56.0)
- added F12: 3588-20, 3588-20:358820, F.Cu at (259.1, 55.9)
- added F9: 3588-20, 3588-20:358820, F.Cu at (176.5, 54.5)
- added J19: Conn_01x06_Female, Connector_PinSocket_2.54mm:PinSocket_1x06_P2.54mm_Vertical, F.Cu at (184.2, 95.2)
- added J24: Screw_Terminal_01x02, 1190363:1190363, F.Cu at (334.4, 31.9)
- added J26: Screw_Terminal_01x03, 1190364:1190364, F.Cu at (40.4, 31.9)
- added J27: Screw_Terminal_01x03, 1190364:1190364, F.Cu at (62.6, 31.9)
- added J28: Screw_Terminal_01x03, 1190364:1190364, F.Cu at (107.0, 31.9)
- added J4: Screw_Terminal_01x02, 1190363:1190363, F.Cu at (191.4, 150.9)
- added J5: Screw_Terminal_01x02, 1190363:1190363, F.Cu at (285.4, 150.9)
- added R32: 20K, Resistor_SMD:R_1206_3216Metric, F.Cu at (180.9, 47.0)
- added R35: 200, Resistor_SMD:R_1206_3216Metric, F.Cu at (188.9, 57.1)
- added R38: 20K, Resistor_SMD:R_1206_3216Metric, F.Cu at (263.8, 50.9)
- added R41: 200, Resistor_SMD:R_1206_3216Metric, F.Cu at (268.5, 50.9)
- added R58: 68k, Resistor_SMD:R_1206_3216Metric, F.Cu at (262.9, 68.7)
- added R59: 68k, Resistor_SMD:R_1206_3216Metric, F.Cu at (262.9, 65.4)
- added R60: 68k, Resistor_SMD:R_1206_3216Metric, F.Cu at (227.0, 67.4)
- added R61: 68k, Resistor_SMD:R_1206_3216Metric, F.Cu at (232.1, 72.5)
- added R62: 15k, Resistor_SMD:R_1206_3216Metric, F.Cu at (268.5, 68.7)
- added R63: 15k, Resistor_SMD:R_1206_3216Metric, F.Cu at (226.5, 72.6)
- added R64: 10k, Resistor_SMD:R_1206_3216Metric, F.Cu at (268.5, 65.4)
- added R65: 10k, Resistor_SMD:R_1206_3216Metric, F.Cu at (232.1, 67.4)
- added RV3: 30k, 3296W-1-303LF:TRIM_3296W-1-303LF, F.Cu at (189.0, 48.1)
- added RV6: 30k, 3296W-1-303LF:TRIM_3296W-1-303LF, F.Cu at (267.5, 45.8)
- added U10: LM324DT, Package_SO:SOIC-14_3.9x8.7mm_P1.27mm, F.Cu at (242.6, 80.0)
- added U5: MCP6N11T-001E, Package_DFN_QFN:TDFN-8-1EP_3x2mm_P0.5mm_EP1.80x1.65mm, F.Cu at (179.8, 52.1)
- added U8: MCP6N11T-001E, Package_DFN_QFN:TDFN-8-1EP_3x2mm_P0.5mm_EP1.80x1.65mm, F.Cu at (275.1, 56.0)
- F1, F4, F7: footprint karca_custom_footprints:3588-20 fuse -> 3588-20:358820
- F10: renamed from F8; footprint karca_custom_footprints:3588-20 fuse -> 3588-20:358820
- F11: renamed from F10; footprint karca_custom_footprints:3588-20 fuse -> 3588-20:358820
- F13: renamed from F14; footprint karca_custom_footprints:3588-20 fuse -> 3588-20:358820
- F14: renamed from F11; footprint karca_custom_footprints:3588-20 fuse -> 3588-20:358820
- F15: renamed from F12; footprint karca_custom_footprints:3588-20 fuse -> 3588-20:358820
- F16: renamed from F13; footprint karca_custom_footprints:3588-20 fuse -> 3588-20:358820
- F17: renamed from F15; footprint karca_custom_footprints:3588-20 fuse -> 3588-20:358820
- F18: renamed from F16; footprint karca_custom_footprints:3588-20 fuse -> 3588-20:358820
- F19: renamed from F17; footprint karca_custom_footprints:3588-20 fuse -> 3588-20:358820
- F2: renamed from F3; footprint karca_custom_footprints:3588-20 fuse -> 3588-20:358820
- F20: renamed from F18; footprint karca_custom_footprints:3588-20 fuse -> 3588-20:358820
- F3: renamed from F5; footprint karca_custom_footprints:3588-20 fuse -> 3588-20:358820
- F5: renamed from F6; footprint karca_custom_footprints:3588-20 fuse -> 3588-20:358820
- F6: renamed from F2; footprint karca_custom_footprints:3588-20 fuse -> 3588-20:358820
- F8: renamed from F9; footprint karca_custom_footprints:3588-20 fuse -> 3588-20:358820
- J10, J11, J2, J21, J22, J23, J3, J7, J8: value Conn_01x02_Female -> Screw_Terminal_01x02; footprint Connector_PinHeader_2.54mm:PinHeader_1x02_P2.54mm_Vertical -> 1190363:1190363
- J12: value Conn_01x02_Female -> Conn_01x08_Female; footprint Connector_PinHeader_2.54mm:PinHeader_1x02_P2.54mm_Vertical -> Connector_PinSocket_2.54mm:PinSocket_1x08_P2.54mm_Vertical
- J13: value Conn_01x02_Female -> Screw_Terminal_01x04; footprint Connector_PinHeader_2.54mm:PinHeader_1x02_P2.54mm_Vertical -> 1190365:1190365
- J14, J17, J18: value Conn_01x04_Female -> Screw_Terminal_01x04; footprint karca_custom_footprints:LPTA-4pos -> 1190365:1190365
- J15: value Conn_01x04_Female -> Screw_Terminal_01x04; footprint Connector_PinHeader_2.54mm:PinHeader_1x04_P2.54mm_Vertical -> 1190365:1190365
- J16: value Conn_01x08_Female -> Screw_Terminal_01x04; footprint Connector_PinSocket_2.54mm:PinSocket_1x08_P2.54mm_Vertical -> 1190365:1190365
- J20: value Conn_01x02_Female -> Conn_02x06_Odd_Even; footprint Connector_PinHeader_2.54mm:PinHeader_1x02_P2.54mm_Vertical -> Connector_PinSocket_2.54mm:PinSocket_2x06_P2.54mm_Vertical
- J29: value Conn_01x03_Female -> Screw_Terminal_01x03; footprint Connector_PinSocket_2.54mm:PinSocket_1x03_P2.54mm_Vertical -> 1190364:1190364
- J6: value Conn_01x04_Female -> Screw_Terminal_01x02; footprint karca_custom_footprints:LPTA-4pos -> 1190363:1190363
- J9: value Conn_01x08_Female -> Screw_Terminal_01x02; footprint Connector_PinSocket_2.54mm:PinSocket_1x08_P2.54mm_Vertical -> 1190363:1190363
- moved J9 653.3 mm to (356.4, 147.4), turned to 90 degrees
- moved D11 652.0 mm to (424.2, 88.9)
- moved R10 652.0 mm to (423.1, 96.5)
- moved D14 652.0 mm to (433.3, 91.4)
- moved R13 652.0 mm to (429.3, 99.1)
- moved D9 651.5 mm to (444.5, 91.4)
- moved R7 651.5 mm to (444.5, 96.5)
- moved Q1 638.7 mm to (395.3, 74.9), turned to 90 degrees
- moved D13 636.7 mm to (403.7, 67.9)
- moved D8 636.7 mm to (424.1, 80.6)
- moved F1 636.7 mm to (416.6, 74.9)
- moved R15 636.7 mm to (407.4, 75.6)
- moved R16 636.5 mm to (436.9, 99.1)
- moved R6 634.5 mm to (412.6, 77.5)
- moved R9 634.5 mm to (414.0, 82.5)
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- renumbered C2 to C1, C6 to C10, C16 to C11, C14 to C13, C10 to C14, C13 to C15, C17 to C16, C9 to C17, C11 to C18, C15 to C19, C4 to C2, C26 to C25, C20 to C26, C24 to C27, C18 to C28, C21 to C29, C1 to C3, C25 to C30, C19 to C31, C23 to C32, C22 to C33, C27 to C34, C28 to C35, C29 to C36, C3 to C4, C7 to C6, D19 to D10, D17 to D11, D23 to D12, D9 to D13, D16 to D14, D21 to D15, D14 to D16, D18 to D17, D20 to D18, D8 to D19, D24 to D20, D12 to D21, D15 to D22, D22 to D23, D10 to D24, D6 to D4, D4 to D5, D5 to D6, D11 to D8, D13 to D9, J4 to J1, J19 to J25, J33 to J30, J34 to J31, J35 to J32, J36 to J33, Q3 to Q2, Q5 to Q3, Q6 to Q5, Q2 to Q6, R20 to R10, R28 to R11, R6 to R12, R14 to R13, R22 to R14, R7 to R15, R15 to R16, R23 to R17, R19 to R18, R27 to R19, R3 to R2, R11 to R20, R29 to R22, R13 to R23, R16 to R24, R24 to R25, R8 to R26, R17 to R27, R25 to R28, R9 to R29, R5 to R3, R34 to R31, R31 to R33, R35 to R34, R32 to R36, R36 to R37, R33 to R39, R2 to R4, R37 to R40, R46 to R42, R48 to R43, R38 to R44, R40 to R45, R50 to R46, R42 to R47, R51 to R48, R43 to R49, R4 to R5, R39 to R50, R41 to R51, R47 to R52, R49 to R53, R44 to R54, R52 to R55, R45 to R56, R53 to R57, R10 to R6, R67 to R66, R69 to R67, R56 to R68, R58 to R69, R18 to R7, R65 to R70, R72 to R71, R54 to R72, R60 to R73, R73 to R74, R61 to R75, R57 to R76, R59 to R77, R66 to R78, R68 to R79, R26 to R8, R55 to R80, R62 to R81, R64 to R82, R70 to R83, R63 to R84, R71 to R85, R74 to R86, R75 to R87, R76 to R88, R77 to R89, R12 to R9, RV3 to RV2, RV2 to RV4, RV4 to RV5, SW2 to SW1, SW1 to SW2, U8 to U11, U9 to U12, U10 to U13, U11 to U14, U5 to U4, U4 to U6, U6 to U7, U7 to U9
Connections:
- net /ADCs/adc1_nc5 renamed /ADCs/LC5_CAL
- net /ADCs/adc1_nc6 renamed /ADCs/LC6_CAL
- F10 pad 2: Net-(F8-Pad2) -> Net-(F10-Pad2)
- F11 pad 2: Net-(F10-Pad2) -> Net-(F11-Pad2)
- F13 pad 2: Net-(F14-Pad2) -> Net-(F13-Pad2)
- F14 pad 2: Net-(F11-Pad2) -> Net-(F14-Pad2)
- F15 pad 2: Net-(F12-Pad2) -> Net-(F15-Pad2)
- F16 pad 2: Net-(F13-Pad2) -> Net-(F16-Pad2)
- F17 pad 2: Net-(F15-Pad2) -> Net-(F17-Pad2)
- F20 pad 2: Net-(F18-Pad2) (its old number) -> Net-(F20-Pad2)
- F8 pad 2: Net-(F9-Pad2) -> Net-(F8-Pad2)
- J10 pad 1: /Drivers/DRV_POS_2 -> /Drivers/DRV_POS_6
- J10 pad 2: /Drivers/DRV_NEG_2 -> /Drivers/DRV_NEG_6
- J11 pad 1: /Drivers/DRV_POS_5 -> /Drivers/DRV_POS_4
- J11 pad 2: /Drivers/DRV_NEG_5 -> /Drivers/DRV_NEG_4
- J12 pad 1: /Drivers/DRV_POS_3 -> DRV_CTL_1
- J12 pad 2: /Drivers/DRV_NEG_3 -> DRV_CTL_2
- J13 pad 1: /Drivers/DRV_POS_6 -> Net-(F7-Pad2)
- J13 pad 2: /Drivers/DRV_NEG_6 -> /Load Cell Inamps/LC1-
- J14 pad 1: Net-(F7-Pad2) -> Net-(F8-Pad2)
- J14 pad 2: /Load Cell Inamps/LC1- -> /Load Cell Inamps/LC2-
- J14 pad 3: /Load Cell Inamps/LC1+ -> /Load Cell Inamps/LC2+
- J15 pad 1: LC1_PREC -> Net-(F9-Pad2)
- J15 pad 2: LC2_PREC -> /Load Cell Inamps/LC3-
- J15 pad 3: LC3_PREC -> /Load Cell Inamps/LC3+
- J15 pad 4: LC4_PREC -> GND
- J16 pad 1: /Load Cell Inamps/LC1+ -> Net-(F10-Pad2)
- J16 pad 2: /Load Cell Inamps/LC1- -> /Load Cell Inamps/LC4-
- J16 pad 3: /Load Cell Inamps/LC2+ -> /Load Cell Inamps/LC4+
- J16 pad 4: /Load Cell Inamps/LC2- -> GND
- J16 pad 5: /Load Cell Inamps/LC3+ -> (no net)
- J16 pad 6: /Load Cell Inamps/LC3- -> (no net)
- J16 pad 7: /Load Cell Inamps/LC4+ -> (no net)
- J16 pad 8: /Load Cell Inamps/LC4- -> (no net)
- J17 pad 1: Net-(F9-Pad2) -> Net-(F11-Pad2)
- J17 pad 2: /Load Cell Inamps/LC2- -> /Load Cell Inamps/LC5-
- J17 pad 3: /Load Cell Inamps/LC2+ -> /Load Cell Inamps/LC5+
- J18 pad 1: Net-(F10-Pad2) -> Net-(F12-Pad2)
- J18 pad 2: /Load Cell Inamps/LC4- -> /Load Cell Inamps/LC6-
- J18 pad 3: /Load Cell Inamps/LC4+ -> /Load Cell Inamps/LC6+
- J20 pad 1: Net-(F11-Pad2) -> /Load Cell Inamps/LC1+
- J20 pad 2: /PT Amplification/PT1- -> /Load Cell Inamps/LC1-
- J21 pad 1: Net-(F12-Pad2) -> Net-(F13-Pad2)
- J21 pad 2: /PT Amplification/PT3- -> /PT Amplification/PT2-
- J22 pad 1: Net-(F13-Pad2) -> Net-(F14-Pad2)
- J22 pad 2: /PT Amplification/PT4- -> /PT Amplification/PT1-
- J23 pad 1: Net-(F14-Pad2) -> Net-(F15-Pad2)
- J23 pad 2: /PT Amplification/PT2- -> /PT Amplification/PT3-
- J29 pad 1: Net-(F15-Pad2) -> Net-(F20-Pad2)
- J29 pad 2: TC1 -> TC4
- J31 pad 1: /ADCs/LC1_CAL -> /ADCs/PT1_CAL
- J31 pad 2: /ADCs/LC2_CAL -> /ADCs/PT2_CAL
- J31 pad 3: /ADCs/LC3_CAL -> /ADCs/PT3_CAL
- J31 pad 4: /ADCs/LC4_CAL -> /ADCs/PT4_CAL
- J6 pad 1: Net-(F8-Pad2) -> /Drivers/DRV_POS_1
- J6 pad 2: /Load Cell Inamps/LC3- -> /Drivers/DRV_NEG_1
- J6 pad 3: /Load Cell Inamps/LC3+ -> (no net)
- J6 pad 4: GND -> (no net)
- J7 pad 1: /Drivers/DRV_POS_1 -> /Drivers/DRV_POS_2
- J7 pad 2: /Drivers/DRV_NEG_1 -> /Drivers/DRV_NEG_2
- J8 pad 1: /Drivers/DRV_POS_4 -> /Drivers/DRV_POS_3
- J8 pad 2: /Drivers/DRV_NEG_4 -> /Drivers/DRV_NEG_3
- J9 pad 1: DRV_CTL_1 -> /Drivers/DRV_POS_5
- J9 pad 2: DRV_CTL_2 -> /Drivers/DRV_NEG_5
- J9 pad 3: DRV_CTL_3 -> (no net)
- J9 pad 4: DRV_CTL_4 -> (no net)
- R36 pad 1: LC3_PREC -> LC4_PREC
- R37 pad 1: LC4_PREC -> LC5_PREC
- R39 pad 2: LC3_PREC -> LC4_PREC
- R40 pad 2: LC4_PREC -> LC5_PREC
- U13 pad 1: /ADCs/LC1_CAL -> /ADCs/PT1_CAL
- U13 pad 2: /ADCs/LC2_CAL -> /ADCs/PT2_CAL
- U13 pad 3: /ADCs/LC3_CAL -> /ADCs/PT3_CAL
- U13 pad 4: /ADCs/LC4_CAL -> /ADCs/PT4_CAL
- U6 pad 2: /Load Cell Inamps/LC3- -> /Load Cell Inamps/LC4-
- U6 pad 3: /Load Cell Inamps/LC3+ -> /Load Cell Inamps/LC4+
- U6 pad 6: LC3_PREC -> LC4_PREC
- U7 pad 2: /Load Cell Inamps/LC4- -> /Load Cell Inamps/LC5-
- U7 pad 3: /Load Cell Inamps/LC4+ -> /Load Cell Inamps/LC5+
- U7 pad 6: LC4_PREC -> LC5_PREC
Routing:
- added copper zone on B.Cu, net +10V
- added copper zone on B.Cu, net +12V
- added copper zone on B.Cu, net +5V
- added copper zone on In1.Cu, net GND
Other:
- board text added: "load cells"
- board text added: "thermocouples"

Commit message: fixed pwr planes
Parts:
- removed the J5 at (307.3, -58.4)
- moved C3 303.6 mm to (57.3, 150.9)
- moved C4 303.6 mm to (59.8, 145.8)
- moved D5 303.6 mm to (63.5, 140.7)
- moved D6 303.6 mm to (57.3, 158.5)
- moved R5 303.6 mm to (64.9, 150.9)
- moved U2 303.6 mm to (81.8, 153.4)
- moved J1 208.1 mm to (260.4, 130.8), turned to 90 degrees
- moved D1 198.5 mm to (290.8, 130.8)
- moved D2 198.5 mm to (313.7, 125.7)
- moved J1 198.5 mm to (308.6, 118.1)
- moved R1 198.5 mm to (313.7, 130.8)
- moved SW2 198.5 mm to (298.4, 118.1)
- moved C1 155.3 mm to (224.0, 110.5)
- moved C2 155.3 mm to (213.8, 120.7)
- moved D3 155.3 mm to (221.4, 120.7)
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Routing:
- net (no net): vias 0 -> 6

Commit message: some minor schematic cleanup
Parts:
- J12: value Conn_01x08_Female -> Conn_01x06_Female; footprint Connector_PinSocket_2.54mm:PinSocket_1x08_P2.54mm_Vertical -> Connector_PinSocket_2.54mm:PinSocket_1x06_P2.54mm_Vertical
- Q1, Q2, Q3, Q4, Q5, Q6: footprint Package_TO_SOT_THT:TO-220-3_Horizontal_TabDown -> Package_TO_SOT_THT:TO-220-3_Vertical
- moved D7 22.0 mm to (422.0, 83.8)
- moved D8 22.0 mm to (445.8, 84.5)
- moved R12 22.0 mm to (412.8, 83.8)
- moved R15 22.0 mm to (429.1, 79.4)
- moved R9 22.0 mm to (435.8, 86.4)
- moved D13 22.0 mm to (425.5, 71.8)
- moved F1 22.0 mm to (438.3, 78.7)
- moved Q1 22.0 mm to (417.1, 78.7)
- moved R6 22.0 mm to (434.3, 81.3)

Commit message: shuffle around some parts
Parts:
- added SW1: S101031MS02Q, S101031MS02Q:S101031MS02Q, F.Cu at (264.2, 177.8)
- added SW2: S101031MS02Q, S101031MS02Q:S101031MS02Q, F.Cu at (246.6, 177.8)
- C1, C2, C3, C4: value 10uF -> 10u
- C10, C5, C6, C7, C8, C9: value 1uF -> 1u
- C11, C12, C13, C14, C15, C16, C18, C19, C20, C22, C23, C24, C25, C26, C27, C28, C29, C30, C31, C32: value 1nF -> 1n
- C17, C21, C33, C34, C35, C36: value 100nF -> 100n
- DRV_STAT_1: renamed from D7; value DRV_STAT_1 -> YLW
- DRV_STAT_2: renamed from D9; value DRV_STAT_2 -> YLW
- DRV_STAT_3: renamed from D10; value DRV_STAT_3 -> YLW
- DRV_STAT_4: renamed from D19; value DRV_STAT_4 -> YLW
- DRV_STAT_5: renamed from D16; value DRV_STAT_5 -> YLW
- DRV_STAT_6: renamed from D18; value DRV_STAT_6 -> YLW
- F1, F10, F11, F12, F13, F14, F15, F16, F17, F18, F19, F2, F20, F3, F7, F8, F9: value 3588-20 -> 178.6165; footprint 3588-20:358820 -> 178.6165:17861650002
- F4: renamed from F6; value 3588-20 -> 178.6165; footprint 3588-20:358820 -> 178.6165:17861650002
- F5: renamed from F4; value 3588-20 -> 178.6165; footprint 3588-20:358820 -> 178.6165:17861650002
- F6: renamed from F5; value 3588-20 -> 178.6165; footprint 3588-20:358820 -> 178.6165:17861650002
- FS_STAT_1: renamed from D8; value FS_STAT_1 -> BLU
- FS_STAT_2: renamed from D11; value FS_STAT_2 -> BLU
- FS_STAT_3: renamed from D12; value FS_STAT_3 -> BLU
- FS_STAT_4: renamed from D21; value FS_STAT_4 -> BLU
- FS_STAT_5: renamed from D17; value FS_STAT_5 -> BLU
- FS_STAT_6: renamed from D20; value FS_STAT_6 -> BLU
- HBT1: renamed from D25; value HBT -> BLU
- LED_10V1: renamed from D4; value PWR_10V -> RED
- LED_12V1: renamed from D2; value PWR_12V -> RED
- LED_5V1: renamed from D6; value PWR_5V -> RED
- RV1, RV2, RV3, RV4, RV5, RV6: footprint 3296W-1-303LF:TRIM_3296W-1-303LF -> Potentiometer_THT:Potentiometer_Bourns_3296W_Vertical
- moved F1 19.8 mm to (447.0, 61.0)
- moved R15 13.2 mm to (432.8, 66.7)
- moved R6 13.2 mm to (438.0, 68.6)
- moved R9 13.2 mm to (439.4, 73.7)
- moved D13 13.2 mm to (429.1, 59.1)
- moved DRV_STAT_1 13.2 mm to (425.6, 71.1)
- moved Q1 13.2 mm to (420.7, 66.0)
- moved R12 13.2 mm to (416.4, 71.1)
- moved FS_STAT_1 13.2 mm to (449.5, 71.8)
- moved F17 0.66 mm to (30.5, 50.8)
- renumbered J5 to J1, J9 to J10, J10 to J11, J1 to J5, J11 to J9, Q6 to Q4, Q4 to Q5, Q5 to Q6
Connections:
- net Net-(F13-Pad2) renamed /PT Amplification/PT2+
- net Net-(F14-Pad2) renamed /PT Amplification/PT1+
- net Net-(F15-Pad2) renamed /PT Amplification/PT3+
- net Net-(F16-Pad2) renamed /PT Amplification/PT4+
- J30 pad 1: /ADCs/LC1_CAL -> LC1_CAL
- J30 pad 2: /ADCs/LC2_CAL -> LC2_CAL
- J30 pad 3: /ADCs/LC3_CAL -> LC3_CAL
- J30 pad 4: /ADCs/LC4_CAL -> LC4_CAL
- J30 pad 5: /ADCs/LC5_CAL -> LC5_CAL
- J30 pad 6: /ADCs/LC6_CAL -> LC6_CAL
- J31 pad 1: /ADCs/PT1_CAL -> PT1_CAL
- J31 pad 2: /ADCs/PT2_CAL -> PT2_CAL
- J31 pad 3: /ADCs/PT3_CAL -> PT3_CAL
- J31 pad 4: /ADCs/PT4_CAL -> PT4_CAL
- J32 pad 1: /ADCs/TC1 -> TC1
- J32 pad 2: /ADCs/TC2 -> TC2
- J32 pad 3: /ADCs/TC3 -> TC3
- J32 pad 4: /ADCs/TC4 -> TC4
- U12 pad 1: /ADCs/LC1_CAL -> LC1_CAL
- U12 pad 2: /ADCs/LC2_CAL -> LC2_CAL
- U12 pad 3: /ADCs/LC3_CAL -> LC3_CAL
- U12 pad 4: /ADCs/LC4_CAL -> LC4_CAL
- U12 pad 5: /ADCs/LC5_CAL -> LC5_CAL
- U12 pad 6: /ADCs/LC6_CAL -> LC6_CAL
- U13 pad 1: /ADCs/PT1_CAL -> PT1_CAL
- U13 pad 2: /ADCs/PT2_CAL -> PT2_CAL
- U13 pad 3: /ADCs/PT3_CAL -> PT3_CAL
- U13 pad 4: /ADCs/PT4_CAL -> PT4_CAL
- U14 pad 1: /ADCs/TC1 -> TC1
- U14 pad 2: /ADCs/TC2 -> TC2
- U14 pad 3: /ADCs/TC3 -> TC3
- U14 pad 4: /ADCs/TC4 -> TC4

Commit message: add overvoltage diodes
Parts:
- added D10: SS54, karca_custom_footprints:DO-214AC, F.Cu at (332.5, 215.9)
- added D11: SS54, karca_custom_footprints:DO-214AC, F.Cu at (325.1, 212.4)
- added D12: SS54, karca_custom_footprints:DO-214AC, F.Cu at (332.5, 212.4)
- added D16: SS54, karca_custom_footprints:DO-214AC, F.Cu at (325.1, 215.9)
- added D2: SS54, karca_custom_footprints:DO-214AC, F.Cu at (302.3, 215.9)
- added D4: SS54, karca_custom_footprints:DO-214AC, F.Cu at (302.3, 212.4)
- added D6: SS54, karca_custom_footprints:DO-214AC, F.Cu at (302.3, 219.4)
- added D7: SS54, karca_custom_footprints:DO-214AC, F.Cu at (309.6, 212.4)
- added D8: SS54, karca_custom_footprints:DO-214AC, F.Cu at (309.6, 215.9)
- added D9: SS54, karca_custom_footprints:DO-214AC, F.Cu at (309.6, 219.4)
- moved C9 3.07 mm to (262.2, 69.8)
- moved F12 3.07 mm to (259.1, 50.8)
- moved R58 3.07 mm to (264.7, 81.3)
- moved R59 3.07 mm to (264.7, 78.0)
- moved C10 3.07 mm to (206.3, 68.6)
- moved C16 3.07 mm to (206.3, 85.1)
- moved C19 3.07 mm to (212.4, 82.5)
- moved C21 3.07 mm to (245.6, 91.4)
- moved C22 3.07 mm to (238.0, 88.9)
- moved C24 3.07 mm to (231.5, 88.9)
- moved F10 3.07 mm to (204.7, 50.8)
- moved J17 3.07 mm to (246.1, 31.9)
- moved J20 3.07 mm to (216.5, 97.8)
- moved R36 3.07 mm to (217.7, 67.3)
- moved R37 3.07 mm to (243.1, 58.4)
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