File: karca.kicad_pcb (KiCad board)
At the start: 4 copper layers, 355.6 x 152.4 mm, 244 parts, among them J1 Conn_01x02_Female, J1 Screw_Terminal_01x02, J10 Screw_Terminal_01x02, J11 Screw_Terminal_01x02, J12 Conn_01x06_Female, J13 Screw_Terminal_01x04, J14 Screw_Terminal_01x04, J15 Screw_Terminal_01x04, J16 Screw_Terminal_01x04, J17 Screw_Terminal_01x04, J18 Screw_Terminal_01x04, J19 Conn_01x06_Female, J2 Screw_Terminal_01x02, J20 Conn_02x06_Odd_Even, J21 Screw_Terminal_01x02, J22 Screw_Terminal_01x02, J23 Screw_Terminal_01x02, J24 Screw_Terminal_01x02, J25 Conn_01x04_Female, J26 Screw_Terminal_01x03, J27 Screw_Terminal_01x03, J28 Screw_Terminal_01x03, J29 Screw_Terminal_01x03, J3 Screw_Terminal_01x02, J30 Conn_01x08_Female, J31 Conn_01x08_Female, J32 Conn_01x08_Female, J33 2540-5, J4 Screw_Terminal_01x02, J5 Conn_01x04_Female, J6 Screw_Terminal_01x02, J7 Screw_Terminal_01x02, J8 Screw_Terminal_01x02, J9 Screw_Terminal_01x02, Q1 FQP30N06, Q2 FQP30N06, Q3 FQP30N06, Q4 FQP30N06, Q5 FQP30N06, Q6 FQP30N06, SW1 1101M2S3CQE2, SW1 S101031MS02Q, SW2 1101M2S3CQE2, SW2 S101031MS02Q, U1 LM1084-ADJ, U10 LM324DT, U11 LM324DT, U12 MCP3208-CI/SL, U13 MCP3208-CI/SL, U14 MCP3208-CI/SL, U2 LM1084-5.0, U3 MCP6N11T-001E, U4 MCP6N11T-001E, U5 MCP6N11T-001E, U6 MCP6N11T-001E, U7 MCP6N11T-001E, U8 MCP6N11T-001E, U9 LM324DT

Commit message: positioning for LC connectors
Parts:
- added REF**: MountingHole_3.2mm_M3, MountingHole:MountingHole_3.2mm_M3, F.Cu at (30.5, 30.5)
- added REF**: MountingHole_3.2mm_M3, MountingHole:MountingHole_3.2mm_M3, F.Cu at (203.2, 172.7)
- added REF**: MountingHole_3.2mm_M3, MountingHole:MountingHole_3.2mm_M3, F.Cu at (30.5, 172.7)
- added REF**: MountingHole_3.2mm_M3, MountingHole:MountingHole_3.2mm_M3, F.Cu at (203.2, 30.5)
- U3, U4, U5, U6, U7, U8: value MCP6N11T-001E -> MCP6N11; footprint Package_DFN_QFN:TDFN-8-1EP_3x2mm_P0.5mm_EP1.80x1.65mm -> Package_SO:SOIC-8_3.9x4.9mm_P1.27mm
- moved RV6 236.4 mm to (38.1, 81.3)
- moved R41 233.3 mm to (40.6, 73.7)
- moved U8 229.2 mm to (43.2, 61.0), turned to -90 degrees
- moved CON_LC6 225.1 mm to (48.3, 38.1)
- moved R38 217.9 mm to (45.7, 73.7)
- moved C9 216.4 mm to (45.7, 68.6)
- moved J32 210.9 mm to (-54.3, 34.2), turned to 90 degrees
- moved F12 203.6 mm to (55.9, 63.5)
- moved R88 199.1 mm to (-55.9, 43.2), turned to 90 degrees
- moved U14 192.3 mm to (-45.7, 45.7), turned to 90 degrees
- moved RV5 183.1 mm to (63.5, 81.3)
- moved C36 180.8 mm to (-53.3, 55.9), turned to 90 degrees
- moved R40 177.3 mm to (66.0, 73.7)
- moved R37 172.7 mm to (71.1, 73.7)
- moved CON_LC5 172.6 mm to (73.7, 38.1)
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- renumbered J13 to CON_LC1, J14 to CON_LC2, J15 to CON_LC3, J16 to CON_LC4, J17 to CON_LC5, J18 to CON_LC6
Routing:
- net (no net): vias 6 -> 0

Commit message: complete arrangement for load cells
Parts:
- removed R86, R87, R88: 100k, Resistor_SMD:R_1206_3216Metric
- added J13: Conn_01x02_Female, Connector_PinHeader_2.54mm:PinHeader_1x02_P2.54mm_Vertical, F.Cu at (62.2, 94.0)
- moved F17 349.2 mm to (264.2, 63.5)
- moved J26 349.2 mm to (259.1, 38.1)
- moved J27 349.2 mm to (279.4, 38.1)
- moved F18 346.6 mm to (284.5, 63.5)
- moved J32 322.8 mm to (265.4, 78.8), turned to -90 degrees
- moved C36 317.5 mm to (261.6, 96.5), turned to 0 degrees
- moved U14 305.3 mm to (256.6, 88.9), turned to -90 degrees
- moved J28 269.0 mm to (238.8, 38.1)
- moved J29 269.0 mm to (218.4, 38.1)
- moved F20 266.5 mm to (223.5, 63.5)
- moved F19 264.0 mm to (243.8, 63.5)
- moved C20 242.0 mm to (40.6, 101.5), turned to -90 degrees
- moved R62 239.6 mm to (43.2, 106.6)
- moved R64 231.9 mm to (50.8, 106.6)
- moved R58 229.9 mm to (48.3, 94.0), turned to -90 degrees
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Connections:
- J19 pad 5: LC5_PREC -> (no net)
- J19 pad 6: LC6_PREC -> (no net)

Commit message: laid out ignition and PTs
Parts:
- removed J1: Conn_01x02_Female, Connector_PinHeader_2.54mm:PinHeader_1x02_P2.54mm_Vertical
- removed the SW1 at (139.7, 195.6)
- removed the SW2 at (306.1, 128.3)
- added H3: MountingHole_2.2mm_M2, MountingHole:MountingHole_2.2mm_M2, F.Cu at (363.2, 30.5)
- added H6: MountingHole_2.2mm_M2, MountingHole:MountingHole_2.2mm_M2, F.Cu at (363.2, 185.4)
- D10, D11, D12, D13, D14, D15, D16, D2, D22, D23, D24, D3, D4, D5, D6, D7, D8, D9: value SS54 -> DO-214AC
- moved D8 257.2 mm to (83.9, 118.0), turned to 90 degrees
- moved D2 255.1 mm to (78.8, 118.0), turned to 90 degrees
- moved D9 234.8 mm to (100.4, 139.6), turned to 90 degrees
- moved D6 231.7 mm to (95.3, 142.1), turned to 90 degrees
- moved J12 230.8 mm to (248.9, 144.8), turned to 180 degrees
- moved D7 224.6 mm to (110.6, 134.5), turned to 90 degrees
- moved D4 221.6 mm to (105.5, 137.0), turned to 90 degrees
- moved R27 181.0 mm to (289.6, 86.4)
- moved F1 180.4 mm to (307.3, 175.3)
- moved D10 179.7 mm to (195.6, 119.3), turned to 90 degrees
- moved D11 177.0 mm to (185.4, 124.4), turned to 90 degrees
- moved D16 176.1 mm to (190.8, 121.9), turned to 90 degrees
- moved R15 176.1 mm to (289.6, 167.6), turned to 180 degrees
- moved D12 175.0 mm to (200.7, 116.8), turned to 90 degrees
- moved FS_STAT_1 172.3 mm to (317.5, 182.9), turned to 180 degrees
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- renumbered J1 to CON_BAT1, J6 to CON_DRV1, J7 to CON_DRV2, J8 to CON_DRV3, J9 to CON_DRV4, J10 to CON_DRV5, J11 to CON_DRV6, J2 to CON_FAN1, J4 to CON_IGN_12, J22 to CON_PT1, J21 to CON_PT2, J23 to CON_PT3, J24 to CON_PT4, J3 to CON_ROUTER1, J26 to CON_TC1, J27 to CON_TC2, J28 to CON_TC3, J29 to CON_TC4, REF** to H1, REF** to H2, REF** to H4, REF** to H5
Routing:
- net LC4_CAL: track 0.00 -> 28.6 mm
- net LC3_CAL: track 0.00 -> 24.0 mm
- net LC6_CAL: track 0.00 -> 21.8 mm
- net LC2_CAL: track 0.00 -> 19.5 mm
- net Net-(C24-Pad1): track 0.00 -> 18.0 mm
- net LC1_CAL: track 0.00 -> 14.9 mm
- net Net-(C22-Pad1): track 0.00 -> 12.3 mm
- net Net-(C23-Pad1): track 0.00 -> 10.3 mm
- net +10V: track 0.00 -> 8.69 mm
- net LC5_CAL: track 0.00 -> 7.93 mm
Other:
- board size 355.6 x 152.4 mm -> 342.9 x 165.1 mm

Commit message: nearly done with part layout
Parts:
- moved C36 135.2 mm to (58.4, 157.5)
- moved J32 135.2 mm to (78.7, 160.0)
- moved U14 135.2 mm to (68.6, 152.4)
- moved D4 124.9 mm to (132.1, 259.1), turned to 180 degrees
- moved D7 124.7 mm to (106.7, 259.1), turned to 0 degrees
- moved D16 124.1 mm to (81.3, 180.3)
- moved D10 123.9 mm to (86.4, 177.8)
- moved D12 123.9 mm to (91.4, 175.3)
- moved D11 123.9 mm to (76.2, 182.9)
- moved C35 123.9 mm to (50.8, 177.8)
- moved J31 123.9 mm to (71.1, 180.3)
- moved U13 123.9 mm to (61.0, 172.7)
- moved R4 94.0 mm to (121.9, 183.7), turned to 180 degrees
- moved U1 93.9 mm to (134.6, 171.0)
- moved LED_12V1 90.1 mm to (231.1, 167.6), turned to 90 degrees
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Connections:
- net /Raspberry Pi/HBT renamed Net-(J33-Pad29)
Routing:
- net LC4_CAL: track 28.6 -> 1.91 mm
- net LC3_CAL: track 24.0 -> 0.00 mm
- net LC2_CAL: track 19.5 -> 0.00 mm
- net LC6_CAL: track 21.8 -> 6.59 mm
- net LC1_CAL: track 14.9 -> 1.03 mm
- net Net-(C20-Pad1): track 0.00 -> 12.3 mm
- net Net-(C23-Pad1): track 10.3 -> 18.0 mm
- net Net-(R63-Pad2): track 0.00 -> 4.70 mm
- net Net-(R62-Pad2): track 0.00 -> 4.70 mm
- net LC5_PREC: track 0.00 -> 2.16 mm
- removed copper zone on B.Cu, net +10V
- removed copper zone on B.Cu, net +12V
- removed copper zone on B.Cu, net +5V

Commit message: finish putting shit together
Parts:
- removed F10, F11, F12, F13, F14, F15, F16, F17, F18, F19, F20, F7, F8, F9: 178.6165, 178.6165:17861650002
- moved D4 155.6 mm to (81.3, 112.0)
- moved D7 144.4 mm to (81.2, 117.0), turned to 180 degrees
- moved D6 95.8 mm to (81.2, 127.1)
- moved D9 89.9 mm to (81.2, 122.1), turned to 180 degrees
- moved D8 45.6 mm to (38.1, 101.6)
- moved J25 26.2 mm to (279.4, 72.4)
- moved J33 26.0 mm to (38.7, 139.7)
- moved D2 22.8 mm to (88.9, 101.6)
- moved D12 20.5 mm to (81.3, 157.5), turned to 180 degrees
- moved C34 20.2 mm to (50.8, 124.5)
- moved U12 19.8 mm to (61.0, 119.4)
- moved J30 19.8 mm to (71.1, 128.3)
- moved R67 18.3 mm to (231.1, 101.6)
- moved C25 18.3 mm to (238.8, 101.6)
- moved C26 18.3 mm to (198.1, 101.6)
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Connections:
- CON_LC1 pad 1: Net-(CON_LC1-Pad1) -> +5V
- CON_LC2 pad 1: Net-(CON_LC2-Pad1) -> +5V
- CON_LC3 pad 1: Net-(CON_LC3-Pad1) -> +5V
- CON_LC4 pad 1: Net-(CON_LC4-Pad1) -> +5V
- CON_LC5 pad 1: Net-(CON_LC5-Pad1) -> +5V
- CON_LC6 pad 1: Net-(CON_LC6-Pad1) -> +5V
- CON_PT1 pad 1: /PT Amplification/PT1+ -> +10V
- CON_PT2 pad 1: /PT Amplification/PT2+ -> +10V
- CON_PT3 pad 1: /PT Amplification/PT3+ -> +10V
- CON_PT4 pad 1: /PT Amplification/PT4+ -> +10V
- CON_TC1 pad 1: Net-(CON_TC1-Pad1) -> +5V
- CON_TC2 pad 1: Net-(CON_TC2-Pad1) -> +5V
- CON_TC3 pad 1: Net-(CON_TC3-Pad1) -> +5V
Routing:
- net Net-(C24-Pad1): track 18.0 -> 0.00 mm
- net Net-(C23-Pad1): track 18.0 -> 0.00 mm
- net Net-(C22-Pad1): track 12.3 -> 0.00 mm
- net Net-(C20-Pad1): track 12.3 -> 0.00 mm
- net +10V: track 8.69 -> 0.00 mm
- net LC5_CAL: track 7.51 -> 0.00 mm
- net LC6_CAL: track 6.59 -> 0.00 mm
- net Net-(R63-Pad2): track 4.70 -> 0.00 mm
- net Net-(R62-Pad2): track 4.70 -> 0.00 mm
- net LC5_PREC: track 2.16 -> 0.00 mm
- net LC4_CAL: track 1.91 -> 0.00 mm
- net LC1_CAL: track 1.03 -> 0.00 mm
- removed copper zone on In1.Cu, net GND
Other:
- board size 342.9 x 165.1 mm -> 342.9 x 152.4 mm

Commit message: copper pours done
Connections:
- CON_TC4 pad 1: Net-(CON_TC4-Pad1) -> +5V
- RV1 pad 1: +5V -> +10V
- RV2 pad 1: +5V -> +10V
- RV3 pad 1: +5V -> +10V
- RV4 pad 1: +5V -> +10V
- RV5 pad 1: +5V -> +10V
- RV6 pad 1: +5V -> +10V
Routing:
- net /Drivers/DRV_NEG_1: track 0.00 -> 52.1 mm
- net /Drivers/DRV_POS_1: track 0.00 -> 33.2 mm
- added copper zone on In2.Cu, net +10V
- added copper zone on In2.Cu, net +12V
- added copper zone on In2.Cu, net +5V
