File: karca.kicad_pcb (KiCad board)
At the start: 4 copper layers, 342.9 x 152.4 mm, 231 parts, among them J12 Conn_01x06_Female, J13 Conn_01x02_Female, J19 Conn_01x06_Female, J20 Conn_02x06_Odd_Even, J25 Conn_01x04_Female, J30 Conn_01x08_Female, J31 Conn_01x08_Female, J32 Conn_01x08_Female, J33 2540-5, J5 Conn_01x04_Female, Q1 FQP30N06, Q2 FQP30N06, Q3 FQP30N06, Q4 FQP30N06, Q5 FQP30N06, Q6 FQP30N06, SW1 S101031MS02Q, SW2 S101031MS02Q, U1 LM1084-ADJ, U10 LM324DT, U11 LM324DT, U12 MCP3208-CI/SL, U13 MCP3208-CI/SL, U14 MCP3208-CI/SL, U2 LM1084-5.0, U3 MCP6N11, U4 MCP6N11, U5 MCP6N11, U6 MCP6N11, U7 MCP6N11, U8 MCP6N11, U9 LM324DT

Commit message: starting on routing
Parts:
- moved C11 15.2 mm to (149.9, 88.9)
- moved C13 15.2 mm to (149.9, 104.1)
- moved C15 15.2 mm to (124.5, 88.9)
- moved C18 15.2 mm to (124.5, 104.1)
- moved FS_STAT_1 2.54 mm to (317.5, 172.7)
- moved LED_10V1 0.21 mm to (147.3, 153.7)
- moved R3 0.21 mm to (154.9, 153.7), turned to 0 degrees
- moved C12 0.07 mm to (149.9, 129.5)
- moved C14 0.07 mm to (149.9, 114.3)
- moved R43 0.07 mm to (149.9, 96.5)
- moved R45 0.07 mm to (149.9, 121.9)
- moved C16 0.06 mm to (124.5, 129.5)
- moved C19 0.06 mm to (124.5, 114.3)
- moved R53 0.06 mm to (124.5, 121.9)
- moved R54 0.06 mm to (132.1, 91.4)
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Connections:
- net Net-(CON_FAN1-Pad1) renamed /regulators/FAN_PWR
- net Net-(D1-Pad2) renamed /regulators/12V_PRERECT
Routing:
- net /PT Amplification/PT1-: track 0.00 -> 186.9 mm
- net /PT Amplification/PT2-: track 0.00 -> 146.2 mm
- net /PT Amplification/PT4-: track 0.00 -> 110.2 mm
- net /PT Amplification/PT3-: track 0.00 -> 105.5 mm
- net DRV_CTL_1: track 0.00 -> 81.7 mm
- net DRV_CTL_3: track 0.00 -> 78.1 mm
- net DRV_CTL_2: track 0.00 -> 74.3 mm
- net /Drivers/DRV_POS_4: track 0.00 -> 69.1 mm
- net /Drivers/DRV_POS_2: track 0.00 -> 69.1 mm
- net /Drivers/DRV_POS_5: track 0.00 -> 67.0 mm
- net /Drivers/DRV_POS_6: track 0.00 -> 64.4 mm
- net /Drivers/DRV_POS_3: track 0.00 -> 62.8 mm
- net /Drivers/DRV_NEG_5: track 0.00 -> 59.9 mm
- net /Drivers/DRV_NEG_2: track 0.00 -> 58.3 mm
- net /Drivers/DRV_NEG_4: track 0.00 -> 57.1 mm
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- added copper zone on In1.Cu, net GND
