File: pt_amps.kicad_sch (KiCad schematic)
At the start: 39 parts, among them J21 Screw_Terminal_01x02, J22 Screw_Terminal_01x02, J23 Screw_Terminal_01x02, J24 Screw_Terminal_01x02, J25 Conn_01x04_Female, U11 LM324DT

Commit message: some minor schematic cleanup
Parts:
- C25, C26, C27, C28, C29, C30, C31, C32: value 1nF -> 1n
- C33: value 100nF -> 100n
Connections:
- net PT3+: now reaches F15.2, J23.1 (Pin_1)
- net PT1+: now reaches F14.2, J22.1 (Pin_1)
- net PT2+: now reaches F13.2, J21.1 (Pin_1)
- net PT4+: now reaches F16.2, J24.1 (Pin_1)
Changed lines of the file:
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@@
+    (effects (font (size 1.27 1.27)) (justify left bottom))
+  )
+  (label "PT2+" (at 149.86 44.45 0)
     (effects (font (size 1.27 1.27)) (justify left bottom))
   )
@@
     (effects (font (size 1.27 1.27)) (justify left bottom))
   )
+  (label "PT4+" (at 148.59 106.68 0)
+    (effects (font (size 1.27 1.27)) (justify left bottom))
+  )
   (label "PT1-" (at 34.29 49.53 0)
     (effects (font (size 1.27 1.27)) (justify left bottom))
   )
+  (label "PT3+" (at 34.29 105.41 0)
+    (effects (font (size 1.27 1.27)) (justify left bottom))
+  )
   (label "PT2-" (at 149.86 48.26 0)
     (effects (font (size 1.27 1.27)) (justify left bottom))
   )
   (label "PT3-" (at 34.29 109.22 0)
+    (effects (font (size 1.27 1.27)) (justify left bottom))
+  )
+  (label "PT1+" (at 34.29 45.72 0)
     (effects (font (size 1.27 1.27)) (justify left bottom))
   )
@@
       (effects (font (size 1.27 1.27)) hide)
     )
-    (property "Datasheet" "https://media.digikey.com/pdf/Data%20Sheets/Rohm%20PDFs/LM358,LM324,LM2904,LM2902.pdf" (id 3) (at 81.28 46.99 0)
+    (property "Datasheet" "http://www.ti.com/lit/ds/symlink/lm2902-n.pdf" (id 3) (at 81.28 46.99 0)
       (effects (font (size 1.27 1.27)) hide)
     )
@@
       (effects (font (size 1.27 1.27)) (justify left))
     )
-    (property "Value" "1nF" (id 1) (at 66.04 59.6899 0)
+    (property "Value" "1n" (id 1) (at 66.04 59.6899 0)
       (effects (font (size 1.27 1.27)) (justify left))
     )
@@
       (effects (font (size 1.27 1.27)) hide)
     )
-    (property "Datasheet" "https://media.digikey.com/pdf/Data%20Sheets/Rohm%20PDFs/LM358,LM324,LM2904,LM2902.pdf" (id 3) (at 78.74 161.29 0)
+    (property "Datasheet" "http://www.ti.com/lit/ds/symlink/lm2902-n.pdf" (id 3) (at 78.74 161.29 0)
       (effects (font (size 1.27 1.27)) hide)
     )
@@
       (effects (font (size 1.27 1.27)) hide)
     )
-    (property "Datasheet" "https://media.digikey.com/pdf/Data%20Sheets/Rohm%20PDFs/LM358,LM324,LM2904,LM2902.pdf" (id 3) (at 81.28 106.68 0)
+    (property "Datasheet" "http://www.ti.com/lit/ds/symlink/lm2902-n.pdf" (id 3) (at 81.28 106.68 0)
       (effects (font (size 1.27 1.27)) hide)
     )
@@
     (in_bom yes) (on_board yes) (fields_autoplaced)
     (property "Reference" "C26" (id 0) (at 64.77 31.75 90))
-    (property "Value" "1nF" (id 1) (at 64.77 34.29 90))
+    (property "Value" "1n" (id 1) (at 64.77 34.29 90))
     (property "Footprint" "Capacitor_SMD:C_1206_3216Metric" (id 2) (at 68.58 38.4048 0)
       (effects (font (size 1.27 1.27)) hide)
@@
       (effects (font (size 1.27 1.27)) hide)
     )
-    (property "Datasheet" "https://www.phoenixcontact.com/en-us/products/printed-circuit-board-terminal-lpta-25-2-50-1190363" (id 3) (at 29.21 106.68 0)
+    (property "Datasheet" "~" (id 3) (at 29.21 106.68 0)
       (effects (font (size 1.27 1.27)) hide)
     )
@@
       (effects (font (size 1.27 1.27)) hide)
     )
-    (property "Datasheet" "https://www.mouser.com/datasheet/2/215/588-20-1622270.pdf" (id 3) (at 34.29 39.37 0)
+    (property "Datasheet" "~" (id 3) (at 34.29 39.37 0)
       (effects (font (size 1.27 1.27)) hide)
     )
@@
       (effects (font (size 1.27 1.27)) hide)
     )
-    (property "Datasheet" "https://www.phoenixcontact.com/en-us/products/printed-circuit-board-terminal-lpta-25-2-50-1190363" (id 3) (at 29.21 46.99 0)
+    (property "Datasheet" "~" (id 3) (at 29.21 46.99 0)
       (effects (font (size 1.27 1.27)) hide)
     )
@@
       (effects (font (size 1.27 1.27)) (justify left))
     )
-    (property "Value" "1nF" (id 1) (at 66.04 119.3799 0)
+    (property "Value" "1n" (id 1) (at 66.04 119.3799 0)
       (effects (font (size 1.27 1.27)) (justify left))
     )
@@
       (effects (font (size 1.27 1.27)) hide)
     )
-    (property "Datasheet" "https://media.digikey.com/pdf/Data%20Sheets/Rohm%20PDFs/LM358,LM324,LM2904,LM2902.pdf" (id 3) (at 195.58 107.95 0)
+    (property "Datasheet" "http://www.ti.com/lit/ds/symlink/lm2902-n.pdf" (id 3) (at 195.58 107.95 0)
       (effects (font (size 1.27 1.27)) hide)
     )
@@
       (effects (font (size 1.27 1.27)) hide)
     )
-    (property "Datasheet" "https://www.phoenixcontact.com/en-us/products/printed-circuit-board-terminal-lpta-25-2-50-1190363" (id 3) (at 144.78 45.72 0)
+    (property "Datasheet" "~" (id 3) (at 144.78 45.72 0)
       (effects (font (size 1.27 1.27)) hide)
     )
@@
       (effects (font (size 1.27 1.27)) hide)
     )
-    (property "Datasheet" "https://www.mouser.com/datasheet/2/215/588-20-1622270.pdf" (id 3) (at 149.86 38.1 0)
+    (property "Datasheet" "~" (id 3) (at 149.86 38.1 0)
       (effects (font (size 1.27 1.27)) hide)
     )
@@
       (effects (font (size 1.27 1.27)) hide)
     )
-    (property "Datasheet" "https://www.phoenixcontact.com/en-us/products/printed-circuit-board-terminal-lpta-25-2-50-1190363" (id 3) (at 143.51 107.95 0)
+    (property "Datasheet" "~" (id 3) (at 143.51 107.95 0)
       (effects (font (size 1.27 1.27)) hide)
     )
@@
       (effects (font (size 1.27 1.27)) hide)
     )
-    (property "Datasheet" "https://www.mouser.com/datasheet/2/215/588-20-1622270.pdf" (id 3) (at 34.29 99.06 0)
+    (property "Datasheet" "~" (id 3) (at 34.29 99.06 0)
       (effects (font (size 1.27 1.27)) hide)
     )
@@
       (effects (font (size 1.27 1.27)) (justify left))
     )
-    (property "Value" "1nF" (id 1) (at 181.61 58.4199 0)
+    (property "Value" "1n" (id 1) (at 181.61 58.4199 0)
       (effects (font (size 1.27 1.27)) (justify left))
     )
@@
     (in_bom yes) (on_board yes) (fields_autoplaced)
     (property "Reference" "C30" (id 0) (at 179.07 92.71 90))
-    (property "Value" "1nF" (id 1) (at 179.07 95.25 90))
+    (property "Value" "1n" (id 1) (at 179.07 95.25 90))
     (property "Footprint" "Capacitor_SMD:C_1206_3216Metric" (id 2) (at 182.88 99.3648 0)
       (effects (font (size 1.27 1.27)) hide)
@@
       (effects (font (size 1.27 1.27)) (justify left))
     )
-    (property "Value" "100nF" (id 1) (at 55.88 167.64 0)
+    (property "Value" "100n" (id 1) (at 55.88 167.64 0)
       (effects (font (size 1.27 1.27)) (justify left))
     )
@@
       (effects (font (size 1.27 1.27)) (justify left))
     )
-    (property "Value" "1nF" (id 1) (at 180.34 120.6499 0)
+    (property "Value" "1n" (id 1) (at 180.34 120.6499 0)
       (effects (font (size 1.27 1.27)) (justify left))
     )
@@
     (in_bom yes) (on_board yes) (fields_autoplaced)
     (property "Reference" "C29" (id 0) (at 64.77 91.44 90))
-    (property "Value" "1nF" (id 1) (at 64.77 93.98 90))
+    (property "Value" "1n" (id 1) (at 64.77 93.98 90))
     (property "Footprint" "Capacitor_SMD:C_1206_3216Metric" (id 2) (at 68.58 98.0948 0)
       (effects (font (size 1.27 1.27)) hide)
@@
       (effects (font (size 1.27 1.27)) hide)
     )
-    (property "Datasheet" "https://www.mouser.com/datasheet/2/215/588-20-1622270.pdf" (id 3) (at 148.59 100.33 0)
+    (property "Datasheet" "~" (id 3) (at 148.59 100.33 0)
       (effects (font (size 1.27 1.27)) hide)
     )
@@
     (in_bom yes) (on_board yes) (fields_autoplaced)
     (property "Reference" "C25" (id 0) (at 180.34 30.48 90))
-    (property "Value" "1nF" (id 1) (at 180.34 33.02 90))
+    (property "Value" "1n" (id 1) (at 180.34 33.02 90))
     (property "Footprint" "Capacitor_SMD:C_1206_3216Metric" (id 2) (at 184.15 37.1348 0)
       (effects (font (size 1.27 1.27)) hide)
@@
       (effects (font (size 1.27 1.27)) hide)
     )
-    (property "Datasheet" "https://media.digikey.com/pdf/Data%20Sheets/Rohm%20PDFs/LM358,LM324,LM2904,LM2902.pdf" (id 3) (at 196.85 45.72 0)
-      (effects (font (size 1.27 1.27)) hide)
-    )
+    (property "Datasheet" "http://www.ti.com/lit/ds/symlink/lm2902-n.pdf" (id 3) (at 196.85 45.72 0)
+      (effects (font (size 1.27 1.27)) hide)
+    )

Commit message: shuffle around some parts
Parts:
- F13, F14, F15, F16: value 3588-20 -> 178.6165; footprint 3588-20:358820 -> 178.6165:17861650002
Changed lines of the file:
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@@
       (effects (font (size 1.27 1.27)) (justify left))
     )
-    (property "Value" "3588-20" (id 1) (at 36.83 40.6399 0)
-      (effects (font (size 1.27 1.27)) (justify left))
-    )
-    (property "Footprint" "3588-20:358820" (id 2) (at 32.512 39.37 90)
+    (property "Value" "178.6165" (id 1) (at 36.83 40.6399 0)
+      (effects (font (size 1.27 1.27)) (justify left))
+    )
+    (property "Footprint" "178.6165:17861650002" (id 2) (at 32.512 39.37 90)
       (effects (font (size 1.27 1.27)) hide)
     )
@@
       (effects (font (size 1.27 1.27)) (justify left))
     )
-    (property "Value" "3588-20" (id 1) (at 152.4 39.3699 0)
-      (effects (font (size 1.27 1.27)) (justify left))
-    )
-    (property "Footprint" "3588-20:358820" (id 2) (at 148.082 38.1 90)
+    (property "Value" "178.6165" (id 1) (at 152.4 39.3699 0)
+      (effects (font (size 1.27 1.27)) (justify left))
+    )
+    (property "Footprint" "178.6165:17861650002" (id 2) (at 148.082 38.1 90)
       (effects (font (size 1.27 1.27)) hide)
     )
@@
       (effects (font (size 1.27 1.27)) (justify left))
     )
-    (property "Value" "3588-20" (id 1) (at 36.83 100.3299 0)
-      (effects (font (size 1.27 1.27)) (justify left))
-    )
-    (property "Footprint" "3588-20:358820" (id 2) (at 32.512 99.06 90)
+    (property "Value" "178.6165" (id 1) (at 36.83 100.3299 0)
+      (effects (font (size 1.27 1.27)) (justify left))
+    )
+    (property "Footprint" "178.6165:17861650002" (id 2) (at 32.512 99.06 90)
       (effects (font (size 1.27 1.27)) hide)
     )
@@
       (effects (font (size 1.27 1.27)) (justify left))
     )
-    (property "Value" "3588-20" (id 1) (at 151.13 101.5999 0)
-      (effects (font (size 1.27 1.27)) (justify left))
-    )
-    (property "Footprint" "3588-20:358820" (id 2) (at 146.812 100.33 90)
-      (effects (font (size 1.27 1.27)) hide)
-    )
+    (property "Value" "178.6165" (id 1) (at 151.13 101.5999 0)
+      (effects (font (size 1.27 1.27)) (justify left))
+    )
+    (property "Footprint" "178.6165:17861650002" (id 2) (at 146.812 100.33 90)
+      (effects (font (size 1.27 1.27)) hide)
+    )
