File: pt_amps.kicad_sch (KiCad schematic)
At the start: 43 parts, among them J21 Screw_Terminal_01x02, J22 Screw_Terminal_01x02, J23 Screw_Terminal_01x02, J24 Screw_Terminal_01x02, J25 Conn_01x04_Female, U11 LM324DT

Commit message: laid out ignition and PTs
Parts:
- D10, D11, D12, D16: value SS54 -> DO-214AC
- renumbered J22 to CON_PT1, J21 to CON_PT2, J23 to CON_PT3, J24 to CON_PT4
Changed lines of the file:
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@@
       (effects (font (size 1.27 1.27)) (justify left))
     )
-    (property "Value" "SS54" (id 1) (at 104.14 49.2124 90)
+    (property "Value" "DO-214AC" (id 1) (at 104.14 49.2124 90)
       (effects (font (size 1.27 1.27)) (justify left))
     )
@@
   (symbol (lib_id "Connector:Screw_Terminal_01x02") (at 29.21 106.68 0) (mirror y) (unit 1)
     (in_bom yes) (on_board yes)
-    (property "Reference" "J23" (id 0) (at 26.67 107.9499 0)
+    (property "Reference" "CON_PT3" (id 0) (at 26.67 107.9499 0)
       (effects (font (size 1.27 1.27)) (justify left))
     )
@@
       (effects (font (size 1.27 1.27)) (justify left))
     )
-    (property "Value" "SS54" (id 1) (at 218.44 47.9424 90)
+    (property "Value" "DO-214AC" (id 1) (at 218.44 47.9424 90)
       (effects (font (size 1.27 1.27)) (justify left))
     )
@@
   (symbol (lib_id "Connector:Screw_Terminal_01x02") (at 29.21 46.99 0) (mirror y) (unit 1)
     (in_bom yes) (on_board yes)
-    (property "Reference" "J22" (id 0) (at 26.67 48.2599 0)
+    (property "Reference" "CON_PT1" (id 0) (at 26.67 48.2599 0)
       (effects (font (size 1.27 1.27)) (justify left))
     )
@@
       (effects (font (size 1.27 1.27)) (justify left))
     )
-    (property "Value" "SS54" (id 1) (at 217.17 110.1724 90)
+    (property "Value" "DO-214AC" (id 1) (at 217.17 110.1724 90)
       (effects (font (size 1.27 1.27)) (justify left))
     )
@@
   (symbol (lib_id "Connector:Screw_Terminal_01x02") (at 144.78 45.72 0) (mirror y) (unit 1)
     (in_bom yes) (on_board yes)
-    (property "Reference" "J21" (id 0) (at 142.24 46.9899 0)
+    (property "Reference" "CON_PT2" (id 0) (at 142.24 46.9899 0)
       (effects (font (size 1.27 1.27)) (justify left))
     )
@@
   (symbol (lib_id "Connector:Screw_Terminal_01x02") (at 143.51 107.95 0) (mirror y) (unit 1)
     (in_bom yes) (on_board yes)
-    (property "Reference" "J24" (id 0) (at 140.97 109.2199 0)
+    (property "Reference" "CON_PT4" (id 0) (at 140.97 109.2199 0)
       (effects (font (size 1.27 1.27)) (justify left))
     )
@@
       (effects (font (size 1.27 1.27)) (justify left))
     )
-    (property "Value" "SS54" (id 1) (at 102.87 108.9024 90)
-      (effects (font (size 1.27 1.27)) (justify left))
-    )
+    (property "Value" "DO-214AC" (id 1) (at 102.87 108.9024 90)
+      (effects (font (size 1.27 1.27)) (justify left))
+    )

Commit message: finish putting shit together
Parts:
- removed F13, F14, F15, F16: 178.6165, 178.6165:17861650002, symbol Device:Fuse
Connections:
- net PT1+ is gone; now on net +10V: CON_PT1.1 (Pin_1)
- net PT2+ is gone; now on net +10V: CON_PT2.1 (Pin_1)
- net PT3+ is gone; now on net +10V: CON_PT3.1 (Pin_1)
- net PT4+ is gone; now on net +10V: CON_PT4.1 (Pin_1)
Changed lines of the file:
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@@
-    (effects (font (size 1.27 1.27)) (justify left bottom))
-  )
-  (label "PT2+" (at 149.86 44.45 0)
     (effects (font (size 1.27 1.27)) (justify left bottom))
   )
@@
     (effects (font (size 1.27 1.27)) (justify left bottom))
   )
-  (label "PT4+" (at 148.59 106.68 0)
-    (effects (font (size 1.27 1.27)) (justify left bottom))
-  )
   (label "PT1-" (at 34.29 49.53 0)
     (effects (font (size 1.27 1.27)) (justify left bottom))
   )
-  (label "PT3+" (at 34.29 105.41 0)
-    (effects (font (size 1.27 1.27)) (justify left bottom))
-  )
   (label "PT2-" (at 149.86 48.26 0)
     (effects (font (size 1.27 1.27)) (justify left bottom))
   )
   (label "PT3-" (at 34.29 109.22 0)
-    (effects (font (size 1.27 1.27)) (justify left bottom))
-  )
-  (label "PT1+" (at 34.29 45.72 0)
     (effects (font (size 1.27 1.27)) (justify left bottom))
   )
@@
     (pin "4")
   )
-  (symbol (lib_id "power:+10V") (at 34.29 95.25 0) (unit 1)
-    (in_bom yes) (on_board yes) (fields_autoplaced)
-    (property "Reference" "#PWR0119" (id 0) (at 34.29 99.06 0)
-      (effects (font (size 1.27 1.27)) hide)
-    )
-    (property "Value" "+10V" (id 1) (at 34.29 90.17 0))
-    (property "Footprint" "" (id 2) (at 34.29 95.25 0)
-      (effects (font (size 1.27 1.27)) hide)
-    )
-    (property "Datasheet" "" (id 3) (at 34.29 95.25 0)
+  (symbol (lib_id "power:+10V") (at 34.29 102.87 0) (unit 1)
+    (in_bom yes) (on_board yes) (fields_autoplaced)
+    (property "Reference" "#PWR0119" (id 0) (at 34.29 106.68 0)
+      (effects (font (size 1.27 1.27)) hide)
+    )
+    (property "Value" "+10V" (id 1) (at 34.29 97.79 0))
+    (property "Footprint" "" (id 2) (at 34.29 102.87 0)
+      (effects (font (size 1.27 1.27)) hide)
+    )
+    (property "Datasheet" "" (id 3) (at 34.29 102.87 0)
       (effects (font (size 1.27 1.27)) hide)
     )
@@
     (pin "2")
   )
-  (symbol (lib_id "power:+10V") (at 148.59 96.52 0) (unit 1)
-    (in_bom yes) (on_board yes) (fields_autoplaced)
-    (property "Reference" "#PWR0120" (id 0) (at 148.59 100.33 0)
-      (effects (font (size 1.27 1.27)) hide)
-    )
-    (property "Value" "+10V" (id 1) (at 148.59 91.44 0))
-    (property "Footprint" "" (id 2) (at 148.59 96.52 0)
-      (effects (font (size 1.27 1.27)) hide)
-    )
-    (property "Datasheet" "" (id 3) (at 148.59 96.52 0)
+  (symbol (lib_id "power:+10V") (at 148.59 104.14 0) (unit 1)
+    (in_bom yes) (on_board yes) (fields_autoplaced)
+    (property "Reference" "#PWR0120" (id 0) (at 148.59 107.95 0)
+      (effects (font (size 1.27 1.27)) hide)
+    )
+    (property "Value" "+10V" (id 1) (at 148.59 99.06 0))
+    (property "Footprint" "" (id 2) (at 148.59 104.14 0)
+      (effects (font (size 1.27 1.27)) hide)
+    )
+    (property "Datasheet" "" (id 3) (at 148.59 104.14 0)
       (effects (font (size 1.27 1.27)) hide)
     )
@@
     )
     (property "Datasheet" "~" (id 3) (at 95.25 57.15 0)
-      (effects (font (size 1.27 1.27)) hide)
-    )
-    (pin "1")
-    (pin "2")
-  )
-  (symbol (lib_id "Device:Fuse") (at 34.29 39.37 0) (unit 1)
-    (in_bom yes) (on_board yes) (fields_autoplaced)
-    (property "Reference" "F14" (id 0) (at 36.83 38.0999 0)
-      (effects (font (size 1.27 1.27)) (justify left))
-    )
-    (property "Value" "178.6165" (id 1) (at 36.83 40.6399 0)
-      (effects (font (size 1.27 1.27)) (justify left))
-    )
-    (property "Footprint" "178.6165:17861650002" (id 2) (at 32.512 39.37 90)
-      (effects (font (size 1.27 1.27)) hide)
-    )
-    (property "Datasheet" "~" (id 3) (at 34.29 39.37 0)
       (effects (font (size 1.27 1.27)) hide)
     )
@@
     (pin "1")
   )
-  (symbol (lib_id "Device:Fuse") (at 149.86 38.1 0) (unit 1)
-    (in_bom yes) (on_board yes) (fields_autoplaced)
-    (property "Reference" "F13" (id 0) (at 152.4 36.8299 0)
-      (effects (font (size 1.27 1.27)) (justify left))
-    )
-    (property "Value" "178.6165" (id 1) (at 152.4 39.3699 0)
-      (effects (font (size 1.27 1.27)) (justify left))
-    )
-    (property "Footprint" "178.6165:17861650002" (id 2) (at 148.082 38.1 90)
-      (effects (font (size 1.27 1.27)) hide)
-    )
-    (property "Datasheet" "~" (id 3) (at 149.86 38.1 0)
-      (effects (font (size 1.27 1.27)) hide)
-    )
-    (pin "1")
-    (pin "2")
-  )
   (symbol (lib_id "Device:R_US") (at 209.55 129.54 0) (unit 1)
     (in_bom yes) (on_board yes) (fields_autoplaced)
@@
     (pin "2")
   )
-  (symbol (lib_id "Device:Fuse") (at 34.29 99.06 0) (unit 1)
-    (in_bom yes) (on_board yes) (fields_autoplaced)
-    (property "Reference" "F15" (id 0) (at 36.83 97.7899 0)
-      (effects (font (size 1.27 1.27)) (justify left))
-    )
-    (property "Value" "178.6165" (id 1) (at 36.83 100.3299 0)
-      (effects (font (size 1.27 1.27)) (justify left))
-    )
-    (property "Footprint" "178.6165:17861650002" (id 2) (at 32.512 99.06 90)
-      (effects (font (size 1.27 1.27)) hide)
-    )
-    (property "Datasheet" "~" (id 3) (at 34.29 99.06 0)
-      (effects (font (size 1.27 1.27)) hide)
-    )
-    (pin "1")
-    (pin "2")
-  )
   (symbol (lib_id "Device:C") (at 177.8 57.15 0) (unit 1)
     (in_bom yes) (on_board yes) (fields_autoplaced)
@@
     (pin "2")
   )
-  (symbol (lib_id "power:+10V") (at 149.86 34.29 0) (unit 1)
-    (in_bom yes) (on_board yes) (fields_autoplaced)
-    (property "Reference" "#PWR0111" (id 0) (at 149.86 38.1 0)
-      (effects (font (size 1.27 1.27)) hide)
-    )
-    (property "Value" "+10V" (id 1) (at 149.86 29.21 0))
-    (property "Footprint" "" (id 2) (at 149.86 34.29 0)
-      (effects (font (size 1.27 1.27)) hide)
-    )
-    (property "Datasheet" "" (id 3) (at 149.86 34.29 0)
+  (symbol (lib_id "power:+10V") (at 149.86 41.91 0) (unit 1)
+    (in_bom yes) (on_board yes) (fields_autoplaced)
+    (property "Reference" "#PWR0111" (id 0) (at 149.86 45.72 0)
+      (effects (font (size 1.27 1.27)) hide)
+    )
+    (property "Value" "+10V" (id 1) (at 149.86 36.83 0))
+    (property "Footprint" "" (id 2) (at 149.86 41.91 0)
+      (effects (font (size 1.27 1.27)) hide)
+    )
+    (property "Datasheet" "" (id 3) (at 149.86 41.91 0)
       (effects (font (size 1.27 1.27)) hide)
     )
@@
     (pin "1")
   )
-  (symbol (lib_id "Device:Fuse") (at 148.59 100.33 0) (unit 1)
-    (in_bom yes) (on_board yes) (fields_autoplaced)
-    (property "Reference" "F16" (id 0) (at 151.13 99.0599 0)
-      (effects (font (size 1.27 1.27)) (justify left))
-    )
-    (property "Value" "178.6165" (id 1) (at 151.13 101.5999 0)
-      (effects (font (size 1.27 1.27)) (justify left))
-    )
-    (property "Footprint" "178.6165:17861650002" (id 2) (at 146.812 100.33 90)
-      (effects (font (size 1.27 1.27)) hide)
-    )
-    (property "Datasheet" "~" (id 3) (at 148.59 100.33 0)
-      (effects (font (size 1.27 1.27)) hide)
-    )
-    (pin "1")
-    (pin "2")
-  )
   (symbol (lib_id "Device:R_US") (at 34.29 57.15 180) (unit 1)
     (in_bom yes) (on_board yes) (fields_autoplaced)
@@
     (pin "2")
   )
-  (symbol (lib_id "power:+10V") (at 34.29 35.56 0) (unit 1)
-    (in_bom yes) (on_board yes) (fields_autoplaced)
-    (property "Reference" "#PWR0112" (id 0) (at 34.29 39.37 0)
-      (effects (font (size 1.27 1.27)) hide)
-    )
-    (property "Value" "+10V" (id 1) (at 34.29 30.48 0))
-    (property "Footprint" "" (id 2) (at 34.29 35.56 0)
-      (effects (font (size 1.27 1.27)) hide)
-    )
-    (property "Datasheet" "" (id 3) (at 34.29 35.56 0)
-      (effects (font (size 1.27 1.27)) hide)
-    )
+  (symbol (lib_id "power:+10V") (at 34.29 43.18 0) (unit 1)
+    (in_bom yes) (on_board yes) (fields_autoplaced)
+    (property "Reference" "#PWR0112" (id 0) (at 34.29 46.99 0)
+      (effects (font (size 1.27 1.27)) hide)
+    )
+    (property "Value" "+10V" (id 1) (at 34.29 38.1 0))
+    (property "Footprint" "" (id 2) (at 34.29 43.18 0)
+      (effects (font (size 1.27 1.27)) hide)
+    )
+    (property "Datasheet" "" (id 3) (at 34.29 43.18 0)
+      (effects (font (size 1.27 1.27)) hide)
+    )

Commit message: not sure if anything has changed but this is the last commit before moving to two LCs
Parts:
- J25: footprint Connector_PinHeader_2.54mm:PinHeader_1x04_P2.54mm_Vertical -> Connector_PinSocket_2.54mm:PinSocket_1x04_P2.54mm_Vertical
Changed lines of the file:
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@@
       (effects (font (size 1.27 1.27)) (justify left) hide)
     )
-    (property "Footprint" "Connector_PinHeader_2.54mm:PinHeader_1x04_P2.54mm_Vertical" (id 2) (at 127 163.83 0)
+    (property "Footprint" "Connector_PinSocket_2.54mm:PinSocket_1x04_P2.54mm_Vertical" (id 2) (at 127 163.83 0)
       (effects (font (size 1.27 1.27)) hide)
     )

Commit message: done schematiccing after design review
Parts:
- removed CON_PT1, CON_PT2, CON_PT3, CON_PT4: Screw_Terminal_01x02, 1190363:1190363, symbol Connector:Screw_Terminal_01x02
- removed J25: Conn_01x04_Female, Connector_PinSocket_2.54mm:PinSocket_1x04_P2.54mm_Vertical, symbol Connector:Conn_01x04_Female
- added ADC2: MCP3208-CI/SL, Package_SO:SOIC-16_3.9x9.9mm_P1.27mm, symbol Analog_ADC:MCP3208
- added C19: 100n, Capacitor_SMD:C_1206_3216Metric, symbol Device:C
- added D34, D35, D36, D37, D38, D39, D40, D41: CDBA340-HF, Diode_SMD:D_SMA, symbol Device:D_Schottky
- added J6: Screw_Terminal_01x08, symbol Connector:Screw_Terminal_01x08
- added J7: Conn_01x08_Female, Connector_PinSocket_2.54mm:PinSocket_1x08_P2.54mm_Vertical, symbol Connector:Conn_01x08_Female
- added TP24, TP25, TP26, TP27: TestPoint, symbol Connector:TestPoint
- D10, D11, D12, D16: value DO-214AC -> CDBA340-HF; footprint karca_custom_footprints:DO-214AC -> Diode_SMD:D_SMA
Connections:
- net +10V: now also D34.1 (K), D36.1 (K), D38.1 (K), D40.1 (K), J6.1 (Pin_1), J6.3 (Pin_3), J6.5 (Pin_5), J6.7 (Pin_7)
- net +5V: now also ADC2.15 (Vref), ADC2.16 (Vdd), C19.2
- net GND: now also ADC2.14 (AGND), ADC2.9 (DGND), C19.1, D35.2 (A), D37.2 (A), D39.2 (A), D41.2 (A)
- net PT1-: now also D34.2 (A), D35.1 (K), J6.2 (Pin_2), TP25.1
- net PT1_CAL: now also ADC2.1 (CH0), J7.1 (Pin_1)
- net PT2-: now also D36.2 (A), D37.1 (K), J6.4 (Pin_4), TP26.1
- net PT2_CAL: now also ADC2.2 (CH1), J7.2 (Pin_2)
- net PT3-: now also D38.2 (A), D39.1 (K), J6.6 (Pin_6), TP27.1
- net PT3_CAL: now also ADC2.3 (CH2), J7.3 (Pin_3)
- net PT4-: now also D40.2 (A), D41.1 (K), J6.8 (Pin_8), TP24.1
- net PT4_CAL: now also ADC2.4 (CH3), J7.4 (Pin_4)
- new net: ADC2.5 (CH4), J7.5 (Pin_5)
- new net: ADC2.6 (CH5), J7.6 (Pin_6)
- new net: ADC2.7 (CH6), J7.7 (Pin_7)
- new net: ADC2.8 (CH7), J7.8 (Pin_8)
- new net CS: ADC2.10 (~{CS}/SHDN)
- new net SPI_CLK: ADC2.13 (CLK)
- new net SPI_MISO: ADC2.12 (Dout)
- new net SPI_MOSI: ADC2.11 (Din)
Other:
- moved on the sheet: C25, C26, C27, C28, C29, C30, C31, C32, C33, D10, D11, D12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

Commit message: cleaned up PT footprint
Parts:
- J6: footprint (none) -> 1190370:1190370
- TP24, TP25, TP26, TP27: footprint (none) -> TestPoint:TestPoint_Pad_D2.0mm
Changed lines of the file:
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@@
     (property "Reference" "J6" (id 0) (at 28.575 88.265 0))
     (property "Value" "Screw_Terminal_01x08" (id 1) (at 28.575 90.805 0))
-    (property "Footprint" "" (id 2) (at 28.575 102.235 0)
+    (property "Footprint" "1190370:1190370" (id 2) (at 28.575 102.235 0)
       (effects (font (size 1.27 1.27)) hide)
     )
@@
       (effects (font (size 1.27 1.27)) (justify left) hide)
     )
-    (property "Footprint" "" (id 2) (at 83.185 76.835 0)
+    (property "Footprint" "TestPoint:TestPoint_Pad_D2.0mm" (id 2) (at 83.185 76.835 0)
       (effects (font (size 1.27 1.27)) hide)
     )
@@
       (effects (font (size 1.27 1.27)) (justify left) hide)
     )
-    (property "Footprint" "" (id 2) (at 83.1205 163.83 0)
+    (property "Footprint" "TestPoint:TestPoint_Pad_D2.0mm" (id 2) (at 83.1205 163.83 0)
       (effects (font (size 1.27 1.27)) hide)
     )
@@
       (effects (font (size 1.27 1.27)) (justify left) hide)
     )
-    (property "Footprint" "" (id 2) (at 83.185 120.015 0)
+    (property "Footprint" "TestPoint:TestPoint_Pad_D2.0mm" (id 2) (at 83.185 120.015 0)
       (effects (font (size 1.27 1.27)) hide)
     )
@@
       (effects (font (size 1.27 1.27)) (justify left) hide)
     )
-    (property "Footprint" "" (id 2) (at 83.185 33.655 0)
-      (effects (font (size 1.27 1.27)) hide)
-    )
+    (property "Footprint" "TestPoint:TestPoint_Pad_D2.0mm" (id 2) (at 83.185 33.655 0)
+      (effects (font (size 1.27 1.27)) hide)
+    )

Commit message: my body is a machine that takes in peanut m&ms and puts out rocket engine controllers
Parts:
- ADC2: LCSC (none) -> C16939
- C19, C33: LCSC (none) -> C377067
- C25, C26, C27, C28, C29, C30, C31, C32: LCSC (none) -> C1845
- D10, D11, D12, D16, D34, D35, D36, D37, D38, D39, D40, D41: LCSC (none) -> C14996
- R66, R67, R68, R69, R76, R77, R78, R79: LCSC (none) -> C102381
- R70, R72, R80, R82: LCSC (none) -> C17958
- R71, R73, R81, R83: LCSC (none) -> C168584
- R74, R75, R84, R85: LCSC (none) -> C26033
- U11: value LM324DT -> LM324; LCSC (none) -> C71035
