File: lc_anti_alias.kicad_sch (KiCad schematic)
At the start: 30 parts

Commit message: first revision of full schematic copied over
Parts:
- removed C? (x8): 1nF, symbol Device:C_Polarized
- removed C?: 100nF, symbol Device:C_Polarized
- added C? (x8): 1nF, symbol Device:C
- added C?: 100nF, symbol Device:C
Connections:
- net +10V: now also C?.1
- net GND: now also C?.2, C?.2, C?.2, C?.2, C?.2
- net LC1_CAL: now also C?.2
- net LC2_CAL: now also C?.2
- net LC3_CAL: now also C?.2
- net LC4_CAL: now also C?.2
- net at R?.1, R?.2: now also C?.1 (x4)
- net at R?.2, U?.12 (+): now also C?.1
- net at R?.2, U?.3 (+): now also C?.1
- net at R?.2, U?.10 (+): now also C?.1
- net at R?.2, U?.5 (+): now also C?.1
Other:
- company: (none) -> Rice Eclipse
- title: (none) -> Load Cell Anti-Aliasing

Commit message: added schematic pdf for review
Parts:
- gave numbers to parts that had none: 26

Commit message: added footprints and started schematic review revisions
Parts:
- C10, C11, C12, C13, C14, C15, C16, C17, C9: footprint (none) -> Capacitor_SMD:C_1206_3216Metric
- R38, R39, R40, R41, R42, R43, R44, R45, R46, R47, R48, R49, R50, R51, R52, R53: footprint (none) -> Resistor_SMD:R_1206_3216Metric
- U7: value LM324 -> LM324DT; footprint (none) -> Package_SO:SOIC-14_3.9x8.7mm_P1.27mm

Commit message: preliminary layout and started pwr plane config
Parts:
- added C20, C22, C23, C24: 1nF, Capacitor_SMD:C_1206_3216Metric, symbol Device:C
- added C21: 100nF, Capacitor_SMD:C_1206_3216Metric, symbol Device:C
- added R58, R59, R60, R61: 68k, Resistor_SMD:R_1206_3216Metric, symbol Device:R_US
- added R62, R63: 15k, Resistor_SMD:R_1206_3216Metric, symbol Device:R_US
- added R64, R65: 10k, Resistor_SMD:R_1206_3216Metric, symbol Device:R_US
- added U10: LM324DT, Package_SO:SOIC-14_3.9x8.7mm_P1.27mm, symbol Amplifier_Operational:LM324
- renumbered C16 to C11, C14 to C13, C10 to C14, C13 to C15, C17 to C16, C9 to C17, C11 to C18, C15 to C19, R46 to R42, R48 to R43, R38 to R44, R40 to R45, R50 to R46, R42 to R47, R51 to R48, R43 to R49, R39 to R50, R41 to R51, R47 to R52, R49 to R53, R44 to R54, R52 to R55, R45 to R56, R53 to R57, U7 to U9
Connections:
- net +10V: now also C21.1, U10.4 (V+)
- net GND: now also C21.2, C23.2, C24.2, R64.2, R65.2, U10.11 (V-)
- new net: C20.1, R58.2, R59.1
- new net: C23.1, R59.2, U10.5 (+)
- new net: R63.2, R65.1, U10.2 (-)
- new net: C22.1, R60.2, R61.1
- new net: R62.2, R64.1, U10.6 (-)
- new net: C24.1, R61.2, U10.3 (+)
- new net LC5_CAL: C22.2, R63.1, U10.1
- new net LC5_PREC: R60.1
- new net LC6_CAL: C20.2, R62.1, U10.7
- new net LC6_PREC: R58.1
- no-connect marks 0 -> 6
Other:
- moved on the sheet: C11, C12, C13, C14, C15, C16, C17, C18, C19, R42, R43, R44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

Commit message: some minor schematic cleanup
Parts:
- C11, C12, C13, C14, C15, C16, C18, C19, C20, C22, C23, C24: value 1nF -> 1n
- C17, C21: value 100nF -> 100n
Changed lines of the file:
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@@
       (effects (font (size 1.27 1.27)) hide)
     )
-    (property "Datasheet" "https://media.digikey.com/pdf/Data%20Sheets/Rohm%20PDFs/LM358,LM324,LM2904,LM2902.pdf" (id 3) (at 91.44 33.02 0)
+    (property "Datasheet" "http://www.ti.com/lit/ds/symlink/lm2902-n.pdf" (id 3) (at 91.44 33.02 0)
       (effects (font (size 1.27 1.27)) hide)
     )
@@
       (effects (font (size 1.27 1.27)) (justify left))
     )
-    (property "Value" "1nF" (id 1) (at 76.2 43.1799 0)
+    (property "Value" "1n" (id 1) (at 76.2 43.1799 0)
       (effects (font (size 1.27 1.27)) (justify left))
     )
@@
       (effects (font (size 1.27 1.27)) (justify left))
     )
-    (property "Value" "1nF" (id 1) (at 106.68 132.0799 0)
+    (property "Value" "1n" (id 1) (at 106.68 132.0799 0)
       (effects (font (size 1.27 1.27)) (justify left))
     )
@@
       (effects (font (size 1.27 1.27)) (justify left))
     )
-    (property "Value" "1nF" (id 1) (at 207.01 80.0099 0)
+    (property "Value" "1n" (id 1) (at 207.01 80.0099 0)
       (effects (font (size 1.27 1.27)) (justify left))
     )
@@
       (effects (font (size 1.27 1.27)) (justify left))
     )
-    (property "Value" "1nF" (id 1) (at 176.53 140.9699 0)
+    (property "Value" "1n" (id 1) (at 176.53 140.9699 0)
       (effects (font (size 1.27 1.27)) (justify left))
     )
@@
       (effects (font (size 1.27 1.27)) (justify left))
     )
-    (property "Value" "100nF" (id 1) (at 246.38 130.81 0)
+    (property "Value" "100n" (id 1) (at 246.38 130.81 0)
       (effects (font (size 1.27 1.27)) (justify left))
     )
@@
       (effects (font (size 1.27 1.27)) (justify left))
     )
-    (property "Value" "1nF" (id 1) (at 74.93 142.2399 0)
+    (property "Value" "1n" (id 1) (at 74.93 142.2399 0)
       (effects (font (size 1.27 1.27)) (justify left))
     )
@@
       (effects (font (size 1.27 1.27)) (justify left))
     )
-    (property "Value" "1nF" (id 1) (at 76.2 88.8999 0)
+    (property "Value" "1n" (id 1) (at 76.2 88.8999 0)
       (effects (font (size 1.27 1.27)) (justify left))
     )
@@
       (effects (font (size 1.27 1.27)) (justify left))
     )
-    (property "Value" "1nF" (id 1) (at 208.28 31.7499 0)
+    (property "Value" "1n" (id 1) (at 208.28 31.7499 0)
       (effects (font (size 1.27 1.27)) (justify left))
     )
@@
       (effects (font (size 1.27 1.27)) (justify left))
     )
-    (property "Value" "1nF" (id 1) (at 176.53 41.9099 0)
+    (property "Value" "1n" (id 1) (at 176.53 41.9099 0)
       (effects (font (size 1.27 1.27)) (justify left))
     )
@@
       (effects (font (size 1.27 1.27)) (justify left))
     )
-    (property "Value" "1nF" (id 1) (at 208.28 130.8099 0)
+    (property "Value" "1n" (id 1) (at 208.28 130.8099 0)
       (effects (font (size 1.27 1.27)) (justify left))
     )
@@
       (effects (font (size 1.27 1.27)) hide)
     )
-    (property "Datasheet" "https://media.digikey.com/pdf/Data%20Sheets/Rohm%20PDFs/LM358,LM324,LM2904,LM2902.pdf" (id 3) (at 191.77 31.75 0)
+    (property "Datasheet" "http://www.ti.com/lit/ds/symlink/lm2902-n.pdf" (id 3) (at 191.77 31.75 0)
       (effects (font (size 1.27 1.27)) hide)
     )
@@
       (effects (font (size 1.27 1.27)) hide)
     )
-    (property "Datasheet" "https://media.digikey.com/pdf/Data%20Sheets/Rohm%20PDFs/LM358,LM324,LM2904,LM2902.pdf" (id 3) (at 190.5 80.01 0)
+    (property "Datasheet" "http://www.ti.com/lit/ds/symlink/lm2902-n.pdf" (id 3) (at 190.5 80.01 0)
       (effects (font (size 1.27 1.27)) hide)
     )
@@
       (effects (font (size 1.27 1.27)) (justify left))
     )
-    (property "Value" "1nF" (id 1) (at 107.95 78.7399 0)
+    (property "Value" "1n" (id 1) (at 107.95 78.7399 0)
       (effects (font (size 1.27 1.27)) (justify left))
     )
@@
       (effects (font (size 1.27 1.27)) hide)
     )
-    (property "Datasheet" "https://media.digikey.com/pdf/Data%20Sheets/Rohm%20PDFs/LM358,LM324,LM2904,LM2902.pdf" (id 3) (at 270.51 73.66 0)
+    (property "Datasheet" "http://www.ti.com/lit/ds/symlink/lm2902-n.pdf" (id 3) (at 270.51 73.66 0)
       (effects (font (size 1.27 1.27)) hide)
     )
@@
       (effects (font (size 1.27 1.27)) hide)
     )
-    (property "Datasheet" "https://media.digikey.com/pdf/Data%20Sheets/Rohm%20PDFs/LM358,LM324,LM2904,LM2902.pdf" (id 3) (at 91.44 78.74 0)
+    (property "Datasheet" "http://www.ti.com/lit/ds/symlink/lm2902-n.pdf" (id 3) (at 91.44 78.74 0)
       (effects (font (size 1.27 1.27)) hide)
     )
@@
       (effects (font (size 1.27 1.27)) (justify left))
     )
-    (property "Value" "100nF" (id 1) (at 247.65 80.01 0)
+    (property "Value" "100n" (id 1) (at 247.65 80.01 0)
       (effects (font (size 1.27 1.27)) (justify left))
     )
@@
       (effects (font (size 1.27 1.27)) (justify left))
     )
-    (property "Value" "1nF" (id 1) (at 107.95 33.0199 0)
+    (property "Value" "1n" (id 1) (at 107.95 33.0199 0)
       (effects (font (size 1.27 1.27)) (justify left))
     )
@@
       (effects (font (size 1.27 1.27)) (justify left))
     )
-    (property "Value" "1nF" (id 1) (at 175.26 90.1699 0)
-      (effects (font (size 1.27 1.27)) (justify left))
-    )
+    (property "Value" "1n" (id 1) (at 175.26 90.1699 0)
+      (effects (font (size 1.27 1.27)) (justify left))
+    )

Commit message: shuffle around some parts
Changed lines of the file:
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@@
   (junction (at 158.75 34.29) (diameter 0) (color 0 0 0 0)
   )
-  (no_connect (at 83.82 181.61))
-  (no_connect (at 83.82 186.69))
-  (no_connect (at 106.68 184.15))
-  (no_connect (at 39.37 181.61))
-  (no_connect (at 39.37 186.69))
-  (no_connect (at 60.96 184.15))
-  (wire (pts (xy 39.37 186.69) (xy 43.18 186.69))
-    (stroke (width 0) (type default) (color 0 0 0 0))
-  )
+  (no_connect (at 87.63 181.61))
+  (no_connect (at 87.63 186.69))
+  (no_connect (at 102.87 184.15))
+  (no_connect (at 43.18 181.61))
+  (no_connect (at 43.18 186.69))
+  (no_connect (at 58.42 184.15))
   (wire (pts (xy 204.47 135.89) (xy 204.47 133.35))
     (stroke (width 0) (type default) (color 0 0 0 0))
@@
     (stroke (width 0) (type default) (color 0 0 0 0))
   )
-  (wire (pts (xy 83.82 181.61) (xy 87.63 181.61))
-    (stroke (width 0) (type default) (color 0 0 0 0))
-  )
   (wire (pts (xy 58.42 35.56) (xy 58.42 24.13))
     (stroke (width 0) (type default) (color 0 0 0 0))
@@
     (stroke (width 0) (type default) (color 0 0 0 0))
   )
-  (wire (pts (xy 58.42 184.15) (xy 60.96 184.15))
-    (stroke (width 0) (type default) (color 0 0 0 0))
-  )
   (wire (pts (xy 203.2 85.09) (xy 204.47 85.09))
     (stroke (width 0) (type default) (color 0 0 0 0))
@@
     (stroke (width 0) (type default) (color 0 0 0 0))
   )
-  (wire (pts (xy 102.87 184.15) (xy 106.68 184.15))
-    (stroke (width 0) (type default) (color 0 0 0 0))
-  )
   (wire (pts (xy 72.39 35.56) (xy 82.55 35.56))
     (stroke (width 0) (type default) (color 0 0 0 0))
@@
     (stroke (width 0) (type default) (color 0 0 0 0))
   )
-  (wire (pts (xy 83.82 186.69) (xy 87.63 186.69))
-    (stroke (width 0) (type default) (color 0 0 0 0))
-  )
   (wire (pts (xy 172.72 34.29) (xy 182.88 34.29))
     (stroke (width 0) (type default) (color 0 0 0 0))
@@
     (stroke (width 0) (type default) (color 0 0 0 0))
   )
-  (wire (pts (xy 39.37 181.61) (xy 43.18 181.61))
-    (stroke (width 0) (type default) (color 0 0 0 0))
-  )

Commit message: add overvoltage diodes
Parts:
- added D2, D4, D6, D7, D8, D9: SS54, karca_custom_footprints:DO-214AC, symbol Device:D_Schottky
Connections:
- net LC1_CAL: now also D6.2 (A)
- net LC2_CAL: now also D9.2 (A)
- net LC3_CAL: now also D4.2 (A)
- net LC4_CAL: now also D7.2 (A)
- net LC5_CAL: now also D2.2 (A)
- net LC6_CAL: now also D8.2 (A)
- new net +5V: D2.1 (K), D4.1 (K), D6.1 (K), D7.1 (K), D8.1 (K), D9.1 (K)

Commit message: laid out ignition and PTs
Parts:
- D2, D4, D6, D7, D8, D9: value SS54 -> DO-214AC
Changed lines of the file:
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@@
       (effects (font (size 1.27 1.27)) (justify left))
     )
-    (property "Value" "SS54" (id 1) (at 116.205 80.9624 90)
+    (property "Value" "DO-214AC" (id 1) (at 116.205 80.9624 90)
       (effects (font (size 1.27 1.27)) (justify left))
     )
@@
       (effects (font (size 1.27 1.27)) (justify left))
     )
-    (property "Value" "SS54" (id 1) (at 114.935 134.3024 90)
+    (property "Value" "DO-214AC" (id 1) (at 114.935 134.3024 90)
       (effects (font (size 1.27 1.27)) (justify left))
     )
@@
       (effects (font (size 1.27 1.27)) (justify left))
     )
-    (property "Value" "SS54" (id 1) (at 215.9 82.2324 90)
+    (property "Value" "DO-214AC" (id 1) (at 215.9 82.2324 90)
       (effects (font (size 1.27 1.27)) (justify left))
     )
@@
       (effects (font (size 1.27 1.27)) (justify left))
     )
-    (property "Value" "SS54" (id 1) (at 118.11 35.2424 90)
+    (property "Value" "DO-214AC" (id 1) (at 118.11 35.2424 90)
       (effects (font (size 1.27 1.27)) (justify left))
     )
@@
       (effects (font (size 1.27 1.27)) (justify left))
     )
-    (property "Value" "SS54" (id 1) (at 216.535 133.0324 90)
+    (property "Value" "DO-214AC" (id 1) (at 216.535 133.0324 90)
       (effects (font (size 1.27 1.27)) (justify left))
     )
@@
       (effects (font (size 1.27 1.27)) (justify left))
     )
-    (property "Value" "SS54" (id 1) (at 217.17 33.9724 90)
-      (effects (font (size 1.27 1.27)) (justify left))
-    )
+    (property "Value" "DO-214AC" (id 1) (at 217.17 33.9724 90)
+      (effects (font (size 1.27 1.27)) (justify left))
+    )
