File: lc_anti_alias.kicad_sch (KiCad schematic)
At the start: 46 parts, among them U10 LM324DT, U9 LM324DT

Commit message: enshrinkening of the board
Parts:
- removed C20, C22, C23, C24: 1n, Capacitor_SMD:C_1206_3216Metric, symbol Device:C
- removed C21: 100n, Capacitor_SMD:C_1206_3216Metric, symbol Device:C
- removed D2, D8: DO-214AC, karca_custom_footprints:DO-214AC, symbol Device:D_Schottky
- removed R58, R59, R60, R61: 68k, Resistor_SMD:R_1206_3216Metric, symbol Device:R_US
- removed R62, R63: 15k, Resistor_SMD:R_1206_3216Metric, symbol Device:R_US
- removed R64, R65: 10k, Resistor_SMD:R_1206_3216Metric, symbol Device:R_US
- removed U10: LM324DT, Package_SO:SOIC-14_3.9x8.7mm_P1.27mm, symbol Amplifier_Operational:LM324
Connections:
- no-connect marks 6 -> 0

Commit message: done schematiccing after design review
Parts:
- removed C11, C12, C13, C14, C15, C16, C18, C19: 1n, Capacitor_SMD:C_1206_3216Metric, symbol Device:C
- removed C17: 100n, Capacitor_SMD:C_1206_3216Metric, symbol Device:C
- removed D4, D6, D7, D9: DO-214AC, karca_custom_footprints:DO-214AC, symbol Device:D_Schottky
- removed R42, R43, R44, R45, R50, R51, R52, R53: 68k, Resistor_SMD:R_1206_3216Metric, symbol Device:R_US
- removed R46, R47, R54, R55: 15k, Resistor_SMD:R_1206_3216Metric, symbol Device:R_US
- removed R48, R49, R56, R57: 10k, Resistor_SMD:R_1206_3216Metric, symbol Device:R_US
- removed U9: LM324DT, Package_SO:SOIC-14_3.9x8.7mm_P1.27mm, symbol Amplifier_Operational:LM324
