File: thermocouples.kicad_sch (KiCad schematic)
At the start: 0 parts

Commit message: first revision of full schematic copied over
Parts:
- added F? (x4): Fuse, symbol Device:Fuse
- added J? (x4): Conn_01x03_Female, symbol Connector:Conn_01x03_Female
Connections:
- new net: F?.2, J?.1 (Pin_1) (x4)
- new net +5V: F?.1, F?.1, F?.1, F?.1
- new net GND: J?.3 (Pin_3), J?.3 (Pin_3), J?.3 (Pin_3), J?.3 (Pin_3)
- new net TC1: J?.2 (Pin_2)
- new net TC2: J?.2 (Pin_2)
- new net TC3: J?.2 (Pin_2)
- new net TC4: J?.2 (Pin_2)
Other:
- company: (none) -> Rice Eclipse
- title: (none) -> Thermocouple Ports

Commit message: added schematic pdf for review
Parts:
- gave numbers to parts that had none: 8
Changed lines of the file:
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@@
   (symbol (lib_id "power:+5V") (at 43.18 134.62 0) (unit 1)
     (in_bom yes) (on_board yes) (fields_autoplaced)
-    (property "Reference" "#PWR?" (id 0) (at 43.18 138.43 0)
+    (property "Reference" "#PWR0109" (id 0) (at 43.18 138.43 0)
       (effects (font (size 1.27 1.27)) hide)
     )
@@
   (symbol (lib_id "Device:Fuse") (at 43.18 99.06 0) (unit 1)
     (in_bom yes) (on_board yes) (fields_autoplaced)
-    (property "Reference" "F?" (id 0) (at 45.72 97.7899 0)
+    (property "Reference" "F17" (id 0) (at 45.72 97.7899 0)
       (effects (font (size 1.27 1.27)) (justify left))
     )
@@
   (symbol (lib_id "Connector:Conn_01x03_Female") (at 34.29 73.66 0) (mirror y) (unit 1)
     (in_bom yes) (on_board yes) (fields_autoplaced)
-    (property "Reference" "J?" (id 0) (at 34.925 66.04 0))
+    (property "Reference" "J30" (id 0) (at 34.925 66.04 0))
     (property "Value" "Conn_01x03_Female" (id 1) (at 34.925 68.58 0))
     (property "Footprint" "" (id 2) (at 34.29 73.66 0)
@@
   (symbol (lib_id "Connector:Conn_01x03_Female") (at 34.29 147.32 0) (mirror y) (unit 1)
     (in_bom yes) (on_board yes) (fields_autoplaced)
-    (property "Reference" "J?" (id 0) (at 34.925 139.7 0))
+    (property "Reference" "J32" (id 0) (at 34.925 139.7 0))
     (property "Value" "Conn_01x03_Female" (id 1) (at 34.925 142.24 0))
     (property "Footprint" "" (id 2) (at 34.29 147.32 0)
@@
   (symbol (lib_id "power:+5V") (at 43.18 60.96 0) (unit 1)
     (in_bom yes) (on_board yes) (fields_autoplaced)
-    (property "Reference" "#PWR?" (id 0) (at 43.18 64.77 0)
+    (property "Reference" "#PWR0105" (id 0) (at 43.18 64.77 0)
       (effects (font (size 1.27 1.27)) hide)
     )
@@
   (symbol (lib_id "power:+5V") (at 43.18 25.4 0) (unit 1)
     (in_bom yes) (on_board yes) (fields_autoplaced)
-    (property "Reference" "#PWR?" (id 0) (at 43.18 29.21 0)
+    (property "Reference" "#PWR0103" (id 0) (at 43.18 29.21 0)
       (effects (font (size 1.27 1.27)) hide)
     )
@@
   (symbol (lib_id "Device:Fuse") (at 43.18 138.43 0) (unit 1)
     (in_bom yes) (on_board yes) (fields_autoplaced)
-    (property "Reference" "F?" (id 0) (at 45.72 137.1599 0)
+    (property "Reference" "F18" (id 0) (at 45.72 137.1599 0)
       (effects (font (size 1.27 1.27)) (justify left))
     )
@@
   (symbol (lib_id "power:GND") (at 43.18 44.45 0) (unit 1)
     (in_bom yes) (on_board yes) (fields_autoplaced)
-    (property "Reference" "#PWR?" (id 0) (at 43.18 50.8 0)
+    (property "Reference" "#PWR0104" (id 0) (at 43.18 50.8 0)
       (effects (font (size 1.27 1.27)) hide)
     )
@@
   (symbol (lib_id "power:GND") (at 43.18 114.3 0) (unit 1)
     (in_bom yes) (on_board yes) (fields_autoplaced)
-    (property "Reference" "#PWR?" (id 0) (at 43.18 120.65 0)
+    (property "Reference" "#PWR0108" (id 0) (at 43.18 120.65 0)
       (effects (font (size 1.27 1.27)) hide)
     )
@@
   (symbol (lib_id "power:GND") (at 43.18 153.67 0) (unit 1)
     (in_bom yes) (on_board yes) (fields_autoplaced)
-    (property "Reference" "#PWR?" (id 0) (at 43.18 160.02 0)
+    (property "Reference" "#PWR0110" (id 0) (at 43.18 160.02 0)
       (effects (font (size 1.27 1.27)) hide)
     )
@@
   (symbol (lib_id "Device:Fuse") (at 43.18 29.21 0) (unit 1)
     (in_bom yes) (on_board yes) (fields_autoplaced)
-    (property "Reference" "F?" (id 0) (at 45.72 27.9399 0)
+    (property "Reference" "F15" (id 0) (at 45.72 27.9399 0)
       (effects (font (size 1.27 1.27)) (justify left))
     )
@@
   (symbol (lib_id "Connector:Conn_01x03_Female") (at 34.29 38.1 0) (mirror y) (unit 1)
     (in_bom yes) (on_board yes) (fields_autoplaced)
-    (property "Reference" "J?" (id 0) (at 34.925 30.48 0))
+    (property "Reference" "J29" (id 0) (at 34.925 30.48 0))
     (property "Value" "Conn_01x03_Female" (id 1) (at 34.925 33.02 0))
     (property "Footprint" "" (id 2) (at 34.29 38.1 0)
@@
   (symbol (lib_id "power:+5V") (at 43.18 95.25 0) (unit 1)
     (in_bom yes) (on_board yes) (fields_autoplaced)
-    (property "Reference" "#PWR?" (id 0) (at 43.18 99.06 0)
+    (property "Reference" "#PWR0107" (id 0) (at 43.18 99.06 0)
       (effects (font (size 1.27 1.27)) hide)
     )
@@
   (symbol (lib_id "Device:Fuse") (at 43.18 64.77 0) (unit 1)
     (in_bom yes) (on_board yes) (fields_autoplaced)
-    (property "Reference" "F?" (id 0) (at 45.72 63.4999 0)
+    (property "Reference" "F16" (id 0) (at 45.72 63.4999 0)
       (effects (font (size 1.27 1.27)) (justify left))
     )
@@
   (symbol (lib_id "Connector:Conn_01x03_Female") (at 34.29 107.95 0) (mirror y) (unit 1)
     (in_bom yes) (on_board yes) (fields_autoplaced)
-    (property "Reference" "J?" (id 0) (at 34.925 100.33 0))
+    (property "Reference" "J31" (id 0) (at 34.925 100.33 0))
     (property "Value" "Conn_01x03_Female" (id 1) (at 34.925 102.87 0))
     (property "Footprint" "" (id 2) (at 34.29 107.95 0)
@@
   (symbol (lib_id "power:GND") (at 43.18 80.01 0) (unit 1)
     (in_bom yes) (on_board yes) (fields_autoplaced)
-    (property "Reference" "#PWR?" (id 0) (at 43.18 86.36 0)
-      (effects (font (size 1.27 1.27)) hide)
-    )
+    (property "Reference" "#PWR0106" (id 0) (at 43.18 86.36 0)
+      (effects (font (size 1.27 1.27)) hide)
+    )

Commit message: added footprints and started schematic review revisions
Parts:
- F15, F16, F17, F18: value Fuse -> 3588-20; footprint (none) -> karca_custom_footprints:3588-20 fuse
Changed lines of the file:
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@@
       (effects (font (size 1.27 1.27)) (justify left))
     )
-    (property "Value" "Fuse" (id 1) (at 45.72 100.3299 0)
+    (property "Value" "3588-20" (id 1) (at 45.72 100.3299 0)
       (effects (font (size 1.27 1.27)) (justify left))
     )
-    (property "Footprint" "" (id 2) (at 41.402 99.06 90)
+    (property "Footprint" "karca_custom_footprints:3588-20 fuse" (id 2) (at 41.402 99.06 90)
       (effects (font (size 1.27 1.27)) hide)
     )
-    (property "Datasheet" "~" (id 3) (at 43.18 99.06 0)
+    (property "Datasheet" "https://www.mouser.com/datasheet/2/215/588-20-1622270.pdf" (id 3) (at 43.18 99.06 0)
       (effects (font (size 1.27 1.27)) hide)
     )
@@
       (effects (font (size 1.27 1.27)) (justify left))
     )
-    (property "Value" "Fuse" (id 1) (at 45.72 139.6999 0)
+    (property "Value" "3588-20" (id 1) (at 45.72 139.6999 0)
       (effects (font (size 1.27 1.27)) (justify left))
     )
-    (property "Footprint" "" (id 2) (at 41.402 138.43 90)
+    (property "Footprint" "karca_custom_footprints:3588-20 fuse" (id 2) (at 41.402 138.43 90)
       (effects (font (size 1.27 1.27)) hide)
     )
-    (property "Datasheet" "~" (id 3) (at 43.18 138.43 0)
+    (property "Datasheet" "https://www.mouser.com/datasheet/2/215/588-20-1622270.pdf" (id 3) (at 43.18 138.43 0)
       (effects (font (size 1.27 1.27)) hide)
     )
@@
       (effects (font (size 1.27 1.27)) (justify left))
     )
-    (property "Value" "Fuse" (id 1) (at 45.72 30.4799 0)
+    (property "Value" "3588-20" (id 1) (at 45.72 30.4799 0)
       (effects (font (size 1.27 1.27)) (justify left))
     )
-    (property "Footprint" "" (id 2) (at 41.402 29.21 90)
+    (property "Footprint" "karca_custom_footprints:3588-20 fuse" (id 2) (at 41.402 29.21 90)
       (effects (font (size 1.27 1.27)) hide)
     )
-    (property "Datasheet" "~" (id 3) (at 43.18 29.21 0)
+    (property "Datasheet" "https://www.mouser.com/datasheet/2/215/588-20-1622270.pdf" (id 3) (at 43.18 29.21 0)
       (effects (font (size 1.27 1.27)) hide)
     )
@@
       (effects (font (size 1.27 1.27)) (justify left))
     )
-    (property "Value" "Fuse" (id 1) (at 45.72 66.0399 0)
+    (property "Value" "3588-20" (id 1) (at 45.72 66.0399 0)
       (effects (font (size 1.27 1.27)) (justify left))
     )
-    (property "Footprint" "" (id 2) (at 41.402 64.77 90)
+    (property "Footprint" "karca_custom_footprints:3588-20 fuse" (id 2) (at 41.402 64.77 90)
       (effects (font (size 1.27 1.27)) hide)
     )
-    (property "Datasheet" "~" (id 3) (at 43.18 64.77 0)
+    (property "Datasheet" "https://www.mouser.com/datasheet/2/215/588-20-1622270.pdf" (id 3) (at 43.18 64.77 0)
       (effects (font (size 1.27 1.27)) hide)
     )

Commit message: updated all footprints, resolved most ERC & setup layout
Parts:
- J29, J30, J31, J32: footprint (none) -> Connector_PinSocket_2.54mm:PinSocket_1x03_P2.54mm_Vertical
Changed lines of the file:
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@@
     (property "Reference" "J30" (id 0) (at 34.925 66.04 0))
     (property "Value" "Conn_01x03_Female" (id 1) (at 34.925 68.58 0))
-    (property "Footprint" "" (id 2) (at 34.29 73.66 0)
+    (property "Footprint" "Connector_PinSocket_2.54mm:PinSocket_1x03_P2.54mm_Vertical" (id 2) (at 34.29 73.66 0)
       (effects (font (size 1.27 1.27)) hide)
     )
@@
     (property "Reference" "J32" (id 0) (at 34.925 139.7 0))
     (property "Value" "Conn_01x03_Female" (id 1) (at 34.925 142.24 0))
-    (property "Footprint" "" (id 2) (at 34.29 147.32 0)
+    (property "Footprint" "Connector_PinSocket_2.54mm:PinSocket_1x03_P2.54mm_Vertical" (id 2) (at 34.29 147.32 0)
       (effects (font (size 1.27 1.27)) hide)
     )
@@
     (property "Reference" "J29" (id 0) (at 34.925 30.48 0))
     (property "Value" "Conn_01x03_Female" (id 1) (at 34.925 33.02 0))
-    (property "Footprint" "" (id 2) (at 34.29 38.1 0)
+    (property "Footprint" "Connector_PinSocket_2.54mm:PinSocket_1x03_P2.54mm_Vertical" (id 2) (at 34.29 38.1 0)
       (effects (font (size 1.27 1.27)) hide)
     )
@@
     (property "Reference" "J31" (id 0) (at 34.925 100.33 0))
     (property "Value" "Conn_01x03_Female" (id 1) (at 34.925 102.87 0))
-    (property "Footprint" "" (id 2) (at 34.29 107.95 0)
+    (property "Footprint" "Connector_PinSocket_2.54mm:PinSocket_1x03_P2.54mm_Vertical" (id 2) (at 34.29 107.95 0)
       (effects (font (size 1.27 1.27)) hide)
     )

Commit message: preliminary layout and started pwr plane config
Parts:
- removed J29, J30, J31, J32: Conn_01x03_Female, Connector_PinSocket_2.54mm:PinSocket_1x03_P2.54mm_Vertical, symbol Connector:Conn_01x03_Female
- added J26, J27, J28, J29: Screw_Terminal_01x03, 1190364:1190364, symbol Connector:Screw_Terminal_01x03
- F17: renamed from F15; footprint karca_custom_footprints:3588-20 fuse -> 3588-20:358820
- F18: renamed from F16; footprint karca_custom_footprints:3588-20 fuse -> 3588-20:358820
- F19: renamed from F17; footprint karca_custom_footprints:3588-20 fuse -> 3588-20:358820
- F20: renamed from F18; footprint karca_custom_footprints:3588-20 fuse -> 3588-20:358820
Connections:
- net GND: now also J26.3 (Pin_3), J27.3 (Pin_3), J28.3 (Pin_3), J29.3 (Pin_3)
- net TC1: now also J26.2 (Pin_2)
- net TC2: now also J27.2 (Pin_2)
- net TC3: now also J28.2 (Pin_2)
- net TC4: now also J29.2 (Pin_2)
- net at F19.2: now also J28.1 (Pin_1)
- net at F18.2: now also J27.1 (Pin_1)
- net at F20.2: now also J29.1 (Pin_1)
- net at F17.2: now also J26.1 (Pin_1)
Changed lines of the file:
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@@
     )
+  )
+  (symbol (lib_id "Connector:Screw_Terminal_01x03") (at 34.29 73.66 0) (mirror y) (unit 1)
+    (in_bom yes) (on_board yes) (fields_autoplaced)
+    (property "Reference" "J27" (id 0) (at 34.29 67.31 0))
+    (property "Value" "Screw_Terminal_01x03" (id 1) (at 34.29 67.31 0)
+      (effects (font (size 1.27 1.27)) hide)
+    )
+    (property "Footprint" "1190364:1190364" (id 2) (at 34.29 73.66 0)
+      (effects (font (size 1.27 1.27)) hide)
+    )
+    (property "Datasheet" "https://www.mouser.com/ProductDetail/Phoenix-Contact/1190364?qs=QNEnbhJQKvaxxoSFQSEyNA%3D%3D" (id 3) (at 34.29 73.66 0)
+      (effects (font (size 1.27 1.27)) hide)
+    )
+    (pin "1")
+    (pin "2")
+    (pin "3")
   )
   (symbol (lib_id "power:+5V") (at 43.18 134.62 0) (unit 1)
     (in_bom yes) (on_board yes) (fields_autoplaced)
-    (property "Reference" "#PWR0109" (id 0) (at 43.18 138.43 0)
+    (property "Reference" "#PWR0135" (id 0) (at 43.18 138.43 0)
       (effects (font (size 1.27 1.27)) hide)
     )
@@
   (symbol (lib_id "Device:Fuse") (at 43.18 99.06 0) (unit 1)
     (in_bom yes) (on_board yes) (fields_autoplaced)
-    (property "Reference" "F17" (id 0) (at 45.72 97.7899 0)
+    (property "Reference" "F19" (id 0) (at 45.72 97.7899 0)
       (effects (font (size 1.27 1.27)) (justify left))
     )
@@
       (effects (font (size 1.27 1.27)) (justify left))
     )
-    (property "Footprint" "karca_custom_footprints:3588-20 fuse" (id 2) (at 41.402 99.06 90)
+    (property "Footprint" "3588-20:358820" (id 2) (at 41.402 99.06 90)
       (effects (font (size 1.27 1.27)) hide)
     )
@@
     (pin "2")
   )
-  (symbol (lib_id "Connector:Conn_01x03_Female") (at 34.29 73.66 0) (mirror y) (unit 1)
-    (in_bom yes) (on_board yes) (fields_autoplaced)
-    (property "Reference" "J30" (id 0) (at 34.925 66.04 0))
-    (property "Value" "Conn_01x03_Female" (id 1) (at 34.925 68.58 0))
-    (property "Footprint" "Connector_PinSocket_2.54mm:PinSocket_1x03_P2.54mm_Vertical" (id 2) (at 34.29 73.66 0)
-      (effects (font (size 1.27 1.27)) hide)
-    )
-    (property "Datasheet" "~" (id 3) (at 34.29 73.66 0)
-      (effects (font (size 1.27 1.27)) hide)
-    )
-    (pin "1")
-    (pin "2")
-    (pin "3")
-  )
-  (symbol (lib_id "Connector:Conn_01x03_Female") (at 34.29 147.32 0) (mirror y) (unit 1)
-    (in_bom yes) (on_board yes) (fields_autoplaced)
-    (property "Reference" "J32" (id 0) (at 34.925 139.7 0))
-    (property "Value" "Conn_01x03_Female" (id 1) (at 34.925 142.24 0))
-    (property "Footprint" "Connector_PinSocket_2.54mm:PinSocket_1x03_P2.54mm_Vertical" (id 2) (at 34.29 147.32 0)
-      (effects (font (size 1.27 1.27)) hide)
-    )
-    (property "Datasheet" "~" (id 3) (at 34.29 147.32 0)
-      (effects (font (size 1.27 1.27)) hide)
-    )
-    (pin "1")
-    (pin "2")
-    (pin "3")
-  )
   (symbol (lib_id "power:+5V") (at 43.18 60.96 0) (unit 1)
     (in_bom yes) (on_board yes) (fields_autoplaced)
-    (property "Reference" "#PWR0105" (id 0) (at 43.18 64.77 0)
+    (property "Reference" "#PWR0131" (id 0) (at 43.18 64.77 0)
       (effects (font (size 1.27 1.27)) hide)
     )
@@
   (symbol (lib_id "power:+5V") (at 43.18 25.4 0) (unit 1)
     (in_bom yes) (on_board yes) (fields_autoplaced)
-    (property "Reference" "#PWR0103" (id 0) (at 43.18 29.21 0)
+    (property "Reference" "#PWR0129" (id 0) (at 43.18 29.21 0)
       (effects (font (size 1.27 1.27)) hide)
     )
@@
   (symbol (lib_id "Device:Fuse") (at 43.18 138.43 0) (unit 1)
     (in_bom yes) (on_board yes) (fields_autoplaced)
-    (property "Reference" "F18" (id 0) (at 45.72 137.1599 0)
+    (property "Reference" "F20" (id 0) (at 45.72 137.1599 0)
       (effects (font (size 1.27 1.27)) (justify left))
     )
@@
       (effects (font (size 1.27 1.27)) (justify left))
     )
-    (property "Footprint" "karca_custom_footprints:3588-20 fuse" (id 2) (at 41.402 138.43 90)
+    (property "Footprint" "3588-20:358820" (id 2) (at 41.402 138.43 90)
       (effects (font (size 1.27 1.27)) hide)
     )
@@
   (symbol (lib_id "power:GND") (at 43.18 44.45 0) (unit 1)
     (in_bom yes) (on_board yes) (fields_autoplaced)
-    (property "Reference" "#PWR0104" (id 0) (at 43.18 50.8 0)
+    (property "Reference" "#PWR0130" (id 0) (at 43.18 50.8 0)
       (effects (font (size 1.27 1.27)) hide)
     )
@@
     (pin "1")
   )
+  (symbol (lib_id "Connector:Screw_Terminal_01x03") (at 34.29 107.95 0) (mirror y) (unit 1)
+    (in_bom yes) (on_board yes) (fields_autoplaced)
+    (property "Reference" "J28" (id 0) (at 34.29 101.6 0))
+    (property "Value" "Screw_Terminal_01x03" (id 1) (at 34.29 101.6 0)
+      (effects (font (size 1.27 1.27)) hide)
+    )
+    (property "Footprint" "1190364:1190364" (id 2) (at 34.29 107.95 0)
+      (effects (font (size 1.27 1.27)) hide)
+    )
+    (property "Datasheet" "https://www.mouser.com/ProductDetail/Phoenix-Contact/1190364?qs=QNEnbhJQKvaxxoSFQSEyNA%3D%3D" (id 3) (at 34.29 107.95 0)
+      (effects (font (size 1.27 1.27)) hide)
+    )
+    (pin "1")
+    (pin "2")
+    (pin "3")
+  )
   (symbol (lib_id "power:GND") (at 43.18 114.3 0) (unit 1)
     (in_bom yes) (on_board yes) (fields_autoplaced)
-    (property "Reference" "#PWR0108" (id 0) (at 43.18 120.65 0)
+    (property "Reference" "#PWR0134" (id 0) (at 43.18 120.65 0)
       (effects (font (size 1.27 1.27)) hide)
     )
@@
     (pin "1")
   )
+  (symbol (lib_id "Connector:Screw_Terminal_01x03") (at 34.29 38.1 0) (mirror y) (unit 1)
+    (in_bom yes) (on_board yes) (fields_autoplaced)
+    (property "Reference" "J26" (id 0) (at 34.29 31.75 0))
+    (property "Value" "Screw_Terminal_01x03" (id 1) (at 34.29 31.75 0)
+      (effects (font (size 1.27 1.27)) hide)
+    )
+    (property "Footprint" "1190364:1190364" (id 2) (at 34.29 38.1 0)
+      (effects (font (size 1.27 1.27)) hide)
+    )
+    (property "Datasheet" "https://www.mouser.com/ProductDetail/Phoenix-Contact/1190364?qs=QNEnbhJQKvaxxoSFQSEyNA%3D%3D" (id 3) (at 34.29 38.1 0)
+      (effects (font (size 1.27 1.27)) hide)
+    )
+    (pin "1")
+    (pin "2")
+    (pin "3")
+  )
   (symbol (lib_id "power:GND") (at 43.18 153.67 0) (unit 1)
     (in_bom yes) (on_board yes) (fields_autoplaced)
-    (property "Reference" "#PWR0110" (id 0) (at 43.18 160.02 0)
+    (property "Reference" "#PWR0136" (id 0) (at 43.18 160.02 0)
       (effects (font (size 1.27 1.27)) hide)
     )
@@
   (symbol (lib_id "Device:Fuse") (at 43.18 29.21 0) (unit 1)
     (in_bom yes) (on_board yes) (fields_autoplaced)
-    (property "Reference" "F15" (id 0) (at 45.72 27.9399 0)
+    (property "Reference" "F17" (id 0) (at 45.72 27.9399 0)
       (effects (font (size 1.27 1.27)) (justify left))
     )
@@
       (effects (font (size 1.27 1.27)) (justify left))
     )
-    (property "Footprint" "karca_custom_footprints:3588-20 fuse" (id 2) (at 41.402 29.21 90)
+    (property "Footprint" "3588-20:358820" (id 2) (at 41.402 29.21 90)
       (effects (font (size 1.27 1.27)) hide)
     )
@@
     (pin "2")
   )
-  (symbol (lib_id "Connector:Conn_01x03_Female") (at 34.29 38.1 0) (mirror y) (unit 1)
-    (in_bom yes) (on_board yes) (fields_autoplaced)
-    (property "Reference" "J29" (id 0) (at 34.925 30.48 0))
-    (property "Value" "Conn_01x03_Female" (id 1) (at 34.925 33.02 0))
-    (property "Footprint" "Connector_PinSocket_2.54mm:PinSocket_1x03_P2.54mm_Vertical" (id 2) (at 34.29 38.1 0)
-      (effects (font (size 1.27 1.27)) hide)
-    )
-    (property "Datasheet" "~" (id 3) (at 34.29 38.1 0)
+  (symbol (lib_id "Connector:Screw_Terminal_01x03") (at 34.29 147.32 0) (mirror y) (unit 1)
+    (in_bom yes) (on_board yes) (fields_autoplaced)
+    (property "Reference" "J29" (id 0) (at 34.29 140.97 0))
+    (property "Value" "Screw_Terminal_01x03" (id 1) (at 34.29 140.97 0)
+      (effects (font (size 1.27 1.27)) hide)
+    )
+    (property "Footprint" "1190364:1190364" (id 2) (at 34.29 147.32 0)
+      (effects (font (size 1.27 1.27)) hide)
+    )
+    (property "Datasheet" "https://www.mouser.com/ProductDetail/Phoenix-Contact/1190364?qs=QNEnbhJQKvaxxoSFQSEyNA%3D%3D" (id 3) (at 34.29 147.32 0)
       (effects (font (size 1.27 1.27)) hide)
     )
@@
   (symbol (lib_id "power:+5V") (at 43.18 95.25 0) (unit 1)
     (in_bom yes) (on_board yes) (fields_autoplaced)
-    (property "Reference" "#PWR0107" (id 0) (at 43.18 99.06 0)
+    (property "Reference" "#PWR0133" (id 0) (at 43.18 99.06 0)
       (effects (font (size 1.27 1.27)) hide)
     )
@@
   (symbol (lib_id "Device:Fuse") (at 43.18 64.77 0) (unit 1)
     (in_bom yes) (on_board yes) (fields_autoplaced)
-    (property "Reference" "F16" (id 0) (at 45.72 63.4999 0)
+    (property "Reference" "F18" (id 0) (at 45.72 63.4999 0)
       (effects (font (size 1.27 1.27)) (justify left))
     )
@@
       (effects (font (size 1.27 1.27)) (justify left))
     )
-    (property "Footprint" "karca_custom_footprints:3588-20 fuse" (id 2) (at 41.402 64.77 90)
+    (property "Footprint" "3588-20:358820" (id 2) (at 41.402 64.77 90)
       (effects (font (size 1.27 1.27)) hide)
     )
@@
     (pin "2")
   )
-  (symbol (lib_id "Connector:Conn_01x03_Female") (at 34.29 107.95 0) (mirror y) (unit 1)
-    (in_bom yes) (on_board yes) (fields_autoplaced)
-    (property "Reference" "J31" (id 0) (at 34.925 100.33 0))
-    (property "Value" "Conn_01x03_Female" (id 1) (at 34.925 102.87 0))
-    (property "Footprint" "Connector_PinSocket_2.54mm:PinSocket_1x03_P2.54mm_Vertical" (id 2) (at 34.29 107.95 0)
-      (effects (font (size 1.27 1.27)) hide)
-    )
-    (property "Datasheet" "~" (id 3) (at 34.29 107.95 0)
-      (effects (font (size 1.27 1.27)) hide)
-    )
-    (pin "1")
-    (pin "2")
-    (pin "3")
-  )
   (symbol (lib_id "power:GND") (at 43.18 80.01 0) (unit 1)
     (in_bom yes) (on_board yes) (fields_autoplaced)
-    (property "Reference" "#PWR0106" (id 0) (at 43.18 86.36 0)
-      (effects (font (size 1.27 1.27)) hide)
-    )
+    (property "Reference" "#PWR0132" (id 0) (at 43.18 86.36 0)
+      (effects (font (size 1.27 1.27)) hide)
+    )
