File: thermocouples.kicad_sch (KiCad schematic)
At the start: 8 parts, among them J26 Screw_Terminal_01x03, J27 Screw_Terminal_01x03, J28 Screw_Terminal_01x03, J29 Screw_Terminal_01x03

Commit message: some minor schematic cleanup
Changed lines of the file:
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@@
     (company "Rice Eclipse")
   )
-  (wire (pts (xy 39.37 107.95) (xy 49.53 107.95))
-    (stroke (width 0) (type default) (color 0 0 0 0))
-  )
   (wire (pts (xy 39.37 105.41) (xy 43.18 105.41))
     (stroke (width 0) (type default) (color 0 0 0 0))
@@
     (stroke (width 0) (type default) (color 0 0 0 0))
   )
-  (wire (pts (xy 39.37 147.32) (xy 49.53 147.32))
-    (stroke (width 0) (type default) (color 0 0 0 0))
-  )
   (wire (pts (xy 39.37 71.12) (xy 43.18 71.12))
     (stroke (width 0) (type default) (color 0 0 0 0))
@@
     (stroke (width 0) (type default) (color 0 0 0 0))
   )
-  (wire (pts (xy 39.37 38.1) (xy 49.53 38.1))
-    (stroke (width 0) (type default) (color 0 0 0 0))
-  )
   (wire (pts (xy 43.18 110.49) (xy 43.18 114.3))
     (stroke (width 0) (type default) (color 0 0 0 0))
@@
     (stroke (width 0) (type default) (color 0 0 0 0))
   )
-  (wire (pts (xy 39.37 73.66) (xy 49.53 73.66))
-    (stroke (width 0) (type default) (color 0 0 0 0))
-  )
   (wire (pts (xy 43.18 35.56) (xy 43.18 33.02))
     (stroke (width 0) (type default) (color 0 0 0 0))
@@
     (stroke (width 0) (type default) (color 0 0 0 0))
   )
-  (label "TC3" (at 44.45 107.95 0)
-    (effects (font (size 1.27 1.27)) (justify left bottom))
-  )
-  (label "TC2" (at 44.45 73.66 0)
-    (effects (font (size 1.27 1.27)) (justify left bottom))
-  )
-  (label "TC4" (at 44.45 147.32 0)
-    (effects (font (size 1.27 1.27)) (justify left bottom))
-  )
-  (label "TC1" (at 44.45 38.1 0)
-    (effects (font (size 1.27 1.27)) (justify left bottom))
-  )
-  (global_label "TC4" (shape output) (at 49.53 147.32 0) (fields_autoplaced)
+  (global_label "TC4" (shape output) (at 39.37 147.32 0) (fields_autoplaced)
     (effects (font (size 1.27 1.27)) (justify left))
-    (property "Intersheet References" "${INTERSHEET_REFS}" (id 0) (at 55.3902 147.2406 0)
+    (property "Intersheet References" "${INTERSHEET_REFS}" (id 0) (at 45.2302 147.2406 0)
       (effects (font (size 1.27 1.27)) (justify left) hide)
     )
   )
-  (global_label "TC3" (shape output) (at 49.53 107.95 0) (fields_autoplaced)
+  (global_label "TC3" (shape output) (at 39.37 107.95 0) (fields_autoplaced)
     (effects (font (size 1.27 1.27)) (justify left))
-    (property "Intersheet References" "${INTERSHEET_REFS}" (id 0) (at 55.3902 107.8706 0)
+    (property "Intersheet References" "${INTERSHEET_REFS}" (id 0) (at 45.2302 107.8706 0)
       (effects (font (size 1.27 1.27)) (justify left) hide)
     )
   )
-  (global_label "TC2" (shape output) (at 49.53 73.66 0) (fields_autoplaced)
+  (global_label "TC2" (shape output) (at 39.37 73.66 0) (fields_autoplaced)
     (effects (font (size 1.27 1.27)) (justify left))
-    (property "Intersheet References" "${INTERSHEET_REFS}" (id 0) (at 55.3902 73.5806 0)
+    (property "Intersheet References" "${INTERSHEET_REFS}" (id 0) (at 45.2302 73.5806 0)
       (effects (font (size 1.27 1.27)) (justify left) hide)
     )
   )
-  (global_label "TC1" (shape output) (at 49.53 38.1 0) (fields_autoplaced)
+  (global_label "TC1" (shape output) (at 39.37 38.1 0) (fields_autoplaced)
     (effects (font (size 1.27 1.27)) (justify left))
-    (property "Intersheet References" "${INTERSHEET_REFS}" (id 0) (at 55.3902 38.0206 0)
+    (property "Intersheet References" "${INTERSHEET_REFS}" (id 0) (at 45.2302 38.0206 0)
       (effects (font (size 1.27 1.27)) (justify left) hide)
     )
@@
       (effects (font (size 1.27 1.27)) hide)
     )
-    (property "Datasheet" "https://www.mouser.com/ProductDetail/Phoenix-Contact/1190364?qs=QNEnbhJQKvaxxoSFQSEyNA%3D%3D" (id 3) (at 34.29 73.66 0)
+    (property "Datasheet" "~" (id 3) (at 34.29 73.66 0)
       (effects (font (size 1.27 1.27)) hide)
     )
@@
       (effects (font (size 1.27 1.27)) hide)
     )
-    (property "Datasheet" "https://www.mouser.com/datasheet/2/215/588-20-1622270.pdf" (id 3) (at 43.18 99.06 0)
+    (property "Datasheet" "~" (id 3) (at 43.18 99.06 0)
       (effects (font (size 1.27 1.27)) hide)
     )
@@
       (effects (font (size 1.27 1.27)) hide)
     )
-    (property "Datasheet" "https://www.mouser.com/datasheet/2/215/588-20-1622270.pdf" (id 3) (at 43.18 138.43 0)
+    (property "Datasheet" "~" (id 3) (at 43.18 138.43 0)
       (effects (font (size 1.27 1.27)) hide)
     )
@@
       (effects (font (size 1.27 1.27)) hide)
     )
-    (property "Datasheet" "https://www.mouser.com/ProductDetail/Phoenix-Contact/1190364?qs=QNEnbhJQKvaxxoSFQSEyNA%3D%3D" (id 3) (at 34.29 107.95 0)
+    (property "Datasheet" "~" (id 3) (at 34.29 107.95 0)
       (effects (font (size 1.27 1.27)) hide)
     )
@@
       (effects (font (size 1.27 1.27)) hide)
     )
-    (property "Datasheet" "https://www.mouser.com/ProductDetail/Phoenix-Contact/1190364?qs=QNEnbhJQKvaxxoSFQSEyNA%3D%3D" (id 3) (at 34.29 38.1 0)
+    (property "Datasheet" "~" (id 3) (at 34.29 38.1 0)
       (effects (font (size 1.27 1.27)) hide)
     )
@@
       (effects (font (size 1.27 1.27)) hide)
     )
-    (property "Datasheet" "https://www.mouser.com/datasheet/2/215/588-20-1622270.pdf" (id 3) (at 43.18 29.21 0)
+    (property "Datasheet" "~" (id 3) (at 43.18 29.21 0)
       (effects (font (size 1.27 1.27)) hide)
     )
@@
       (effects (font (size 1.27 1.27)) hide)
     )
-    (property "Datasheet" "https://www.mouser.com/ProductDetail/Phoenix-Contact/1190364?qs=QNEnbhJQKvaxxoSFQSEyNA%3D%3D" (id 3) (at 34.29 147.32 0)
+    (property "Datasheet" "~" (id 3) (at 34.29 147.32 0)
       (effects (font (size 1.27 1.27)) hide)
     )
@@
       (effects (font (size 1.27 1.27)) hide)
     )
-    (property "Datasheet" "https://www.mouser.com/datasheet/2/215/588-20-1622270.pdf" (id 3) (at 43.18 64.77 0)
-      (effects (font (size 1.27 1.27)) hide)
-    )
+    (property "Datasheet" "~" (id 3) (at 43.18 64.77 0)
+      (effects (font (size 1.27 1.27)) hide)
+    )

Commit message: shuffle around some parts
Parts:
- F17, F18, F19, F20: value 3588-20 -> 178.6165; footprint 3588-20:358820 -> 178.6165:17861650002
Changed lines of the file:
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@@
       (effects (font (size 1.27 1.27)) (justify left))
     )
-    (property "Value" "3588-20" (id 1) (at 45.72 100.3299 0)
+    (property "Value" "178.6165" (id 1) (at 45.72 100.3299 0)
       (effects (font (size 1.27 1.27)) (justify left))
     )
-    (property "Footprint" "3588-20:358820" (id 2) (at 41.402 99.06 90)
+    (property "Footprint" "178.6165:17861650002" (id 2) (at 41.402 99.06 90)
       (effects (font (size 1.27 1.27)) hide)
     )
@@
       (effects (font (size 1.27 1.27)) (justify left))
     )
-    (property "Value" "3588-20" (id 1) (at 45.72 139.6999 0)
+    (property "Value" "178.6165" (id 1) (at 45.72 139.6999 0)
       (effects (font (size 1.27 1.27)) (justify left))
     )
-    (property "Footprint" "3588-20:358820" (id 2) (at 41.402 138.43 90)
+    (property "Footprint" "178.6165:17861650002" (id 2) (at 41.402 138.43 90)
       (effects (font (size 1.27 1.27)) hide)
     )
@@
       (effects (font (size 1.27 1.27)) (justify left))
     )
-    (property "Value" "3588-20" (id 1) (at 45.72 30.4799 0)
+    (property "Value" "178.6165" (id 1) (at 45.72 30.4799 0)
       (effects (font (size 1.27 1.27)) (justify left))
     )
-    (property "Footprint" "3588-20:358820" (id 2) (at 41.402 29.21 90)
+    (property "Footprint" "178.6165:17861650002" (id 2) (at 41.402 29.21 90)
       (effects (font (size 1.27 1.27)) hide)
     )
@@
       (effects (font (size 1.27 1.27)) (justify left))
     )
-    (property "Value" "3588-20" (id 1) (at 45.72 66.0399 0)
+    (property "Value" "178.6165" (id 1) (at 45.72 66.0399 0)
       (effects (font (size 1.27 1.27)) (justify left))
     )
-    (property "Footprint" "3588-20:358820" (id 2) (at 41.402 64.77 90)
+    (property "Footprint" "178.6165:17861650002" (id 2) (at 41.402 64.77 90)
       (effects (font (size 1.27 1.27)) hide)
     )

Commit message: laid out ignition and PTs
Parts:
- renumbered J26 to CON_TC1, J27 to CON_TC2, J28 to CON_TC3, J29 to CON_TC4
Changed lines of the file:
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@@
   (symbol (lib_id "Connector:Screw_Terminal_01x03") (at 34.29 73.66 0) (mirror y) (unit 1)
     (in_bom yes) (on_board yes) (fields_autoplaced)
-    (property "Reference" "J27" (id 0) (at 34.29 67.31 0))
+    (property "Reference" "CON_TC2" (id 0) (at 34.29 67.31 0))
     (property "Value" "Screw_Terminal_01x03" (id 1) (at 34.29 67.31 0)
       (effects (font (size 1.27 1.27)) hide)
@@
   (symbol (lib_id "Connector:Screw_Terminal_01x03") (at 34.29 107.95 0) (mirror y) (unit 1)
     (in_bom yes) (on_board yes) (fields_autoplaced)
-    (property "Reference" "J28" (id 0) (at 34.29 101.6 0))
+    (property "Reference" "CON_TC3" (id 0) (at 34.29 101.6 0))
     (property "Value" "Screw_Terminal_01x03" (id 1) (at 34.29 101.6 0)
       (effects (font (size 1.27 1.27)) hide)
@@
   (symbol (lib_id "Connector:Screw_Terminal_01x03") (at 34.29 38.1 0) (mirror y) (unit 1)
     (in_bom yes) (on_board yes) (fields_autoplaced)
-    (property "Reference" "J26" (id 0) (at 34.29 31.75 0))
+    (property "Reference" "CON_TC1" (id 0) (at 34.29 31.75 0))
     (property "Value" "Screw_Terminal_01x03" (id 1) (at 34.29 31.75 0)
       (effects (font (size 1.27 1.27)) hide)
@@
   (symbol (lib_id "Connector:Screw_Terminal_01x03") (at 34.29 147.32 0) (mirror y) (unit 1)
     (in_bom yes) (on_board yes) (fields_autoplaced)
-    (property "Reference" "J29" (id 0) (at 34.29 140.97 0))
+    (property "Reference" "CON_TC4" (id 0) (at 34.29 140.97 0))
     (property "Value" "Screw_Terminal_01x03" (id 1) (at 34.29 140.97 0)
       (effects (font (size 1.27 1.27)) hide)
