File: thermocouples.kicad_sch (KiCad schematic)
At the start: 8 parts

Commit message: finish putting shit together
Parts:
- removed F17, F18, F19, F20: 178.6165, 178.6165:17861650002, symbol Device:Fuse
Connections:
- net +5V: now also CON_TC1.1 (Pin_1), CON_TC2.1 (Pin_1), CON_TC3.1 (Pin_1), CON_TC4.1 (Pin_1)
Changed lines of the file:
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@@
     (pin "3")
   )
-  (symbol (lib_id "power:+5V") (at 43.18 134.62 0) (unit 1)
+  (symbol (lib_id "power:+5V") (at 43.18 142.24 0) (unit 1)
     (in_bom yes) (on_board yes) (fields_autoplaced)
-    (property "Reference" "#PWR0135" (id 0) (at 43.18 138.43 0)
+    (property "Reference" "#PWR0135" (id 0) (at 43.18 146.05 0)
       (effects (font (size 1.27 1.27)) hide)
     )
-    (property "Value" "+5V" (id 1) (at 43.18 129.54 0))
-    (property "Footprint" "" (id 2) (at 43.18 134.62 0)
+    (property "Value" "+5V" (id 1) (at 43.18 137.16 0))
+    (property "Footprint" "" (id 2) (at 43.18 142.24 0)
       (effects (font (size 1.27 1.27)) hide)
     )
-    (property "Datasheet" "" (id 3) (at 43.18 134.62 0)
+    (property "Datasheet" "" (id 3) (at 43.18 142.24 0)
       (effects (font (size 1.27 1.27)) hide)
     )
     (pin "1")
   )
-  (symbol (lib_id "Device:Fuse") (at 43.18 99.06 0) (unit 1)
+  (symbol (lib_id "power:+5V") (at 43.18 68.58 0) (unit 1)
     (in_bom yes) (on_board yes) (fields_autoplaced)
-    (property "Reference" "F19" (id 0) (at 45.72 97.7899 0)
-      (effects (font (size 1.27 1.27)) (justify left))
-    )
-    (property "Value" "178.6165" (id 1) (at 45.72 100.3299 0)
-      (effects (font (size 1.27 1.27)) (justify left))
-    )
-    (property "Footprint" "178.6165:17861650002" (id 2) (at 41.402 99.06 90)
+    (property "Reference" "#PWR0131" (id 0) (at 43.18 72.39 0)
       (effects (font (size 1.27 1.27)) hide)
     )
-    (property "Datasheet" "~" (id 3) (at 43.18 99.06 0)
+    (property "Value" "+5V" (id 1) (at 43.18 63.5 0))
+    (property "Footprint" "" (id 2) (at 43.18 68.58 0)
       (effects (font (size 1.27 1.27)) hide)
     )
-    (pin "1")
-    (pin "2")
-  )
-  (symbol (lib_id "power:+5V") (at 43.18 60.96 0) (unit 1)
-    (in_bom yes) (on_board yes) (fields_autoplaced)
-    (property "Reference" "#PWR0131" (id 0) (at 43.18 64.77 0)
-      (effects (font (size 1.27 1.27)) hide)
-    )
-    (property "Value" "+5V" (id 1) (at 43.18 55.88 0))
-    (property "Footprint" "" (id 2) (at 43.18 60.96 0)
-      (effects (font (size 1.27 1.27)) hide)
-    )
-    (property "Datasheet" "" (id 3) (at 43.18 60.96 0)
+    (property "Datasheet" "" (id 3) (at 43.18 68.58 0)
       (effects (font (size 1.27 1.27)) hide)
     )
     (pin "1")
   )
-  (symbol (lib_id "power:+5V") (at 43.18 25.4 0) (unit 1)
+  (symbol (lib_id "power:+5V") (at 43.18 33.02 0) (unit 1)
     (in_bom yes) (on_board yes) (fields_autoplaced)
-    (property "Reference" "#PWR0129" (id 0) (at 43.18 29.21 0)
+    (property "Reference" "#PWR0129" (id 0) (at 43.18 36.83 0)
       (effects (font (size 1.27 1.27)) hide)
     )
-    (property "Value" "+5V" (id 1) (at 43.18 20.32 0))
-    (property "Footprint" "" (id 2) (at 43.18 25.4 0)
+    (property "Value" "+5V" (id 1) (at 43.18 27.94 0))
+    (property "Footprint" "" (id 2) (at 43.18 33.02 0)
       (effects (font (size 1.27 1.27)) hide)
     )
-    (property "Datasheet" "" (id 3) (at 43.18 25.4 0)
+    (property "Datasheet" "" (id 3) (at 43.18 33.02 0)
       (effects (font (size 1.27 1.27)) hide)
     )
     (pin "1")
-  )
-  (symbol (lib_id "Device:Fuse") (at 43.18 138.43 0) (unit 1)
-    (in_bom yes) (on_board yes) (fields_autoplaced)
-    (property "Reference" "F20" (id 0) (at 45.72 137.1599 0)
-      (effects (font (size 1.27 1.27)) (justify left))
-    )
-    (property "Value" "178.6165" (id 1) (at 45.72 139.6999 0)
-      (effects (font (size 1.27 1.27)) (justify left))
-    )
-    (property "Footprint" "178.6165:17861650002" (id 2) (at 41.402 138.43 90)
-      (effects (font (size 1.27 1.27)) hide)
-    )
-    (property "Datasheet" "~" (id 3) (at 43.18 138.43 0)
-      (effects (font (size 1.27 1.27)) hide)
-    )
-    (pin "1")
-    (pin "2")
   )
   (symbol (lib_id "power:GND") (at 43.18 44.45 0) (unit 1)
@@
     (pin "1")
   )
-  (symbol (lib_id "Device:Fuse") (at 43.18 29.21 0) (unit 1)
-    (in_bom yes) (on_board yes) (fields_autoplaced)
-    (property "Reference" "F17" (id 0) (at 45.72 27.9399 0)
-      (effects (font (size 1.27 1.27)) (justify left))
-    )
-    (property "Value" "178.6165" (id 1) (at 45.72 30.4799 0)
-      (effects (font (size 1.27 1.27)) (justify left))
-    )
-    (property "Footprint" "178.6165:17861650002" (id 2) (at 41.402 29.21 90)
-      (effects (font (size 1.27 1.27)) hide)
-    )
-    (property "Datasheet" "~" (id 3) (at 43.18 29.21 0)
-      (effects (font (size 1.27 1.27)) hide)
-    )
-    (pin "1")
-    (pin "2")
-  )
   (symbol (lib_id "Connector:Screw_Terminal_01x03") (at 34.29 147.32 0) (mirror y) (unit 1)
     (in_bom yes) (on_board yes) (fields_autoplaced)
@@
     (pin "3")
   )
-  (symbol (lib_id "power:+5V") (at 43.18 95.25 0) (unit 1)
+  (symbol (lib_id "power:+5V") (at 43.18 102.87 0) (unit 1)
     (in_bom yes) (on_board yes) (fields_autoplaced)
-    (property "Reference" "#PWR0133" (id 0) (at 43.18 99.06 0)
+    (property "Reference" "#PWR0133" (id 0) (at 43.18 106.68 0)
       (effects (font (size 1.27 1.27)) hide)
     )
-    (property "Value" "+5V" (id 1) (at 43.18 90.17 0))
-    (property "Footprint" "" (id 2) (at 43.18 95.25 0)
+    (property "Value" "+5V" (id 1) (at 43.18 97.79 0))
+    (property "Footprint" "" (id 2) (at 43.18 102.87 0)
       (effects (font (size 1.27 1.27)) hide)
     )
-    (property "Datasheet" "" (id 3) (at 43.18 95.25 0)
+    (property "Datasheet" "" (id 3) (at 43.18 102.87 0)
       (effects (font (size 1.27 1.27)) hide)
     )
     (pin "1")
   )
-  (symbol (lib_id "Device:Fuse") (at 43.18 64.77 0) (unit 1)
-    (in_bom yes) (on_board yes) (fields_autoplaced)
-    (property "Reference" "F18" (id 0) (at 45.72 63.4999 0)
-      (effects (font (size 1.27 1.27)) (justify left))
-    )
-    (property "Value" "178.6165" (id 1) (at 45.72 66.0399 0)
-      (effects (font (size 1.27 1.27)) (justify left))
-    )
-    (property "Footprint" "178.6165:17861650002" (id 2) (at 41.402 64.77 90)
-      (effects (font (size 1.27 1.27)) hide)
-    )
-    (property "Datasheet" "~" (id 3) (at 43.18 64.77 0)
-      (effects (font (size 1.27 1.27)) hide)
-    )
-    (pin "1")
-    (pin "2")
-  )
   (symbol (lib_id "power:GND") (at 43.18 80.01 0) (unit 1)

Commit message: done schematiccing after design review
Parts:
- added ADC3: MCP3208-CI/SL, Package_SO:SOIC-16_3.9x9.9mm_P1.27mm, symbol Analog_ADC:MCP3208
- added C20: 100n, Capacitor_SMD:C_1206_3216Metric, symbol Device:C
- added D42, D43, D44, D45, D46, D47, D48, D49: CDBA340-HF, Diode_SMD:D_SMA, symbol Device:D_Schottky
- added J8: Conn_01x08_Female, Connector_PinSocket_2.54mm:PinSocket_1x08_P2.54mm_Vertical, symbol Connector:Conn_01x08_Female
Connections:
- net +5V: now also ADC3.15 (Vref), ADC3.16 (Vdd), C20.2
- net GND: now also ADC3.14 (AGND), ADC3.9 (DGND), C20.1, D43.2 (A), D45.2 (A), D47.2 (A), D49.2 (A)
- net TC1: now also ADC3.1 (CH0), D42.2 (A), D43.1 (K), J8.1 (Pin_1)
- net TC2: now also ADC3.2 (CH1), D44.2 (A), D45.1 (K), J8.2 (Pin_2)
- net TC3: now also ADC3.3 (CH2), D46.2 (A), D47.1 (K), J8.3 (Pin_3)
- net TC4: now also ADC3.4 (CH3), D48.2 (A), D49.1 (K), J8.4 (Pin_4)
- new net: ADC3.5 (CH4), J8.5 (Pin_5)
- new net: ADC3.6 (CH5), J8.6 (Pin_6)
- new net: ADC3.7 (CH6), J8.7 (Pin_7)
- new net: ADC3.8 (CH7), J8.8 (Pin_8)
- new net +10V: D42.1 (K), D44.1 (K), D46.1 (K), D48.1 (K)
- new net CS: ADC3.10 (~{CS}/SHDN)
- new net SPI_CLK: ADC3.13 (CLK)
- new net SPI_MISO: ADC3.12 (Dout)
- new net SPI_MOSI: ADC3.11 (Din)

Commit message: cleaned up PT footprint
Parts:
- removed CON_TC1, CON_TC2, CON_TC3, CON_TC4: Screw_Terminal_01x03, 1190364:1190364, symbol Connector:Screw_Terminal_01x03
- added J9: Screw_Terminal_01x12, symbol Connector:Screw_Terminal_01x12
Connections:
- net +5V: now also J9.1 (Pin_1), J9.10 (Pin_10), J9.4 (Pin_4), J9.7 (Pin_7)
- net GND: now also J9.12 (Pin_12), J9.3 (Pin_3), J9.6 (Pin_6), J9.9 (Pin_9)
- net TC1: now also J9.2 (Pin_2)
- net TC2: now also J9.5 (Pin_5)
- net TC3: now also J9.8 (Pin_8)
- net TC4: now also J9.11 (Pin_11)
Other:
- moved on the sheet: D46, D47

Commit message: ready for fab
Parts:
- J9: footprint (none) -> 1190374:1190374
Connections:
- net +10V is gone; now on net +5V: D42.1 (K), D44.1 (K), D46.1 (K), D48.1 (K)
Changed lines of the file:
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@@
+    (pin "1")
+  )
+  (symbol (lib_id "power:+5V") (at 48.895 139.7 0) (unit 1)
+    (in_bom yes) (on_board yes) (fields_autoplaced)
+    (property "Reference" "#PWR?" (id 0) (at 48.895 143.51 0)
+      (effects (font (size 1.27 1.27)) hide)
+    )
+    (property "Value" "+5V" (id 1) (at 48.895 134.62 0))
+    (property "Footprint" "" (id 2) (at 48.895 139.7 0)
+      (effects (font (size 1.27 1.27)) hide)
+    )
+    (property "Datasheet" "" (id 3) (at 48.895 139.7 0)
+      (effects (font (size 1.27 1.27)) hide)
+    )
     (pin "1")
   )
@@
     (pin "8")
   )
+  (symbol (lib_id "power:+5V") (at 48.895 66.04 0) (unit 1)
+    (in_bom yes) (on_board yes) (fields_autoplaced)
+    (property "Reference" "#PWR?" (id 0) (at 48.895 69.85 0)
+      (effects (font (size 1.27 1.27)) hide)
+    )
+    (property "Value" "+5V" (id 1) (at 48.895 60.96 0))
+    (property "Footprint" "" (id 2) (at 48.895 66.04 0)
+      (effects (font (size 1.27 1.27)) hide)
+    )
+    (property "Datasheet" "" (id 3) (at 48.895 66.04 0)
+      (effects (font (size 1.27 1.27)) hide)
+    )
+    (pin "1")
+  )
   (symbol (lib_id "Device:C") (at 133.35 82.55 270) (unit 1)
     (in_bom yes) (on_board yes) (fields_autoplaced)
@@
     )
     (property "Datasheet" "" (id 3) (at 48.895 81.28 0)
-      (effects (font (size 1.27 1.27)) hide)
-    )
-    (pin "1")
-  )
-  (symbol (lib_id "power:+10V") (at 48.895 139.7 0) (unit 1)
-    (in_bom yes) (on_board yes) (fields_autoplaced)
-    (property "Reference" "#PWR0120" (id 0) (at 48.895 143.51 0)
-      (effects (font (size 1.27 1.27)) hide)
-    )
-    (property "Value" "+10V" (id 1) (at 48.895 134.62 0))
-    (property "Footprint" "" (id 2) (at 48.895 139.7 0)
-      (effects (font (size 1.27 1.27)) hide)
-    )
-    (property "Datasheet" "" (id 3) (at 48.895 139.7 0)
       (effects (font (size 1.27 1.27)) hide)
     )
@@
     (pin "2")
   )
+  (symbol (lib_id "power:+5V") (at 48.895 105.41 0) (unit 1)
+    (in_bom yes) (on_board yes) (fields_autoplaced)
+    (property "Reference" "#PWR?" (id 0) (at 48.895 109.22 0)
+      (effects (font (size 1.27 1.27)) hide)
+    )
+    (property "Value" "+5V" (id 1) (at 48.895 100.33 0))
+    (property "Footprint" "" (id 2) (at 48.895 105.41 0)
+      (effects (font (size 1.27 1.27)) hide)
+    )
+    (property "Datasheet" "" (id 3) (at 48.895 105.41 0)
+      (effects (font (size 1.27 1.27)) hide)
+    )
+    (pin "1")
+  )
   (symbol (lib_id "Device:D_Schottky") (at 48.895 77.47 270) (unit 1)
     (in_bom yes) (on_board yes)
@@
     (pin "1")
     (pin "2")
-  )
-  (symbol (lib_id "power:+10V") (at 48.895 66.04 0) (unit 1)
-    (in_bom yes) (on_board yes) (fields_autoplaced)
-    (property "Reference" "#PWR0110" (id 0) (at 48.895 69.85 0)
-      (effects (font (size 1.27 1.27)) hide)
-    )
-    (property "Value" "+10V" (id 1) (at 48.895 60.96 0))
-    (property "Footprint" "" (id 2) (at 48.895 66.04 0)
-      (effects (font (size 1.27 1.27)) hide)
-    )
-    (property "Datasheet" "" (id 3) (at 48.895 66.04 0)
-      (effects (font (size 1.27 1.27)) hide)
-    )
-    (pin "1")
-  )
-  (symbol (lib_id "power:+10V") (at 48.895 105.41 0) (unit 1)
-    (in_bom yes) (on_board yes) (fields_autoplaced)
-    (property "Reference" "#PWR0112" (id 0) (at 48.895 109.22 0)
-      (effects (font (size 1.27 1.27)) hide)
-    )
-    (property "Value" "+10V" (id 1) (at 48.895 100.33 0))
-    (property "Footprint" "" (id 2) (at 48.895 105.41 0)
-      (effects (font (size 1.27 1.27)) hide)
-    )
-    (property "Datasheet" "" (id 3) (at 48.895 105.41 0)
-      (effects (font (size 1.27 1.27)) hide)
-    )
-    (pin "1")
   )
   (symbol (lib_id "Connector:Screw_Terminal_01x12") (at 20.955 107.95 0) (mirror y) (unit 1)
@@
     (property "Reference" "J9" (id 0) (at 20.955 88.265 0))
     (property "Value" "Screw_Terminal_01x12" (id 1) (at 20.955 90.805 0))
-    (property "Footprint" "" (id 2) (at 20.955 107.95 0)
+    (property "Footprint" "1190374:1190374" (id 2) (at 20.955 107.95 0)
       (effects (font (size 1.27 1.27)) hide)
     )
@@
     (pin "9")
   )
+  (symbol (lib_id "power:+5V") (at 48.895 30.48 0) (unit 1)
+    (in_bom yes) (on_board yes) (fields_autoplaced)
+    (property "Reference" "#PWR?" (id 0) (at 48.895 34.29 0)
+      (effects (font (size 1.27 1.27)) hide)
+    )
+    (property "Value" "+5V" (id 1) (at 48.895 25.4 0))
+    (property "Footprint" "" (id 2) (at 48.895 30.48 0)
+      (effects (font (size 1.27 1.27)) hide)
+    )
+    (property "Datasheet" "" (id 3) (at 48.895 30.48 0)
+      (effects (font (size 1.27 1.27)) hide)
+    )
+    (pin "1")
+  )
   (symbol (lib_id "power:GND") (at 29.21 125.73 0) (mirror y) (unit 1)
     (in_bom yes) (on_board yes) (fields_autoplaced)
@@
       (effects (font (size 1.27 1.27)) hide)
     )
-    (pin "1")
-  )
-  (symbol (lib_id "power:+10V") (at 48.895 30.48 0) (unit 1)
-    (in_bom yes) (on_board yes) (fields_autoplaced)
-    (property "Reference" "#PWR0108" (id 0) (at 48.895 34.29 0)
-      (effects (font (size 1.27 1.27)) hide)
-    )
-    (property "Value" "+10V" (id 1) (at 48.895 25.4 0))
-    (property "Footprint" "" (id 2) (at 48.895 30.48 0)
-      (effects (font (size 1.27 1.27)) hide)
-    )
-    (property "Datasheet" "" (id 3) (at 48.895 30.48 0)
-      (effects (font (size 1.27 1.27)) hide)
-    )

Commit message: my body is a machine that takes in peanut m&ms and puts out rocket engine controllers
Parts:
- ADC3: LCSC (none) -> C16939
- C20: LCSC (none) -> C377067
- D42, D43, D44, D45, D46, D47, D48, D49: LCSC (none) -> C14996
Changed lines of the file:
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@@
+      (effects (font (size 1.27 1.27)) hide)
+    )
+    (property "LCSC" "C14996" (id 4) (at 48.895 109.22 0)
       (effects (font (size 1.27 1.27)) hide)
     )
@@
     )
     (property "Datasheet" "~" (id 3) (at 48.895 69.85 0)
+      (effects (font (size 1.27 1.27)) hide)
+    )
+    (property "LCSC" "C14996" (id 4) (at 48.895 69.85 0)
       (effects (font (size 1.27 1.27)) hide)
     )
@@
       (effects (font (size 1.27 1.27)) hide)
     )
+    (property "LCSC" "C377067" (id 4) (at 133.35 82.55 0)
+      (effects (font (size 1.27 1.27)) hide)
+    )
     (pin "1")
     (pin "2")
@@
       (effects (font (size 1.27 1.27)) hide)
     )
+    (property "LCSC" "C14996" (id 4) (at 48.895 116.84 0)
+      (effects (font (size 1.27 1.27)) hide)
+    )
     (pin "1")
     (pin "2")
@@
       (effects (font (size 1.27 1.27)) hide)
     )
+    (property "LCSC" "C14996" (id 4) (at 48.895 41.91 0)
+      (effects (font (size 1.27 1.27)) hide)
+    )
     (pin "1")
     (pin "2")
@@
       (effects (font (size 1.27 1.27)) hide)
     )
+    (property "LCSC" "C14996" (id 4) (at 48.895 151.13 0)
+      (effects (font (size 1.27 1.27)) hide)
+    )
     (pin "1")
     (pin "2")
@@
     )
     (property "Datasheet" "http://ww1.microchip.com/downloads/en/DeviceDoc/21298c.pdf" (id 3) (at 127 95.25 0)
+      (effects (font (size 1.27 1.27)) hide)
+    )
+    (property "LCSC" "C16939" (id 4) (at 124.46 97.79 0)
       (effects (font (size 1.27 1.27)) hide)
     )
@@
       (effects (font (size 1.27 1.27)) hide)
     )
+    (property "LCSC" "C14996" (id 4) (at 48.895 34.29 0)
+      (effects (font (size 1.27 1.27)) hide)
+    )
     (pin "1")
     (pin "2")
@@
       (effects (font (size 1.27 1.27)) hide)
     )
+    (property "LCSC" "C14996" (id 4) (at 48.895 143.51 0)
+      (effects (font (size 1.27 1.27)) hide)
+    )
     (pin "1")
     (pin "2")
@@
       (effects (font (size 1.27 1.27)) hide)
     )
+    (property "LCSC" "C14996" (id 4) (at 48.895 77.47 0)
+      (effects (font (size 1.27 1.27)) hide)
+    )
